File: CES/ALU.sch (KiCad schematic (older format))
At the start: 40 parts

Commit message: Registers
Connections:
- net VDB14 is gone; now on net GND: U?.14 (I0c)
- net VDB15 is gone; now on net GND: U?.11 (I0d)
- net GND: now also U?.10 (I1d), U?.13 (I1c)
- net SS14: no longer U?.13 (I1c)
- net SS15: no longer U?.10 (I1d)
- net SME14: no longer names the net of U?.12 (Zc)
- net SME15: no longer names the net of U?.9 (Zd)
- no-connect marks 0 -> 2
Changed lines of the file:
@@
 $Descr A4 8268 11693 portrait
 encoding utf-8
-Sheet 2 11
+Sheet 2 13
 Title ""
 Date ""
@@
 Wire Wire Line
 	5150 7900 5550 7900
-Text GLabel 5150 8200 0    50   Input ~ 0
-SS14
-Wire Wire Line
-	5150 8200 5550 8200
-Text GLabel 5150 8500 0    50   Input ~ 0
-SS15
-Wire Wire Line
-	5150 8500 5550 8500
 Text GLabel 5150 7500 0    50   Input ~ 0
 VDB12
@@
 Wire Wire Line
 	5150 7800 5550 7800
-Text GLabel 5150 8100 0    50   Input ~ 0
-VDB14
-Wire Wire Line
-	5150 8100 5550 8100
-Text GLabel 5150 8400 0    50   Input ~ 0
-VDB15
-Wire Wire Line
-	5150 8400 5550 8400
 $Comp
 L power:GND #PWR?
@@
 Wire Wire Line
 	6550 7800 6700 7800
-Text GLabel 6700 8100 2    50   Output ~ 0
-SME14
-Wire Wire Line
-	6550 8100 6700 8100
-Text GLabel 6700 8400 2    50   Output ~ 0
-SME15
-Wire Wire Line
-	6550 8400 6700 8400
 Wire Wire Line
 	4000 8900 4000 8750
@@
 Wire Wire Line
 	1500 9650 1250 9650
+NoConn ~ 6550 8400
+NoConn ~ 6550 8100
+Wire Wire Line
+	5400 8800 5400 8500
+Connection ~ 5400 8800
+Wire Wire Line
+	5400 8100 5550 8100
+Connection ~ 5400 8200
+Wire Wire Line
+	5400 8200 5550 8200
+Wire Wire Line
+	5400 8200 5400 8100
+Connection ~ 5400 8400
+Wire Wire Line
+	5400 8400 5550 8400
+Wire Wire Line
+	5400 8400 5400 8200
+Connection ~ 5400 8500
+Wire Wire Line
+	5400 8500 5550 8500
+Wire Wire Line
+	5400 8500 5400 8400
 $EndSCHEMATC
