File: CES/ALU.sch (KiCad schematic (older format))
At the start: 40 parts

Commit message: Adding 74HC versions of 74LS chips
Parts:
- removed U?: SM1, symbol 74xx:74LS283
- removed U?: SM3, symbol 74xx:74LS283
- removed U?: SM2, symbol 74xx:74LS283
- removed U?: SM4, symbol 74xx:74LS283
- removed U?: ME1, symbol 74xx:74LS257
- removed U?: ME2, symbol 74xx:74LS257
- removed U?: ME3, symbol 74xx:74LS257
- removed U?: ME4, symbol 74xx:74LS257
- added U?: ME1, symbol CES:74HC257
- added U?: ME2, symbol CES:74HC257
- added U?: ME3, symbol CES:74HC257
- added U?: ME4, symbol CES:74HC257
- added U?: SM1, symbol CES:74HC283
- added U?: SM2, symbol CES:74HC283
- added U?: SM3, symbol CES:74HC283
- added U?: SM4, symbol CES:74HC283
Changed lines of the file:
@@
-$EndComp
-$Comp
-L 74xx:74LS283 U?
-U 1 1 617654FA
-P 3450 1400
-F 0 "U?" H 3650 2050 50  0000 C CNN
-F 1 "SM1" H 3450 1400 50  0000 C CNN
-F 2 "" H 3450 1400 50  0001 C CNN
-F 3 "http://www.ti.com/lit/gpn/sn74LS283" H 3450 1400 50  0001 C CNN
-	1    3450 1400
-	1    0    0    -1
-$EndComp
-$Comp
-L 74xx:74LS283 U?
-U 1 1 61766086
-P 3450 5200
-F 0 "U?" H 3700 5900 50  0000 C CNN
-F 1 "SM3" H 3450 5200 50  0000 C CNN
-F 2 "" H 3450 5200 50  0001 C CNN
-F 3 "http://www.ti.com/lit/gpn/sn74LS283" H 3450 5200 50  0001 C CNN
-	1    3450 5200
-	1    0    0    -1
-$EndComp
-$Comp
-L 74xx:74LS283 U?
-U 1 1 617670F7
-P 3450 3300
-F 0 "U?" H 3700 3950 50  0000 C CNN
-F 1 "SM2" H 3450 3300 50  0000 C CNN
-F 2 "" H 3450 3300 50  0001 C CNN
-F 3 "http://www.ti.com/lit/gpn/sn74LS283" H 3450 3300 50  0001 C CNN
-	1    3450 3300
-	1    0    0    -1
-$EndComp
-$Comp
-L 74xx:74LS283 U?
-U 1 1 617685A6
-P 3450 7150
-F 0 "U?" H 3700 7800 50  0000 C CNN
-F 1 "SM4" H 3450 7150 50  0000 C CNN
-F 2 "" H 3450 7150 50  0001 C CNN
-F 3 "http://www.ti.com/lit/gpn/sn74LS283" H 3450 7150 50  0001 C CNN
-	1    3450 7150
-	1    0    0    -1
-$EndComp
-$Comp
-L 74xx:74LS257 U?
-U 1 1 6176964F
-P 6050 1500
-F 0 "U?" H 6300 2250 50  0000 C CNN
-F 1 "ME1" H 6050 1500 50  0000 C CNN
-F 2 "" H 6050 1500 50  0001 C CNN
-F 3 "http://www.ti.com/lit/gpn/sn74LS257" H 6050 1500 50  0001 C CNN
-	1    6050 1500
-	1    0    0    -1
-$EndComp
-$Comp
-L 74xx:74LS257 U?
-U 1 1 6176B14B
-P 6050 3700
-F 0 "U?" H 6300 4450 50  0000 C CNN
-F 1 "ME2" H 6050 3700 50  0000 C CNN
-F 2 "" H 6050 3700 50  0001 C CNN
-F 3 "http://www.ti.com/lit/gpn/sn74LS257" H 6050 3700 50  0001 C CNN
-	1    6050 3700
-	1    0    0    -1
-$EndComp
-$Comp
-L 74xx:74LS257 U?
-U 1 1 6176CCA9
-P 6050 5900
-F 0 "U?" H 6300 6650 50  0000 C CNN
-F 1 "ME3" H 6050 5900 50  0000 C CNN
-F 2 "" H 6050 5900 50  0001 C CNN
-F 3 "http://www.ti.com/lit/gpn/sn74LS257" H 6050 5900 50  0001 C CNN
-	1    6050 5900
-	1    0    0    -1
-$EndComp
-$Comp
-L 74xx:74LS257 U?
-U 1 1 6176DC0B
-P 6050 8100
-F 0 "U?" H 6300 8850 50  0000 C CNN
-F 1 "ME4" H 6050 8100 50  0000 C CNN
-F 2 "" H 6050 8100 50  0001 C CNN
-F 3 "http://www.ti.com/lit/gpn/sn74LS257" H 6050 8100 50  0001 C CNN
-	1    6050 8100
-	1    0    0    -1
 $EndComp
 $Comp
@@
 Wire Wire Line
 	5400 8500 5400 8400
+$Comp
+L CES:74HC257 U?
+U 1 1 6094D17A
+P 6050 1500
+F 0 "U?" H 6250 2300 50  0000 C CNN
+F 1 "ME1" H 6050 1500 50  0000 C CNN
+F 2 "" H 6050 1500 50  0001 C CNN
+F 3 "http://www.ti.com/lit/gpn/sn74HC257" H 6050 1500 50  0001 C CNN
+	1    6050 1500
+	1    0    0    -1
+$EndComp
+$Comp
+L CES:74HC257 U?
+U 1 1 6094DE29
+P 6050 3700
+F 0 "U?" H 6250 4500 50  0000 C CNN
+F 1 "ME2" H 6050 3700 50  0000 C CNN
+F 2 "" H 6050 3700 50  0001 C CNN
+F 3 "http://www.ti.com/lit/gpn/sn74HC257" H 6050 3700 50  0001 C CNN
+	1    6050 3700
+	1    0    0    -1
+$EndComp
+$Comp
+L CES:74HC257 U?
+U 1 1 6094E47A
+P 6050 5900
+F 0 "U?" H 6250 6700 50  0000 C CNN
+F 1 "ME3" H 6050 5900 50  0000 C CNN
+F 2 "" H 6050 5900 50  0001 C CNN
+F 3 "http://www.ti.com/lit/gpn/sn74HC257" H 6050 5900 50  0001 C CNN
+	1    6050 5900
+	1    0    0    -1
+$EndComp
+$Comp
+L CES:74HC257 U?
+U 1 1 6094ED6B
+P 6050 8100
+F 0 "U?" H 6250 8900 50  0000 C CNN
+F 1 "ME4" H 6050 8100 50  0000 C CNN
+F 2 "" H 6050 8100 50  0001 C CNN
+F 3 "http://www.ti.com/lit/gpn/sn74HC257" H 6050 8100 50  0001 C CNN
+	1    6050 8100
+	1    0    0    -1
+$EndComp
+$Comp
+L CES:74HC283 U?
+U 1 1 6095472F
+P 3450 1400
+F 0 "U?" H 3650 2050 50  0000 C CNN
+F 1 "SM1" H 3450 1400 50  0000 C CNN
+F 2 "" H 3450 1400 50  0001 C CNN
+F 3 "http://www.ti.com/lit/gpn/cd74HC283" H 3450 1400 50  0001 C CNN
+	1    3450 1400
+	1    0    0    -1
+$EndComp
+$Comp
+L CES:74HC283 U?
+U 1 1 609558CF
+P 3450 3300
+F 0 "U?" H 3650 3950 50  0000 C CNN
+F 1 "SM2" H 3450 3300 50  0000 C CNN
+F 2 "" H 3450 3300 50  0001 C CNN
+F 3 "http://www.ti.com/lit/gpn/cd74HC283" H 3450 3300 50  0001 C CNN
+	1    3450 3300
+	1    0    0    -1
+$EndComp
+$Comp
+L CES:74HC283 U?
+U 1 1 6095611B
+P 3450 5200
+F 0 "U?" H 3650 5850 50  0000 C CNN
+F 1 "SM3" H 3450 5200 50  0000 C CNN
+F 2 "" H 3450 5200 50  0001 C CNN
+F 3 "http://www.ti.com/lit/gpn/cd74HC283" H 3450 5200 50  0001 C CNN
+	1    3450 5200
+	1    0    0    -1
+$EndComp
+$Comp
+L CES:74HC283 U?
+U 1 1 609567A2
+P 3450 7150
+F 0 "U?" H 3650 7800 50  0000 C CNN
+F 1 "SM4" H 3450 7150 50  0000 C CNN
+F 2 "" H 3450 7150 50  0001 C CNN
+F 3 "http://www.ti.com/lit/gpn/cd74HC283" H 3450 7150 50  0001 C CNN
+	1    3450 7150
+	1    0    0    -1
+$EndComp
 $EndSCHEMATC

Commit message: Control Unit
Parts:
- gave numbers to parts that had none: 24
Connections:
- net ZComp: now also U201.12, U201.3, U201.6, U201.9

Commit message: Assigning footprints and generating netlist
Parts:
- C201, C202, C203, C204, C205, C206, C207, C208, C209, C210, C211, C212: footprint (none) -> Capacitor_THT:CP_Radial_D5.0mm_P2.50mm
- U201, U202, U203, U204: footprint (none) -> Package_DIP:DIP-14_W7.62mm
- U205, U206, U207, U208, U209, U210, U211, U212: footprint (none) -> Package_DIP:DIP-16_W7.62mm

Commit message: Correcting footprints errors
Parts:
- C201, C202, C203, C204, C205, C206, C207, C208, C209, C210, C211, C212: footprint Capacitor_THT:CP_Radial_D5.0mm_P2.50mm -> Capacitor_THT:C_Disc_D4.3mm_W1.9mm_P5.00mm
- U201: value CD1 -> 74HC02
- U202: value CD2 -> 74HC02
- U203: value CD3 -> 74HC02
- U204: value CD4 -> 74HC02
- U205: value SM1 -> 74HC283
- U206: value SM2 -> 74HC283
- U207: value SM3 -> 74HC283
- U208: value SM4 -> 74HC283
- U209: value ME1 -> 74HC257
- U210: value ME2 -> 74HC257
- U211: value ME3 -> 74HC257
- U212: value ME4 -> 74HC257

Commit message: Starting PCB design
Connections:
- net SRT0: now also U201.5; no longer U201.2
- net SRT1: now also U201.2; no longer U201.5
- net SRT12: now also U204.5; no longer U204.2
- net SRT13: now also U204.2; no longer U204.5
- net SRT4: now also U202.5; no longer U202.2
- net SRT5: now also U202.2; no longer U202.5
- net SRT8: now also U203.5; no longer U203.2
- net SRT9: now also U203.2; no longer U203.5
- net at U205.2 (B2): now also U201.1; no longer U201.4
- net at U205.6 (B1): now also U201.4; no longer U201.1
- net at U206.2 (B2): now also U202.1; no longer U202.4
- net at U206.6 (B1): now also U202.4; no longer U202.1
- net at U207.2 (B2): now also U203.1; no longer U203.4
- net at U207.6 (B1): now also U203.4; no longer U203.1
- net at U208.2 (B2): now also U204.1; no longer U204.4
- net at U208.6 (B1): now also U204.4; no longer U204.1
Other:
- moved on the sheet: U201A, U201B, U202A, U202B, U203A, U203B, U204A, U204B
Changed lines of the file:
@@
 L 74xx:74HC02 U201
 U 1 1 61744753
+P 1300 1100
+F 0 "U201" H 1450 1250 50  0000 C CNN
+F 1 "74HC02" H 1300 1100 50  0000 C CNN
+F 2 "Package_DIP:DIP-14_W7.62mm" H 1300 1100 50  0001 C CNN
+F 3 "http://www.ti.com/lit/gpn/sn74hc02" H 1300 1100 50  0001 C CNN
+	1    1300 1100
+	1    0    0    -1
+$EndComp
+$Comp
+L 74xx:74HC02 U201
+U 2 1 61746BE6
 P 1300 700
-F 0 "U201" H 1450 850 50  0000 C CNN
+F 0 "U201" H 1300 900 50  0000 C CNN
 F 1 "74HC02" H 1300 700 50  0000 C CNN
 F 2 "Package_DIP:DIP-14_W7.62mm" H 1300 700 50  0001 C CNN
 F 3 "http://www.ti.com/lit/gpn/sn74hc02" H 1300 700 50  0001 C CNN
-	1    1300 700
-	1    0    0    -1
-$EndComp
-$Comp
-L 74xx:74HC02 U201
-U 2 1 61746BE6
-P 1300 1100
-F 0 "U201" H 1300 1300 50  0000 C CNN
-F 1 "74HC02" H 1300 1100 50  0000 C CNN
-F 2 "Package_DIP:DIP-14_W7.62mm" H 1300 1100 50  0001 C CNN
-F 3 "http://www.ti.com/lit/gpn/sn74hc02" H 1300 1100 50  0001 C CNN
-	2    1300 1100
+	2    1300 700
 	1    0    0    -1
 $EndComp
@@
 L 74xx:74HC02 U202
 U 1 1 61758CF1
+P 1300 3000
+F 0 "U202" H 1300 3200 50  0000 C CNN
+F 1 "74HC02" H 1300 3000 50  0000 C CNN
+F 2 "Package_DIP:DIP-14_W7.62mm" H 1300 3000 50  0001 C CNN
+F 3 "http://www.ti.com/lit/gpn/sn74hc02" H 1300 3000 50  0001 C CNN
+	1    1300 3000
+	1    0    0    -1
+$EndComp
+$Comp
+L 74xx:74HC02 U202
+U 2 1 61758CF7
 P 1300 2600
 F 0 "U202" H 1300 2800 50  0000 C CNN
@@
 F 2 "Package_DIP:DIP-14_W7.62mm" H 1300 2600 50  0001 C CNN
 F 3 "http://www.ti.com/lit/gpn/sn74hc02" H 1300 2600 50  0001 C CNN
-	1    1300 2600
-	1    0    0    -1
-$EndComp
-$Comp
-L 74xx:74HC02 U202
-U 2 1 61758CF7
-P 1300 3000
-F 0 "U202" H 1300 3200 50  0000 C CNN
-F 1 "74HC02" H 1300 3000 50  0000 C CNN
-F 2 "Package_DIP:DIP-14_W7.62mm" H 1300 3000 50  0001 C CNN
-F 3 "http://www.ti.com/lit/gpn/sn74hc02" H 1300 3000 50  0001 C CNN
-	2    1300 3000
+	2    1300 2600
 	1    0    0    -1
 $EndComp
@@
 L 74xx:74HC02 U203
 U 1 1 6175D579
+P 1300 4900
+F 0 "U203" H 1300 5100 50  0000 C CNN
+F 1 "74HC02" H 1300 4900 50  0000 C CNN
+F 2 "Package_DIP:DIP-14_W7.62mm" H 1300 4900 50  0001 C CNN
+F 3 "http://www.ti.com/lit/gpn/sn74hc02" H 1300 4900 50  0001 C CNN
+	1    1300 4900
+	1    0    0    -1
+$EndComp
+$Comp
+L 74xx:74HC02 U203
+U 2 1 6175D57F
 P 1300 4500
 F 0 "U203" H 1300 4700 50  0000 C CNN
@@
 F 2 "Package_DIP:DIP-14_W7.62mm" H 1300 4500 50  0001 C CNN
 F 3 "http://www.ti.com/lit/gpn/sn74hc02" H 1300 4500 50  0001 C CNN
-	1    1300 4500
-	1    0    0    -1
-$EndComp
-$Comp
-L 74xx:74HC02 U203
-U 2 1 6175D57F
-P 1300 4900
-F 0 "U203" H 1300 5100 50  0000 C CNN
-F 1 "74HC02" H 1300 4900 50  0000 C CNN
-F 2 "Package_DIP:DIP-14_W7.62mm" H 1300 4900 50  0001 C CNN
-F 3 "http://www.ti.com/lit/gpn/sn74hc02" H 1300 4900 50  0001 C CNN
-	2    1300 4900
+	2    1300 4500
 	1    0    0    -1
 $EndComp
@@
 L 74xx:74HC02 U204
 U 2 1 617636E6
+P 1300 6450
+F 0 "U204" H 1300 6650 50  0000 C CNN
+F 1 "74HC02" H 1300 6450 50  0000 C CNN
+F 2 "Package_DIP:DIP-14_W7.62mm" H 1300 6450 50  0001 C CNN
+F 3 "http://www.ti.com/lit/gpn/sn74hc02" H 1300 6450 50  0001 C CNN
+	2    1300 6450
+	1    0    0    -1
+$EndComp
+$Comp
+L 74xx:74HC02 U204
+U 1 1 617636E0
 P 1300 6850
 F 0 "U204" H 1300 7050 50  0000 C CNN
@@
 F 2 "Package_DIP:DIP-14_W7.62mm" H 1300 6850 50  0001 C CNN
 F 3 "http://www.ti.com/lit/gpn/sn74hc02" H 1300 6850 50  0001 C CNN
-	2    1300 6850
-	1    0    0    -1
-$EndComp
-$Comp
-L 74xx:74HC02 U204
-U 1 1 617636E0
-P 1300 6450
-F 0 "U204" H 1300 6650 50  0000 C CNN
-F 1 "74HC02" H 1300 6450 50  0000 C CNN
-F 2 "Package_DIP:DIP-14_W7.62mm" H 1300 6450 50  0001 C CNN
-F 3 "http://www.ti.com/lit/gpn/sn74hc02" H 1300 6450 50  0001 C CNN
-	1    1300 6450
-	1    0    0    -1
-$EndComp
+	1    1300 6850
+	1    0    0    -1
+$EndComp
