File: CES/AddressRegister.sch (KiCad schematic (older format))
At the start: 4 parts

Commit message: Registers
Parts:
- added C? (x4): 100nF, symbol Device:C
Connections:
- net ~SaiRE: now reaches U?.1 (Oe1)
- net ~SaiRE: now also U?.1 (Oe1), U?.1 (Oe1), U?.1 (Oe1)
- net GND: now reaches U?.10 (E2)
- net GND: now also U?.10 (E2), U?.10 (E2), U?.10 (E2), U?.11 (D3), U?.12 (D2), U?.15 (Mr), U?.15 (Mr), U?.15 (Mr), U?.15 (Mr), U?.2 (Oe2), U?.2 (Oe2), U?.2 (Oe2), U?.2 (Oe2), U?.8 (GND), U?.8 (GND), U?.8 (GND), U?.8 (GND), U?.9 (E1), U?.9 (E1), U?.9 (E1), U?.9 (E1), C?.2, C?.2, C?.2, C?.2
- net SME3: now reaches U?.11 (D3)
- net SME2: now reaches U?.12 (D2)
- net SME1: now reaches U?.13 (D1)
- net SME0: now reaches U?.14 (D0)
- net VCC: now reaches U?.16 (VCC)
- net VCC: now also U?.16 (VCC), U?.16 (VCC), U?.16 (VCC), C?.1, C?.1, C?.1, C?.1
- net VEB0: now reaches U?.3 (Q0)
- net VEB1: now reaches U?.4 (Q1)
- net VEB2: now reaches U?.5 (Q2)
- net VEB3: now reaches U?.6 (Q3)
- net Rlg2: now reaches U?.7 (Cp)
- net Rlg2: now also U?.7 (Cp), U?.7 (Cp), U?.7 (Cp)
- net SME7: now reaches U?.11 (D3)
- net SME6: now reaches U?.12 (D2)
- net SME5: now reaches U?.13 (D1)
- net SME4: now reaches U?.14 (D0)
- net VEB4: now reaches U?.3 (Q0)
- net VEB5: now reaches U?.4 (Q1)
- net VEB6: now reaches U?.5 (Q2)
- net VEB7: now reaches U?.6 (Q3)
- net SME11: now reaches U?.11 (D3)
- net SME10: now reaches U?.12 (D2)
- net SME9: now reaches U?.13 (D1)
- net SME8: now reaches U?.14 (D0)
- net VEB8: now reaches U?.3 (Q0)
- net VEB9: now reaches U?.4 (Q1)
- net VEB10: now reaches U?.5 (Q2)
- net VEB11: now reaches U?.6 (Q3)
- net SME13: now reaches U?.13 (D1)
- net SME12: now reaches U?.14 (D0)
- net VEB12: now reaches U?.3 (Q0)
- net VEB13: now reaches U?.4 (Q1)
- no-connect marks 0 -> 2
Other:
- moved on the sheet: U?
