File: CES/CES.sch (KiCad schematic (older format))
At the start: 1 part, among them J101 Barrel_Jack

Commit message: Registers
Parts:
- added C?: 100uF, symbol Device:CP1
- added C?: 10uF, symbol Device:CP1
- added C?: 1000nF, symbol Device:C
Connections:
- net GND: now also C?.2, C?.2, C?.2
- net VCC: now also C?.1, C?.1, C?.1
Changed lines of the file:
@@
 $Descr A4 11693 8268
 encoding utf-8
-Sheet 1 11
+Sheet 1 13
 Title ""
 Date ""
@@
 	8600 1900 9000 1900
 Wire Wire Line
-	9450 1900 9450 1750
+	9450 1900 9450 1800
 $Comp
 L power:GND #PWR0102
@@
 	8600 2100 9000 2100
 Wire Wire Line
-	9450 2100 9450 2300
+	9450 2100 9450 2200
 $Comp
 L power:PWR_FLAG #FLG0101
@@
 EndData
 $EndBitmap
+$Comp
+L Device:CP1 C?
+U 1 1 60A155E7
+P 9800 2000
+F 0 "C?" H 9915 2046 50  0000 L CNN
+F 1 "100uF" H 9915 1955 50  0000 L CNN
+F 2 "" H 9800 2000 50  0001 C CNN
+F 3 "~" H 9800 2000 50  0001 C CNN
+	1    9800 2000
+	1    0    0    -1
+$EndComp
+$Comp
+L Device:CP1 C?
+U 1 1 60A157F1
+P 10350 2000
+F 0 "C?" H 10465 2046 50  0000 L CNN
+F 1 "10uF" H 10465 1955 50  0000 L CNN
+F 2 "" H 10350 2000 50  0001 C CNN
+F 3 "~" H 10350 2000 50  0001 C CNN
+	1    10350 2000
+	1    0    0    -1
+$EndComp
+Wire Wire Line
+	9450 2200 9800 2200
+Wire Wire Line
+	9800 2200 9800 2150
+Connection ~ 9450 2200
+Wire Wire Line
+	9450 2200 9450 2300
+Wire Wire Line
+	9800 2200 10350 2200
+Wire Wire Line
+	10350 2200 10350 2150
+Connection ~ 9800 2200
+Wire Wire Line
+	10350 1850 10350 1800
+Wire Wire Line
+	10350 1800 9800 1800
+Wire Wire Line
+	9800 1800 9800 1850
+Wire Wire Line
+	9800 1800 9450 1800
+Connection ~ 9800 1800
+Connection ~ 9450 1800
+Wire Wire Line
+	9450 1800 9450 1750
+$Comp
+L Device:C C?
+U 1 1 60A17721
+P 10750 2000
+F 0 "C?" H 10865 2046 50  0000 L CNN
+F 1 "1000nF" H 10865 1955 50  0000 L CNN
+F 2 "" H 10788 1850 50  0001 C CNN
+F 3 "~" H 10750 2000 50  0001 C CNN
+	1    10750 2000
+	1    0    0    -1
+$EndComp
+Wire Wire Line
+	10350 1800 10750 1800
+Wire Wire Line
+	10750 1800 10750 1850
+Connection ~ 10350 1800
+Wire Wire Line
+	10350 2200 10750 2200
+Wire Wire Line
+	10750 2200 10750 2150
+Connection ~ 10350 2200
 $EndSCHEMATC
