File: CES/DataRegister.sch (KiCad schematic (older format))
At the start: 4 parts

Commit message: Registers
Parts:
- added C? (x4): 100nF, symbol Device:C
Connections:
- net ~UltC: now reaches U?.1 (Oe1)
- net ~UltC: now also U?.1 (Oe1), U?.1 (Oe1), U?.1 (Oe1)
- net GND: now reaches U?.10 (E2)
- net GND: now also U?.10 (E2), U?.10 (E2), U?.10 (E2), U?.15 (Mr), U?.15 (Mr), U?.15 (Mr), U?.15 (Mr), U?.2 (Oe2), U?.2 (Oe2), U?.2 (Oe2), U?.2 (Oe2), U?.8 (GND), U?.8 (GND), U?.8 (GND), U?.8 (GND), U?.9 (E1), U?.9 (E1), U?.9 (E1), U?.9 (E1), C?.2, C?.2, C?.2, C?.2
- net VDB3: now reaches U?.11 (D3)
- net VDB2: now reaches U?.12 (D2)
- net VDB1: now reaches U?.13 (D1)
- net VDB0: now reaches U?.14 (D0)
- net VCC: now reaches U?.16 (VCC)
- net VCC: now also U?.16 (VCC), U?.16 (VCC), U?.16 (VCC), C?.1, C?.1, C?.1, C?.1
- net ESA0: now reaches U?.3 (Q0)
- net ESA1: now reaches U?.4 (Q1)
- net ESA2: now reaches U?.5 (Q2)
- net ESA3: now reaches U?.6 (Q3)
- net Rlg2: now reaches U?.7 (Cp)
- net Rlg2: now also U?.7 (Cp), U?.7 (Cp), U?.7 (Cp)
- net VDB7: now reaches U?.11 (D3)
- net VDB6: now reaches U?.12 (D2)
- net VDB5: now reaches U?.13 (D1)
- net VDB4: now reaches U?.14 (D0)
- net ESA4: now reaches U?.3 (Q0)
- net ESA5: now reaches U?.4 (Q1)
- net ESA6: now reaches U?.5 (Q2)
- net ESA7: now reaches U?.6 (Q3)
- net VDB11: now reaches U?.11 (D3)
- net VDB10: now reaches U?.12 (D2)
- net VDB9: now reaches U?.13 (D1)
- net VDB8: now reaches U?.14 (D0)
- net ESA8: now reaches U?.3 (Q0)
- net ESA9: now reaches U?.4 (Q1)
- net ESA10: now reaches U?.5 (Q2)
- net ESA11: now reaches U?.6 (Q3)
- net VDB15: now reaches U?.11 (D3)
- net VDB14: now reaches U?.12 (D2)
- net VDB13: now reaches U?.13 (D1)
- net VDB12: now reaches U?.14 (D0)
- net ESA12: now reaches U?.3 (Q0)
- net ESA13: now reaches U?.4 (Q1)
- net ESA14: now reaches U?.5 (Q2)
- net ESA15: now reaches U?.6 (Q3)
Other:
- moved on the sheet: U?
