File: CES/ProgramPointerRegister.sch (KiCad schematic (older format))
At the start: 4 parts

Commit message: Registers
Parts:
- added C? (x4): 100nF, symbol Device:C
Connections:
- net ~SaiRP: now reaches U?.1 (Oe1)
- net ~SaiRP: now also U?.1 (Oe1), U?.1 (Oe1), U?.1 (Oe1)
- net GND: now reaches U?.10 (E2)
- net GND: now also U?.10 (E2), U?.10 (E2), U?.10 (E2), U?.15 (Mr), U?.15 (Mr), U?.15 (Mr), U?.15 (Mr), U?.2 (Oe2), U?.2 (Oe2), U?.2 (Oe2), U?.2 (Oe2), U?.8 (GND), U?.8 (GND), U?.8 (GND), U?.8 (GND), C?.2, C?.2, C?.2, C?.2
- net SS3: now reaches U?.11 (D3)
- net SS2: now reaches U?.12 (D2)
- net SS1: now reaches U?.13 (D1)
- net SS0: now reaches U?.14 (D0)
- net VCC: now reaches U?.16 (VCC)
- net VCC: now also U?.16 (VCC), U?.16 (VCC), U?.16 (VCC), C?.1, C?.1, C?.1, C?.1
- net ESA0: now reaches U?.3 (Q0)
- net ESA1: now reaches U?.4 (Q1)
- net ESA2: now reaches U?.5 (Q2)
- net ESA3: now reaches U?.6 (Q3)
- net Rlg1: now reaches U?.7 (Cp)
- net Rlg1: now also U?.7 (Cp), U?.7 (Cp), U?.7 (Cp)
- net ~EscP: now reaches U?.9 (E1)
- net ~EscP: now also U?.9 (E1), U?.9 (E1), U?.9 (E1)
- net SS7: now reaches U?.11 (D3)
- net SS6: now reaches U?.12 (D2)
- net SS5: now reaches U?.13 (D1)
- net SS4: now reaches U?.14 (D0)
- net ESA4: now reaches U?.3 (Q0)
- net ESA5: now reaches U?.4 (Q1)
- net ESA6: now reaches U?.5 (Q2)
- net ESA7: now reaches U?.6 (Q3)
- net SS11: now reaches U?.11 (D3)
- net SS10: now reaches U?.12 (D2)
- net SS9: now reaches U?.13 (D1)
- net SS8: now reaches U?.14 (D0)
- net ESA8: now reaches U?.3 (Q0)
- net ESA9: now reaches U?.4 (Q1)
- net ESA10: now reaches U?.5 (Q2)
- net ESA11: now reaches U?.6 (Q3)
- net SS15: now reaches U?.11 (D3)
- net SS14: now reaches U?.12 (D2)
- net SS13: now reaches U?.13 (D1)
- net SS12: now reaches U?.14 (D0)
- net ESA12: now reaches U?.3 (Q0)
- net ESA13: now reaches U?.4 (Q1)
- net ESA14: now reaches U?.5 (Q2)
- net ESA15: now reaches U?.6 (Q3)
Other:
- moved on the sheet: U?
