File: CES/ProgramPointerRegister.sch (KiCad schematic (older format))
At the start: 8 parts

Commit message: Adding 74HC versions of 74LS chips
Parts:
- removed U?: RP1, symbol 74xx:74LS173
- removed U?: RP2, symbol 74xx:74LS173
- removed U?: RP3, symbol 74xx:74LS173
- removed U?: RP4, symbol 74xx:74LS173
- added U?: RP1, symbol CES:74HC173
- added U?: RP2, symbol CES:74HC173
- added U?: RP3, symbol CES:74HC173
- added U?: RP4, symbol CES:74HC173
Changed lines of the file:
@@
 $EndDescr
-$Comp
-L 74xx:74LS173 U?
-U 1 1 61BF1A2D
-P 4050 1700
-F 0 "U?" H 4300 2450 50  0000 C CNN
-F 1 "RP1" H 4050 1700 50  0000 C CNN
-F 2 "" H 4050 1700 50  0001 C CNN
-F 3 "http://www.ti.com/lit/gpn/sn74LS173" H 4050 1700 50  0001 C CNN
-	1    4050 1700
-	1    0    0    -1
-$EndComp
-$Comp
-L 74xx:74LS173 U?
-U 1 1 61BF1A33
-P 4050 4050
-F 0 "U?" H 4300 4800 50  0000 C CNN
-F 1 "RP2" H 4050 4050 50  0000 C CNN
-F 2 "" H 4050 4050 50  0001 C CNN
-F 3 "http://www.ti.com/lit/gpn/sn74LS173" H 4050 4050 50  0001 C CNN
-	1    4050 4050
-	1    0    0    -1
-$EndComp
-$Comp
-L 74xx:74LS173 U?
-U 1 1 61BF1A39
-P 4050 6400
-F 0 "U?" H 4300 7150 50  0000 C CNN
-F 1 "RP3" H 4050 6400 50  0000 C CNN
-F 2 "" H 4050 6400 50  0001 C CNN
-F 3 "http://www.ti.com/lit/gpn/sn74LS173" H 4050 6400 50  0001 C CNN
-	1    4050 6400
-	1    0    0    -1
-$EndComp
-$Comp
-L 74xx:74LS173 U?
-U 1 1 61BF1A3F
-P 4050 8750
-F 0 "U?" H 4300 9550 50  0000 C CNN
-F 1 "RP4" H 4050 8750 50  0000 C CNN
-F 2 "" H 4050 8750 50  0001 C CNN
-F 3 "http://www.ti.com/lit/gpn/sn74LS173" H 4050 8750 50  0001 C CNN
-	1    4050 8750
-	1    0    0    -1
-$EndComp
 $Comp
 L power:VCC #PWR?
@@
 Wire Wire Line
 	1500 10250 1350 10250
+$Comp
+L CES:74HC173 U?
+U 1 1 60920B36
+P 4050 1700
+F 0 "U?" H 4300 2450 50  0000 C CNN
+F 1 "RP1" H 4050 1700 50  0000 C CNN
+F 2 "" H 4050 1700 50  0001 C CNN
+F 3 "http://www.ti.com/lit/gpn/cd74HC173" H 4050 1700 50  0001 C CNN
+	1    4050 1700
+	1    0    0    -1
+$EndComp
+$Comp
+L CES:74HC173 U?
+U 1 1 60921962
+P 4050 4050
+F 0 "U?" H 4300 4800 50  0000 C CNN
+F 1 "RP2" H 4050 4050 50  0000 C CNN
+F 2 "" H 4050 4050 50  0001 C CNN
+F 3 "http://www.ti.com/lit/gpn/cd74HC173" H 4050 4050 50  0001 C CNN
+	1    4050 4050
+	1    0    0    -1
+$EndComp
+$Comp
+L CES:74HC173 U?
+U 1 1 6092228C
+P 4050 6400
+F 0 "U?" H 4300 7150 50  0000 C CNN
+F 1 "RP3" H 4050 6400 50  0000 C CNN
+F 2 "" H 4050 6400 50  0001 C CNN
+F 3 "http://www.ti.com/lit/gpn/cd74HC173" H 4050 6400 50  0001 C CNN
+	1    4050 6400
+	1    0    0    -1
+$EndComp
+$Comp
+L CES:74HC173 U?
+U 1 1 60922BFF
+P 4050 8750
+F 0 "U?" H 4300 9500 50  0000 C CNN
+F 1 "RP4" H 4050 8750 50  0000 C CNN
+F 2 "" H 4050 8750 50  0001 C CNN
+F 3 "http://www.ti.com/lit/gpn/cd74HC173" H 4050 8750 50  0001 C CNN
+	1    4050 8750
+	1    0    0    -1
+$EndComp
 $EndSCHEMATC

Commit message: Control Unit
Parts:
- gave numbers to parts that had none: 8
Changed lines of the file:
@@
 $Descr A4 8268 11693 portrait
 encoding utf-8
-Sheet 5 16
+Sheet 5 17
 Title "CES"
 Date "2021-04-24"
@@
 $EndDescr
 $Comp
-L power:VCC #PWR?
+L power:VCC #PWR0507
 U 1 1 609BE1F2
 P 4050 800
-F 0 "#PWR?" H 4050 650 50  0001 C CNN
+F 0 "#PWR0507" H 4050 650 50  0001 C CNN
 F 1 "VCC" H 4065 973 50  0000 C CNN
 F 2 "" H 4050 800 50  0001 C CNN
@@
 $EndComp
 $Comp
-L power:GND #PWR?
+L power:GND #PWR0508
 U 1 1 609BEB3B
 P 4050 2600
-F 0 "#PWR?" H 4050 2350 50  0001 C CNN
+F 0 "#PWR0508" H 4050 2350 50  0001 C CNN
 F 1 "GND" H 4055 2427 50  0000 C CNN
 F 2 "" H 4050 2600 50  0001 C CNN
@@
 $EndComp
 $Comp
-L power:VCC #PWR?
+L power:VCC #PWR0509
 U 1 1 609BF0A7
 P 4050 3150
-F 0 "#PWR?" H 4050 3000 50  0001 C CNN
+F 0 "#PWR0509" H 4050 3000 50  0001 C CNN
 F 1 "VCC" H 4065 3323 50  0000 C CNN
 F 2 "" H 4050 3150 50  0001 C CNN
@@
 $EndComp
 $Comp
-L power:GND #PWR?
+L power:GND #PWR0510
 U 1 1 609C0430
 P 4050 4950
-F 0 "#PWR?" H 4050 4700 50  0001 C CNN
+F 0 "#PWR0510" H 4050 4700 50  0001 C CNN
 F 1 "GND" H 4055 4777 50  0000 C CNN
 F 2 "" H 4050 4950 50  0001 C CNN
@@
 $EndComp
 $Comp
-L power:VCC #PWR?
+L power:VCC #PWR0511
 U 1 1 609C13FE
 P 4050 5500
-F 0 "#PWR?" H 4050 5350 50  0001 C CNN
+F 0 "#PWR0511" H 4050 5350 50  0001 C CNN
 F 1 "VCC" H 4065 5673 50  0000 C CNN
 F 2 "" H 4050 5500 50  0001 C CNN
@@
 $EndComp
 $Comp
-L power:VCC #PWR?
+L power:VCC #PWR0513
 U 1 1 609C28D0
 P 4050 7850
-F 0 "#PWR?" H 4050 7700 50  0001 C CNN
+F 0 "#PWR0513" H 4050 7700 50  0001 C CNN
 F 1 "VCC" H 4065 8023 50  0000 C CNN
 F 2 "" H 4050 7850 50  0001 C CNN
@@
 $EndComp
 $Comp
-L power:GND #PWR?
+L power:GND #PWR0512
 U 1 1 609C2FAA
 P 4050 7300
-F 0 "#PWR?" H 4050 7050 50  0001 C CNN
+F 0 "#PWR0512" H 4050 7050 50  0001 C CNN
 F 1 "GND" H 4055 7127 50  0000 C CNN
 F 2 "" H 4050 7300 50  0001 C CNN
@@
 $EndComp
 $Comp
-L power:GND #PWR?
+L power:GND #PWR0514
 U 1 1 609C3E2C
 P 4050 9650
-F 0 "#PWR?" H 4050 9400 50  0001 C CNN
+F 0 "#PWR0514" H 4050 9400 50  0001 C CNN
 F 1 "GND" H 4055 9477 50  0000 C CNN
 F 2 "" H 4050 9650 50  0001 C CNN
@@
 Connection ~ 3200 2000
 $Comp
-L power:GND #PWR?
+L power:GND #PWR0503
 U 1 1 609C59EF
 P 3200 2400
-F 0 "#PWR?" H 3200 2150 50  0001 C CNN
+F 0 "#PWR0503" H 3200 2150 50  0001 C CNN
 F 1 "GND" H 3205 2227 50  0000 C CNN
 F 2 "" H 3200 2400 50  0001 C CNN
@@
 Connection ~ 3200 4350
 $Comp
-L power:GND #PWR?
+L power:GND #PWR0504
 U 1 1 609C66DC
 P 3200 4750
-F 0 "#PWR?" H 3200 4500 50  0001 C CNN
+F 0 "#PWR0504" H 3200 4500 50  0001 C CNN
 F 1 "GND" H 3205 4577 50  0000 C CNN
 F 2 "" H 3200 4750 50  0001 C CNN
@@
 Connection ~ 3200 6700
 $Comp
-L power:GND #PWR?
+L power:GND #PWR0505
 U 1 1 609C6E61
 P 3200 7100
-F 0 "#PWR?" H 3200 6850 50  0001 C CNN
+F 0 "#PWR0505" H 3200 6850 50  0001 C CNN
 F 1 "GND" H 3205 6927 50  0000 C CNN
 F 2 "" H 3200 7100 50  0001 C CNN
@@
 Connection ~ 3200 9050
 $Comp
-L power:GND #PWR?
+L power:GND #PWR0506
 U 1 1 609C7550
 P 3200 9450
-F 0 "#PWR?" H 3200 9200 50  0001 C CNN
+F 0 "#PWR0506" H 3200 9200 50  0001 C CNN
 F 1 "GND" H 3205 9277 50  0000 C CNN
 F 2 "" H 3200 9450 50  0001 C CNN
@@
 ESA15
 $Comp
-L Device:C C?
+L Device:C C501
 U 1 1 609DA351
 P 1050 10500
-F 0 "C?" H 1100 10600 50  0000 L CNN
+F 0 "C501" H 1100 10600 50  0000 L CNN
 F 1 "100nF" H 1100 10400 50  0000 L CNN
 F 2 "" H 1088 10350 50  0001 C CNN
@@
 $EndComp
 $Comp
-L Device:C C?
+L Device:C C502
 U 1 1 609DA8A0
 P 1350 10500
-F 0 "C?" H 1400 10600 50  0000 L CNN
+F 0 "C502" H 1400 10600 50  0000 L CNN
 F 1 "100nF" H 1400 10400 50  0000 L CNN
 F 2 "" H 1388 10350 50  0001 C CNN
@@
 $EndComp
 $Comp
-L Device:C C?
+L Device:C C503
 U 1 1 609DACD4
 P 1650 10500
-F 0 "C?" H 1700 10600 50  0000 L CNN
+F 0 "C503" H 1700 10600 50  0000 L CNN
 F 1 "100nF" H 1700 10400 50  0000 L CNN
 F 2 "" H 1688 10350 50  0001 C CNN
@@
 $EndComp
 $Comp
-L Device:C C?
+L Device:C C504
 U 1 1 609DB26A
 P 1950 10500
-F 0 "C?" H 2000 10600 50  0000 L CNN
+F 0 "C504" H 2000 10600 50  0000 L CNN
 F 1 "100nF" H 2000 10400 50  0000 L CNN
 F 2 "" H 1988 10350 50  0001 C CNN
@@
 	1350 10750 1500 10750
 $Comp
-L power:GND #PWR?
+L power:GND #PWR0502
 U 1 1 609E816A
 P 1500 10750
-F 0 "#PWR?" H 1500 10500 50  0001 C CNN
+F 0 "#PWR0502" H 1500 10500 50  0001 C CNN
 F 1 "GND" H 1505 10577 50  0000 C CNN
 F 2 "" H 1500 10750 50  0001 C CNN
@@
 	1500 10750 1650 10750
 $Comp
-L power:VCC #PWR?
+L power:VCC #PWR0501
 U 1 1 609E872B
 P 1500 10250
-F 0 "#PWR?" H 1500 10100 50  0001 C CNN
+F 0 "#PWR0501" H 1500 10100 50  0001 C CNN
 F 1 "VCC" H 1515 10423 50  0000 C CNN
 F 2 "" H 1500 10250 50  0001 C CNN
@@
 	1500 10250 1350 10250
 $Comp
-L CES:74HC173 U?
+L CES:74HC173 U501
 U 1 1 60920B36
 P 4050 1700
-F 0 "U?" H 4300 2450 50  0000 C CNN
+F 0 "U501" H 4300 2450 50  0000 C CNN
 F 1 "RP1" H 4050 1700 50  0000 C CNN
 F 2 "" H 4050 1700 50  0001 C CNN
@@
 $EndComp
 $Comp
-L CES:74HC173 U?
+L CES:74HC173 U502
 U 1 1 60921962
 P 4050 4050
-F 0 "U?" H 4300 4800 50  0000 C CNN
+F 0 "U502" H 4300 4800 50  0000 C CNN
 F 1 "RP2" H 4050 4050 50  0000 C CNN
 F 2 "" H 4050 4050 50  0001 C CNN
@@
 $EndComp
 $Comp
-L CES:74HC173 U?
+L CES:74HC173 U503
 U 1 1 6092228C
 P 4050 6400
-F 0 "U?" H 4300 7150 50  0000 C CNN
+F 0 "U503" H 4300 7150 50  0000 C CNN
 F 1 "RP3" H 4050 6400 50  0000 C CNN
 F 2 "" H 4050 6400 50  0001 C CNN
@@
 $EndComp
 $Comp
-L CES:74HC173 U?
+L CES:74HC173 U504
 U 1 1 60922BFF
 P 4050 8750
-F 0 "U?" H 4300 9500 50  0000 C CNN
+F 0 "U504" H 4300 9500 50  0000 C CNN
 F 1 "RP4" H 4050 8750 50  0000 C CNN
 F 2 "" H 4050 8750 50  0001 C CNN

Commit message: Assigning footprints and generating netlist
Parts:
- C501, C502, C503, C504: footprint (none) -> Capacitor_THT:CP_Radial_D5.0mm_P2.50mm
- U501, U502, U503, U504: footprint (none) -> Package_DIP:DIP-16_W7.62mm
Changed lines of the file:
@@
 F 0 "C501" H 1100 10600 50  0000 L CNN
 F 1 "100nF" H 1100 10400 50  0000 L CNN
-F 2 "" H 1088 10350 50  0001 C CNN
+F 2 "Capacitor_THT:CP_Radial_D5.0mm_P2.50mm" H 1088 10350 50  0001 C CNN
 F 3 "~" H 1050 10500 50  0001 C CNN
 	1    1050 10500
@@
 F 0 "C502" H 1400 10600 50  0000 L CNN
 F 1 "100nF" H 1400 10400 50  0000 L CNN
-F 2 "" H 1388 10350 50  0001 C CNN
+F 2 "Capacitor_THT:CP_Radial_D5.0mm_P2.50mm" H 1388 10350 50  0001 C CNN
 F 3 "~" H 1350 10500 50  0001 C CNN
 	1    1350 10500
@@
 F 0 "C503" H 1700 10600 50  0000 L CNN
 F 1 "100nF" H 1700 10400 50  0000 L CNN
-F 2 "" H 1688 10350 50  0001 C CNN
+F 2 "Capacitor_THT:CP_Radial_D5.0mm_P2.50mm" H 1688 10350 50  0001 C CNN
 F 3 "~" H 1650 10500 50  0001 C CNN
 	1    1650 10500
@@
 F 0 "C504" H 2000 10600 50  0000 L CNN
 F 1 "100nF" H 2000 10400 50  0000 L CNN
-F 2 "" H 1988 10350 50  0001 C CNN
+F 2 "Capacitor_THT:CP_Radial_D5.0mm_P2.50mm" H 1988 10350 50  0001 C CNN
 F 3 "~" H 1950 10500 50  0001 C CNN
 	1    1950 10500
@@
 F 0 "U501" H 4300 2450 50  0000 C CNN
 F 1 "RP1" H 4050 1700 50  0000 C CNN
-F 2 "" H 4050 1700 50  0001 C CNN
+F 2 "Package_DIP:DIP-16_W7.62mm" H 4050 1700 50  0001 C CNN
 F 3 "http://www.ti.com/lit/gpn/cd74HC173" H 4050 1700 50  0001 C CNN
 	1    4050 1700
@@
 F 0 "U502" H 4300 4800 50  0000 C CNN
 F 1 "RP2" H 4050 4050 50  0000 C CNN
-F 2 "" H 4050 4050 50  0001 C CNN
+F 2 "Package_DIP:DIP-16_W7.62mm" H 4050 4050 50  0001 C CNN
 F 3 "http://www.ti.com/lit/gpn/cd74HC173" H 4050 4050 50  0001 C CNN
 	1    4050 4050
@@
 F 0 "U503" H 4300 7150 50  0000 C CNN
 F 1 "RP3" H 4050 6400 50  0000 C CNN
-F 2 "" H 4050 6400 50  0001 C CNN
+F 2 "Package_DIP:DIP-16_W7.62mm" H 4050 6400 50  0001 C CNN
 F 3 "http://www.ti.com/lit/gpn/cd74HC173" H 4050 6400 50  0001 C CNN
 	1    4050 6400
@@
 F 0 "U504" H 4300 9500 50  0000 C CNN
 F 1 "RP4" H 4050 8750 50  0000 C CNN
-F 2 "" H 4050 8750 50  0001 C CNN
+F 2 "Package_DIP:DIP-16_W7.62mm" H 4050 8750 50  0001 C CNN
 F 3 "http://www.ti.com/lit/gpn/cd74HC173" H 4050 8750 50  0001 C CNN
 	1    4050 8750
