File: CES/WorkRegister.sch (KiCad schematic (older format))
At the start: 6 parts

Commit message: Registers
Parts:
- added C? (x6): 100nF, symbol Device:C
Connections:
- net GND: now reaches U?.1 (Oe1)
- net GND: now also U?.1 (Oe1), U?.1 (Oe1), U?.1 (Oe1), U?.10 (E2), U?.10 (E2), U?.10 (E2), U?.10 (E2), U?.10 (GND), U?.10 (GND), U?.15 (Mr), U?.15 (Mr), U?.15 (Mr), U?.15 (Mr), U?.2 (Oe2), U?.2 (Oe2), U?.2 (Oe2), U?.2 (Oe2), U?.8 (GND), U?.8 (GND), U?.8 (GND), U?.8 (GND), C?.2, C?.2, C?.2, C?.2, C?.2, C?.2
- net SS3: now reaches U?.11 (D3)
- net SS2: now reaches U?.12 (D2)
- net SS1: now reaches U?.13 (D1)
- net SS0: now reaches U?.14 (D0)
- net VCC: now reaches U?.16 (VCC)
- net VCC: now also U?.16 (VCC), U?.16 (VCC), U?.16 (VCC), U?.20 (VCC), U?.20 (VCC), C?.1, C?.1, C?.1, C?.1, C?.1, C?.1
- net SRT0: now reaches U?.3 (Q0)
- net SRT0: now also U?.2 (1A0)
- net SRT1: now reaches U?.4 (Q1)
- net SRT1: now also U?.4 (1A1)
- net SRT2: now reaches U?.5 (Q2)
- net SRT2: now also U?.6 (1A2)
- net SRT3: now reaches U?.6 (Q3)
- net SRT3: now also U?.8 (1A3)
- net Rlg1: now reaches U?.7 (Cp)
- net Rlg1: now also U?.7 (Cp), U?.7 (Cp), U?.7 (Cp)
- net ~EscT: now reaches U?.9 (E1)
- net ~EscT: now also U?.9 (E1), U?.9 (E1), U?.9 (E1)
- net SS7: now reaches U?.11 (D3)
- net SS6: now reaches U?.12 (D2)
- net SS5: now reaches U?.13 (D1)
- net SS4: now reaches U?.14 (D0)
- net SRT4: now reaches U?.3 (Q0)
- net SRT4: now also U?.17 (2A0)
- net SRT5: now reaches U?.4 (Q1)
- net SRT5: now also U?.13 (2A2), U?.15 (2A1), U?.5 (Q2)
- net SRT7: now reaches U?.6 (Q3)
- net SRT7: now also U?.11 (2A3)
- net SS11: now reaches U?.11 (D3)
- net SS10: now reaches U?.12 (D2)
- net SS9: now reaches U?.13 (D1)
- net SS8: now reaches U?.14 (D0)
- net SRT8: now reaches U?.3 (Q0)
- net SRT8: now also U?.2 (1A0)
- net SRT9: now reaches U?.4 (Q1)
- net SRT9: now also U?.4 (1A1)
- net SRT10: now reaches U?.5 (Q2)
- net SRT10: now also U?.6 (1A2)
- net SRT11: now reaches U?.6 (Q3)
- net SRT11: now also U?.8 (1A3)
- net SS15: now reaches U?.11 (D3)
- net SS14: now reaches U?.12 (D2)
- net SS13: now reaches U?.13 (D1)
- net SS12: now reaches U?.14 (D0)
- net SRT12: now reaches U?.3 (Q0)
- net SRT12: now also U?.17 (2A0)
- net SRT13: now reaches U?.4 (Q1)
- net SRT13: now also U?.15 (2A1)
- net SRT14: now reaches U?.5 (Q2)
- net SRT14: now also U?.13 (2A2)
- net SRT15: now reaches U?.6 (Q3)
- net SRT15: now also U?.11 (2A3)
- net ~EscM: now reaches U?.1 (1OE)
- net ~EscM: now also U?.1 (1OE), U?.19 (2OE), U?.19 (2OE)
- net VDB3: now reaches U?.12 (1Y3)
- net VDB2: now reaches U?.14 (1Y2)
- net VDB1: now reaches U?.16 (1Y1)
- net VDB0: now reaches U?.18 (1Y0)
- net VDB4: now reaches U?.3 (2Y0)
- net VDB5: now reaches U?.5 (2Y1)
- net VDB6: now reaches U?.7 (2Y2)
- net VDB7: now reaches U?.9 (2Y3)
- net VDB11: now reaches U?.12 (1Y3)
- net VDB10: now reaches U?.14 (1Y2)
- net VDB9: now reaches U?.16 (1Y1)
- net VDB8: now reaches U?.18 (1Y0)
- net VDB12: now reaches U?.3 (2Y0)
- net VDB13: now reaches U?.5 (2Y1)
- net VDB14: now reaches U?.7 (2Y2)
- net VDB15: now reaches U?.9 (2Y3)
Other:
- moved on the sheet: U?
