File: CES/WorkRegister.sch (KiCad schematic (older format))
At the start: 12 parts

Commit message: Adding 74HC versions of 74LS chips
Parts:
- removed U?: RT1, symbol 74xx:74LS173
- removed U?: RT2, symbol 74xx:74LS173
- removed U?: RT3, symbol 74xx:74LS173
- removed U?: RT4, symbol 74xx:74LS173
- added U?: RT1, symbol CES:74HC173
- added U?: RT2, symbol CES:74HC173
- added U?: RT3, symbol CES:74HC173
- added U?: RT4, symbol CES:74HC173
Changed lines of the file:
@@
 $EndDescr
-$Comp
-L 74xx:74LS173 U?
-U 1 1 61BEF6BF
-P 2800 8650
-AR Path="/60832B49/61BEF6BF" Ref="U?"  Part="1"
-AR Path="/60832B49/61BE6757/61BEF6BF" Ref="U?"  Part="1"
-F 0 "U?" H 3050 9450 50  0000 C CNN
-F 1 "RT4" H 2800 8650 50  0000 C CNN
-F 2 "" H 2800 8650 50  0001 C CNN
-F 3 "http://www.ti.com/lit/gpn/sn74LS173" H 2800 8650 50  0001 C CNN
-	1    2800 8650
-	1    0    0    -1
-$EndComp
 $Comp
 L 74xx:74HC244 U?
@@
 $EndComp
 $Comp
-L 74xx:74LS173 U?
-U 1 1 61BEF6AD
-P 2800 1600
-AR Path="/60832B49/61BEF6AD" Ref="U?"  Part="1"
-AR Path="/60832B49/61BE6757/61BEF6AD" Ref="U?"  Part="1"
-F 0 "U?" H 3050 2350 50  0000 C CNN
-F 1 "RT1" H 2800 1600 50  0000 C CNN
-F 2 "" H 2800 1600 50  0001 C CNN
-F 3 "http://www.ti.com/lit/gpn/sn74LS173" H 2800 1600 50  0001 C CNN
-	1    2800 1600
-	1    0    0    -1
-$EndComp
-$Comp
 L power:VCC #PWR?
 U 1 1 60860188
@@
 F 3 "https://assets.nexperia.com/documents/data-sheet/74HC_HCT244.pdf" H 5600 7150 50  0001 C CNN
 	1    5600 7150
-	1    0    0    -1
-$EndComp
-$Comp
-L 74xx:74LS173 U?
-U 1 1 61BEF6B9
-P 2800 6300
-AR Path="/60832B49/61BEF6B9" Ref="U?"  Part="1"
-AR Path="/60832B49/61BE6757/61BEF6B9" Ref="U?"  Part="1"
-F 0 "U?" H 3050 7050 50  0000 C CNN
-F 1 "RT3" H 2800 6300 50  0000 C CNN
-F 2 "" H 2800 6300 50  0001 C CNN
-F 3 "http://www.ti.com/lit/gpn/sn74LS173" H 2800 6300 50  0001 C CNN
-	1    2800 6300
 	1    0    0    -1
 $EndComp
@@
 Wire Wire Line
 	4000 2450 4000 3450
-$Comp
-L 74xx:74LS173 U?
-U 1 1 61BEF6B3
-P 2800 3950
-AR Path="/60832B49/61BEF6B3" Ref="U?"  Part="1"
-AR Path="/60832B49/61BE6757/61BEF6B3" Ref="U?"  Part="1"
-F 0 "U?" H 3050 4700 50  0000 C CNN
-F 1 "RT2" H 2800 3950 50  0000 C CNN
-F 2 "" H 2800 3950 50  0001 C CNN
-F 3 "http://www.ti.com/lit/gpn/sn74LS173" H 2800 3950 50  0001 C CNN
-	1    2800 3950
-	1    0    0    -1
-$EndComp
 Wire Wire Line
 	3300 3350 3900 3350
@@
 Wire Wire Line
 	1750 10250 1600 10250
+$Comp
+L CES:74HC173 U?
+U 1 1 60919F92
+P 2800 1600
+F 0 "U?" H 3050 2350 50  0000 C CNN
+F 1 "RT1" H 2800 1600 50  0000 C CNN
+F 2 "" H 2800 1600 50  0001 C CNN
+F 3 "http://www.ti.com/lit/gpn/cd74HC173" H 2800 1600 50  0001 C CNN
+	1    2800 1600
+	1    0    0    -1
+$EndComp
+$Comp
+L CES:74HC173 U?
+U 1 1 6091ACBA
+P 2800 3950
+F 0 "U?" H 3050 4700 50  0000 C CNN
+F 1 "RT2" H 2800 3950 50  0000 C CNN
+F 2 "" H 2800 3950 50  0001 C CNN
+F 3 "http://www.ti.com/lit/gpn/cd74HC173" H 2800 3950 50  0001 C CNN
+	1    2800 3950
+	1    0    0    -1
+$EndComp
+$Comp
+L CES:74HC173 U?
+U 1 1 6091B3BD
+P 2800 6300
+F 0 "U?" H 3050 7050 50  0000 C CNN
+F 1 "RT3" H 2800 6300 50  0000 C CNN
+F 2 "" H 2800 6300 50  0001 C CNN
+F 3 "http://www.ti.com/lit/gpn/cd74HC173" H 2800 6300 50  0001 C CNN
+	1    2800 6300
+	1    0    0    -1
+$EndComp
+$Comp
+L CES:74HC173 U?
+U 1 1 6091B937
+P 2800 8650
+F 0 "U?" H 3050 9400 50  0000 C CNN
+F 1 "RT4" H 2800 8650 50  0000 C CNN
+F 2 "" H 2800 8650 50  0001 C CNN
+F 3 "http://www.ti.com/lit/gpn/cd74HC173" H 2800 8650 50  0001 C CNN
+	1    2800 8650
+	1    0    0    -1
+$EndComp
 $EndSCHEMATC

Commit message: Control Unit
Parts:
- gave numbers to parts that had none: 12
Changed lines of the file:
@@
 $Descr A4 8268 11693 portrait
 encoding utf-8
-Sheet 4 16
+Sheet 4 17
 Title "CES"
 Date "2021-04-24"
@@
 $EndDescr
 $Comp
-L 74xx:74HC244 U?
+L 74xx:74HC244 U405
 U 1 1 61C140C4
 P 5600 2450
-F 0 "U?" H 5850 3100 50  0000 C CNN
+F 0 "U405" H 5850 3100 50  0000 C CNN
 F 1 "BT1" H 5600 2150 50  0000 C CNN
 F 2 "" H 5600 2450 50  0001 C CNN
@@
 $EndComp
 $Comp
-L power:VCC #PWR?
+L power:VCC #PWR0411
 U 1 1 60860188
 P 2800 700
-F 0 "#PWR?" H 2800 550 50  0001 C CNN
+F 0 "#PWR0411" H 2800 550 50  0001 C CNN
 F 1 "VCC" H 2900 800 50  0000 C CNN
 F 2 "" H 2800 700 50  0001 C CNN
@@
 $EndComp
 $Comp
-L power:GND #PWR?
+L power:GND #PWR0412
 U 1 1 608626EF
 P 2800 2500
-F 0 "#PWR?" H 2800 2250 50  0001 C CNN
+F 0 "#PWR0412" H 2800 2250 50  0001 C CNN
 F 1 "GND" H 2800 2300 50  0000 C CNN
 F 2 "" H 2800 2500 50  0001 C CNN
@@
 $EndComp
 $Comp
-L power:VCC #PWR?
+L power:VCC #PWR0415
 U 1 1 60864FFE
 P 2800 5400
-F 0 "#PWR?" H 2800 5250 50  0001 C CNN
+F 0 "#PWR0415" H 2800 5250 50  0001 C CNN
 F 1 "VCC" H 2815 5573 50  0000 C CNN
 F 2 "" H 2800 5400 50  0001 C CNN
@@
 $EndComp
 $Comp
-L power:VCC #PWR?
+L power:VCC #PWR0417
 U 1 1 608662FD
 P 2800 7750
-F 0 "#PWR?" H 2800 7600 50  0001 C CNN
+F 0 "#PWR0417" H 2800 7600 50  0001 C CNN
 F 1 "VCC" H 2815 7923 50  0000 C CNN
 F 2 "" H 2800 7750 50  0001 C CNN
@@
 $EndComp
 $Comp
-L power:GND #PWR?
+L power:GND #PWR0416
 U 1 1 60866ABA
 P 2800 7200
-F 0 "#PWR?" H 2800 6950 50  0001 C CNN
+F 0 "#PWR0416" H 2800 6950 50  0001 C CNN
 F 1 "GND" H 2805 7027 50  0000 C CNN
 F 2 "" H 2800 7200 50  0001 C CNN
@@
 $EndComp
 $Comp
-L power:GND #PWR?
+L power:GND #PWR0418
 U 1 1 60867089
 P 2800 9550
-F 0 "#PWR?" H 2800 9300 50  0001 C CNN
+F 0 "#PWR0418" H 2800 9300 50  0001 C CNN
 F 1 "GND" H 2805 9377 50  0000 C CNN
 F 2 "" H 2800 9550 50  0001 C CNN
@@
 	3300 8050 3900 8050
 $Comp
-L 74xx:74HC244 U?
+L 74xx:74HC244 U406
 U 1 1 61C140CA
 P 5600 7150
-F 0 "U?" H 5850 7800 50  0000 C CNN
+F 0 "U406" H 5850 7800 50  0000 C CNN
 F 1 "BT2" H 5600 6850 50  0000 C CNN
 F 2 "" H 5600 7150 50  0001 C CNN
@@
 Connection ~ 5000 7650
 $Comp
-L power:GND #PWR?
+L power:GND #PWR0420
 U 1 1 60884EA3
 P 5600 3250
-F 0 "#PWR?" H 5600 3000 50  0001 C CNN
+F 0 "#PWR0420" H 5600 3000 50  0001 C CNN
 F 1 "GND" H 5605 3077 50  0000 C CNN
 F 2 "" H 5600 3250 50  0001 C CNN
@@
 $EndComp
 $Comp
-L power:GND #PWR?
+L power:GND #PWR0422
 U 1 1 60885969
 P 5600 7950
-F 0 "#PWR?" H 5600 7700 50  0001 C CNN
+F 0 "#PWR0422" H 5600 7700 50  0001 C CNN
 F 1 "GND" H 5605 7777 50  0000 C CNN
 F 2 "" H 5600 7950 50  0001 C CNN
@@
 $EndComp
 $Comp
-L power:VCC #PWR?
+L power:VCC #PWR0421
 U 1 1 60885F6C
 P 5600 6350
-F 0 "#PWR?" H 5600 6200 50  0001 C CNN
+F 0 "#PWR0421" H 5600 6200 50  0001 C CNN
 F 1 "VCC" H 5615 6523 50  0000 C CNN
 F 2 "" H 5600 6350 50  0001 C CNN
@@
 $EndComp
 $Comp
-L power:VCC #PWR?
+L power:VCC #PWR0419
 U 1 1 608863BE
 P 5600 1650
-F 0 "#PWR?" H 5600 1500 50  0001 C CNN
+F 0 "#PWR0419" H 5600 1500 50  0001 C CNN
 F 1 "VCC" H 5615 1823 50  0000 C CNN
 F 2 "" H 5600 1650 50  0001 C CNN
@@
 SRT8
 $Comp
-L power:GND #PWR?
+L power:GND #PWR0414
 U 1 1 60863E8D
 P 2800 4850
-F 0 "#PWR?" H 2800 4600 50  0001 C CNN
+F 0 "#PWR0414" H 2800 4600 50  0001 C CNN
 F 1 "GND" H 2805 4677 50  0000 C CNN
 F 2 "" H 2800 4850 50  0001 C CNN
@@
 $EndComp
 $Comp
-L power:VCC #PWR?
+L power:VCC #PWR0413
 U 1 1 60863524
 P 2800 3050
-F 0 "#PWR?" H 2800 2900 50  0001 C CNN
+F 0 "#PWR0413" H 2800 2900 50  0001 C CNN
 F 1 "VCC" H 2815 3223 50  0000 C CNN
 F 2 "" H 2800 3050 50  0001 C CNN
@@
 Connection ~ 4200 1000
 $Comp
-L power:GND #PWR?
+L power:GND #PWR0403
 U 1 1 608D82FF
 P 2150 1650
-F 0 "#PWR?" H 2150 1400 50  0001 C CNN
+F 0 "#PWR0403" H 2150 1400 50  0001 C CNN
 F 1 "GND" H 2000 1550 50  0000 C CNN
 F 2 "" H 2150 1650 50  0001 C CNN
@@
 Connection ~ 2150 1600
 $Comp
-L power:GND #PWR?
+L power:GND #PWR0405
 U 1 1 608E9283
 P 2150 4000
-F 0 "#PWR?" H 2150 3750 50  0001 C CNN
+F 0 "#PWR0405" H 2150 3750 50  0001 C CNN
 F 1 "GND" H 2000 3900 50  0000 C CNN
 F 2 "" H 2150 4000 50  0001 C CNN
@@
 Connection ~ 2150 3950
 $Comp
-L power:GND #PWR?
+L power:GND #PWR0407
 U 1 1 608ED229
 P 2150 6350
-F 0 "#PWR?" H 2150 6100 50  0001 C CNN
+F 0 "#PWR0407" H 2150 6100 50  0001 C CNN
 F 1 "GND" H 2000 6250 50  0000 C CNN
 F 2 "" H 2150 6350 50  0001 C CNN
@@
 Connection ~ 2150 6300
 $Comp
-L power:GND #PWR?
+L power:GND #PWR0409
 U 1 1 608F1611
 P 2150 8700
-F 0 "#PWR?" H 2150 8450 50  0001 C CNN
+F 0 "#PWR0409" H 2150 8450 50  0001 C CNN
 F 1 "GND" H 2000 8600 50  0000 C CNN
 F 2 "" H 2150 8700 50  0001 C CNN
@@
 Connection ~ 2150 8650
 $Comp
-L power:GND #PWR?
+L power:GND #PWR0408
 U 1 1 608F5997
 P 2150 6950
-F 0 "#PWR?" H 2150 6700 50  0001 C CNN
+F 0 "#PWR0408" H 2150 6700 50  0001 C CNN
 F 1 "GND" H 2155 6777 50  0000 C CNN
 F 2 "" H 2150 6950 50  0001 C CNN
@@
 	2150 6900 2150 6950
 $Comp
-L power:GND #PWR?
+L power:GND #PWR0410
 U 1 1 608FA806
 P 2150 9300
-F 0 "#PWR?" H 2150 9050 50  0001 C CNN
+F 0 "#PWR0410" H 2150 9050 50  0001 C CNN
 F 1 "GND" H 2155 9127 50  0000 C CNN
 F 2 "" H 2150 9300 50  0001 C CNN
@@
 	2150 9250 2150 9300
 $Comp
-L power:GND #PWR?
+L power:GND #PWR0406
 U 1 1 608FF23E
 P 2150 4600
-F 0 "#PWR?" H 2150 4350 50  0001 C CNN
+F 0 "#PWR0406" H 2150 4350 50  0001 C CNN
 F 1 "GND" H 2155 4427 50  0000 C CNN
 F 2 "" H 2150 4600 50  0001 C CNN
@@
 	2150 4550 2150 4600
 $Comp
-L power:GND #PWR?
+L power:GND #PWR0404
 U 1 1 60903E02
 P 2150 2250
-F 0 "#PWR?" H 2150 2000 50  0001 C CNN
+F 0 "#PWR0404" H 2150 2000 50  0001 C CNN
 F 1 "GND" H 2155 2077 50  0000 C CNN
 F 2 "" H 2150 2250 50  0001 C CNN
@@
 	1150 8350 2300 8350
 $Comp
-L Device:C C?
+L Device:C C401
 U 1 1 60971044
 P 1000 10500
-F 0 "C?" H 1050 10600 50  0000 L CNN
+F 0 "C401" H 1050 10600 50  0000 L CNN
 F 1 "100nF" H 1050 10400 50  0000 L CNN
 F 2 "" H 1038 10350 50  0001 C CNN
@@
 $EndComp
 $Comp
-L Device:C C?
+L Device:C C402
 U 1 1 609716E3
 P 1300 10500
-F 0 "C?" H 1350 10600 50  0000 L CNN
+F 0 "C402" H 1350 10600 50  0000 L CNN
 F 1 "100nF" H 1350 10400 50  0000 L CNN
 F 2 "" H 1338 10350 50  0001 C CNN
@@
 $EndComp
 $Comp
-L Device:C C?
+L Device:C C403
 U 1 1 60971BAE
 P 1600 10500
-F 0 "C?" H 1650 10600 50  0000 L CNN
+F 0 "C403" H 1650 10600 50  0000 L CNN
 F 1 "100nF" H 1650 10400 50  0000 L CNN
 F 2 "" H 1638 10350 50  0001 C CNN
@@
 $EndComp
 $Comp
-L Device:C C?
+L Device:C C404
 U 1 1 6097201C
 P 1900 10500
-F 0 "C?" H 1950 10600 50  0000 L CNN
+F 0 "C404" H 1950 10600 50  0000 L CNN
 F 1 "100nF" H 1950 10400 50  0000 L CNN
 F 2 "" H 1938 10350 50  0001 C CNN
@@
 $EndComp
 $Comp
-L Device:C C?
+L Device:C C405
 U 1 1 60972449
 P 2200 10500
-F 0 "C?" H 2250 10600 50  0000 L CNN
+F 0 "C405" H 2250 10600 50  0000 L CNN
 F 1 "100nF" H 2250 10400 50  0000 L CNN
 F 2 "" H 2238 10350 50  0001 C CNN
@@
 $EndComp
 $Comp
-L Device:C C?
+L Device:C C406
 U 1 1 60972816
 P 2500 10500
-F 0 "C?" H 2550 10600 50  0000 L CNN
+F 0 "C406" H 2550 10600 50  0000 L CNN
 F 1 "100nF" H 2550 10400 50  0000 L CNN
 F 2 "" H 2538 10350 50  0001 C CNN
@@
 	2200 10250 1900 10250
 $Comp
-L power:GND #PWR?
+L power:GND #PWR0402
 U 1 1 609B8FEE
 P 1750 10750
-F 0 "#PWR?" H 1750 10500 50  0001 C CNN
+F 0 "#PWR0402" H 1750 10500 50  0001 C CNN
 F 1 "GND" H 1755 10577 50  0000 C CNN
 F 2 "" H 1750 10750 50  0001 C CNN
@@
 	1750 10750 1900 10750
 $Comp
-L power:VCC #PWR?
+L power:VCC #PWR0401
 U 1 1 609B9780
 P 1750 10250
-F 0 "#PWR?" H 1750 10100 50  0001 C CNN
+F 0 "#PWR0401" H 1750 10100 50  0001 C CNN
 F 1 "VCC" H 1765 10423 50  0000 C CNN
 F 2 "" H 1750 10250 50  0001 C CNN
@@
 	1750 10250 1600 10250
 $Comp
-L CES:74HC173 U?
+L CES:74HC173 U401
 U 1 1 60919F92
 P 2800 1600
-F 0 "U?" H 3050 2350 50  0000 C CNN
+F 0 "U401" H 3050 2350 50  0000 C CNN
 F 1 "RT1" H 2800 1600 50  0000 C CNN
 F 2 "" H 2800 1600 50  0001 C CNN
@@
 $EndComp
 $Comp
-L CES:74HC173 U?
+L CES:74HC173 U402
 U 1 1 6091ACBA
 P 2800 3950
-F 0 "U?" H 3050 4700 50  0000 C CNN
+F 0 "U402" H 3050 4700 50  0000 C CNN
 F 1 "RT2" H 2800 3950 50  0000 C CNN
 F 2 "" H 2800 3950 50  0001 C CNN
@@
 $EndComp
 $Comp
-L CES:74HC173 U?
+L CES:74HC173 U403
 U 1 1 6091B3BD
 P 2800 6300
-F 0 "U?" H 3050 7050 50  0000 C CNN
+F 0 "U403" H 3050 7050 50  0000 C CNN
 F 1 "RT3" H 2800 6300 50  0000 C CNN
 F 2 "" H 2800 6300 50  0001 C CNN
@@
 $EndComp
 $Comp
-L CES:74HC173 U?
+L CES:74HC173 U404
 U 1 1 6091B937
 P 2800 8650
-F 0 "U?" H 3050 9400 50  0000 C CNN
+F 0 "U404" H 3050 9400 50  0000 C CNN
 F 1 "RT4" H 2800 8650 50  0000 C CNN
 F 2 "" H 2800 8650 50  0001 C CNN

Commit message: Assigning footprints and generating netlist
Parts:
- C401, C402, C403, C404, C405, C406: footprint (none) -> Capacitor_THT:CP_Radial_D5.0mm_P2.50mm
- U401, U402, U403, U404: footprint (none) -> Package_DIP:DIP-16_W7.62mm
- U405, U406: footprint (none) -> Package_DIP:DIP-20_W7.62mm
Changed lines of the file:
@@
 F 0 "U405" H 5850 3100 50  0000 C CNN
 F 1 "BT1" H 5600 2150 50  0000 C CNN
-F 2 "" H 5600 2450 50  0001 C CNN
+F 2 "Package_DIP:DIP-20_W7.62mm" H 5600 2450 50  0001 C CNN
 F 3 "https://assets.nexperia.com/documents/data-sheet/74HC_HCT244.pdf" H 5600 2450 50  0001 C CNN
 	1    5600 2450
@@
 F 0 "U406" H 5850 7800 50  0000 C CNN
 F 1 "BT2" H 5600 6850 50  0000 C CNN
-F 2 "" H 5600 7150 50  0001 C CNN
+F 2 "Package_DIP:DIP-20_W7.62mm" H 5600 7150 50  0001 C CNN
 F 3 "https://assets.nexperia.com/documents/data-sheet/74HC_HCT244.pdf" H 5600 7150 50  0001 C CNN
 	1    5600 7150
@@
 F 0 "C401" H 1050 10600 50  0000 L CNN
 F 1 "100nF" H 1050 10400 50  0000 L CNN
-F 2 "" H 1038 10350 50  0001 C CNN
+F 2 "Capacitor_THT:CP_Radial_D5.0mm_P2.50mm" H 1038 10350 50  0001 C CNN
 F 3 "~" H 1000 10500 50  0001 C CNN
 	1    1000 10500
@@
 F 0 "C402" H 1350 10600 50  0000 L CNN
 F 1 "100nF" H 1350 10400 50  0000 L CNN
-F 2 "" H 1338 10350 50  0001 C CNN
+F 2 "Capacitor_THT:CP_Radial_D5.0mm_P2.50mm" H 1338 10350 50  0001 C CNN
 F 3 "~" H 1300 10500 50  0001 C CNN
 	1    1300 10500
@@
 F 0 "C403" H 1650 10600 50  0000 L CNN
 F 1 "100nF" H 1650 10400 50  0000 L CNN
-F 2 "" H 1638 10350 50  0001 C CNN
+F 2 "Capacitor_THT:CP_Radial_D5.0mm_P2.50mm" H 1638 10350 50  0001 C CNN
 F 3 "~" H 1600 10500 50  0001 C CNN
 	1    1600 10500
@@
 F 0 "C404" H 1950 10600 50  0000 L CNN
 F 1 "100nF" H 1950 10400 50  0000 L CNN
-F 2 "" H 1938 10350 50  0001 C CNN
+F 2 "Capacitor_THT:CP_Radial_D5.0mm_P2.50mm" H 1938 10350 50  0001 C CNN
 F 3 "~" H 1900 10500 50  0001 C CNN
 	1    1900 10500
@@
 F 0 "C405" H 2250 10600 50  0000 L CNN
 F 1 "100nF" H 2250 10400 50  0000 L CNN
-F 2 "" H 2238 10350 50  0001 C CNN
+F 2 "Capacitor_THT:CP_Radial_D5.0mm_P2.50mm" H 2238 10350 50  0001 C CNN
 F 3 "~" H 2200 10500 50  0001 C CNN
 	1    2200 10500
@@
 F 0 "C406" H 2550 10600 50  0000 L CNN
 F 1 "100nF" H 2550 10400 50  0000 L CNN
-F 2 "" H 2538 10350 50  0001 C CNN
+F 2 "Capacitor_THT:CP_Radial_D5.0mm_P2.50mm" H 2538 10350 50  0001 C CNN
 F 3 "~" H 2500 10500 50  0001 C CNN
 	1    2500 10500
@@
 F 0 "U401" H 3050 2350 50  0000 C CNN
 F 1 "RT1" H 2800 1600 50  0000 C CNN
-F 2 "" H 2800 1600 50  0001 C CNN
+F 2 "Package_DIP:DIP-16_W7.62mm" H 2800 1600 50  0001 C CNN
 F 3 "http://www.ti.com/lit/gpn/cd74HC173" H 2800 1600 50  0001 C CNN
 	1    2800 1600
@@
 F 0 "U402" H 3050 4700 50  0000 C CNN
 F 1 "RT2" H 2800 3950 50  0000 C CNN
-F 2 "" H 2800 3950 50  0001 C CNN
+F 2 "Package_DIP:DIP-16_W7.62mm" H 2800 3950 50  0001 C CNN
 F 3 "http://www.ti.com/lit/gpn/cd74HC173" H 2800 3950 50  0001 C CNN
 	1    2800 3950
@@
 F 0 "U403" H 3050 7050 50  0000 C CNN
 F 1 "RT3" H 2800 6300 50  0000 C CNN
-F 2 "" H 2800 6300 50  0001 C CNN
+F 2 "Package_DIP:DIP-16_W7.62mm" H 2800 6300 50  0001 C CNN
 F 3 "http://www.ti.com/lit/gpn/cd74HC173" H 2800 6300 50  0001 C CNN
 	1    2800 6300
@@
 F 0 "U404" H 3050 9400 50  0000 C CNN
 F 1 "RT4" H 2800 8650 50  0000 C CNN
-F 2 "" H 2800 8650 50  0001 C CNN
+F 2 "Package_DIP:DIP-16_W7.62mm" H 2800 8650 50  0001 C CNN
 F 3 "http://www.ti.com/lit/gpn/cd74HC173" H 2800 8650 50  0001 C CNN
 	1    2800 8650
