File: CES/AddressDecoding.sch (KiCad schematic (older format))
At the start: 8 parts, among them U1001 74HC02, U1002 74HC30, U1003 74HC10, U1004 74HC08

Commit message: Assigning footprints and generating netlist
Parts:
- C1001, C1002, C1003, C1004: footprint (none) -> Capacitor_THT:CP_Radial_D5.0mm_P2.50mm
- U1001, U1002, U1003, U1004: footprint (none) -> Package_DIP:DIP-14_W7.62mm
Changed lines of the file:
@@
 F 0 "U1001" H 5200 1975 50  0000 C CNN
 F 1 "74HC02" H 5200 1884 50  0000 C CNN
-F 2 "" H 5200 1650 50  0001 C CNN
+F 2 "Package_DIP:DIP-14_W7.62mm" H 5200 1650 50  0001 C CNN
 F 3 "http://www.ti.com/lit/gpn/sn74hc02" H 5200 1650 50  0001 C CNN
 	1    5200 1650
@@
 F 0 "U1001" H 5200 2525 50  0000 C CNN
 F 1 "74HC02" H 5200 2434 50  0000 C CNN
-F 2 "" H 5200 2200 50  0001 C CNN
+F 2 "Package_DIP:DIP-14_W7.62mm" H 5200 2200 50  0001 C CNN
 F 3 "http://www.ti.com/lit/gpn/sn74hc02" H 5200 2200 50  0001 C CNN
 	4    5200 2200
@@
 F 0 "U1001" H 6000 7200 50  0000 L CNN
 F 1 "74HC02" H 5750 6850 50  0000 L CNN
-F 2 "" H 5900 6850 50  0001 C CNN
+F 2 "Package_DIP:DIP-14_W7.62mm" H 5900 6850 50  0001 C CNN
 F 3 "http://www.ti.com/lit/gpn/sn74hc02" H 5900 6850 50  0001 C CNN
 	5    5900 6850
@@
 F 0 "C1001" H 3100 6950 50  0000 L CNN
 F 1 "100nF" H 3100 6750 50  0000 L CNN
-F 2 "" H 3088 6700 50  0001 C CNN
+F 2 "Capacitor_THT:CP_Radial_D5.0mm_P2.50mm" H 3088 6700 50  0001 C CNN
 F 3 "~" H 3050 6850 50  0001 C CNN
 	1    3050 6850
@@
 F 0 "C1002" H 3400 6950 50  0000 L CNN
 F 1 "100nF" H 3400 6750 50  0000 L CNN
-F 2 "" H 3388 6700 50  0001 C CNN
+F 2 "Capacitor_THT:CP_Radial_D5.0mm_P2.50mm" H 3388 6700 50  0001 C CNN
 F 3 "~" H 3350 6850 50  0001 C CNN
 	1    3350 6850
@@
 F 0 "C1003" H 3700 6950 50  0000 L CNN
 F 1 "100nF" H 3700 6750 50  0000 L CNN
-F 2 "" H 3688 6700 50  0001 C CNN
+F 2 "Capacitor_THT:CP_Radial_D5.0mm_P2.50mm" H 3688 6700 50  0001 C CNN
 F 3 "~" H 3650 6850 50  0001 C CNN
 	1    3650 6850
@@
 F 0 "C1004" H 4000 6950 50  0000 L CNN
 F 1 "100nF" H 4000 6750 50  0000 L CNN
-F 2 "" H 3988 6700 50  0001 C CNN
+F 2 "Capacitor_THT:CP_Radial_D5.0mm_P2.50mm" H 3988 6700 50  0001 C CNN
 F 3 "~" H 3950 6850 50  0001 C CNN
 	1    3950 6850
@@
 F 0 "U1001" H 6450 4375 50  0000 C CNN
 F 1 "74HC02" H 6450 4284 50  0000 C CNN
-F 2 "" H 6450 4050 50  0001 C CNN
+F 2 "Package_DIP:DIP-14_W7.62mm" H 6450 4050 50  0001 C CNN
 F 3 "http://www.ti.com/lit/gpn/sn74hc02" H 6450 4050 50  0001 C CNN
 	3    6450 4050
@@
 F 0 "U1004" H 6450 2075 50  0000 C CNN
 F 1 "74HC08" H 6450 1984 50  0000 C CNN
-F 2 "" H 6450 1750 50  0001 C CNN
+F 2 "Package_DIP:DIP-14_W7.62mm" H 6450 1750 50  0001 C CNN
 F 3 "http://www.ti.com/lit/gpn/sn74HC08" H 6450 1750 50  0001 C CNN
 	1    6450 1750
@@
 F 0 "U1004" H 5050 7200 50  0000 L CNN
 F 1 "74HC08" H 4850 6850 50  0000 L CNN
-F 2 "" H 5000 6850 50  0001 C CNN
+F 2 "Package_DIP:DIP-14_W7.62mm" H 5000 6850 50  0001 C CNN
 F 3 "http://www.ti.com/lit/gpn/sn74HC08" H 5000 6850 50  0001 C CNN
 	5    5000 6850
@@
 F 0 "U1003" H 6450 2775 50  0000 C CNN
 F 1 "74HC10" H 6450 2684 50  0000 C CNN
-F 2 "" H 6450 2450 50  0001 C CNN
+F 2 "Package_DIP:DIP-14_W7.62mm" H 6450 2450 50  0001 C CNN
 F 3 "http://www.ti.com/lit/gpn/sn74HC10" H 6450 2450 50  0001 C CNN
 	1    6450 2450
@@
 F 0 "U1003" H 5200 4925 50  0000 C CNN
 F 1 "74HC10" H 5200 4834 50  0000 C CNN
-F 2 "" H 5200 4600 50  0001 C CNN
+F 2 "Package_DIP:DIP-14_W7.62mm" H 5200 4600 50  0001 C CNN
 F 3 "http://www.ti.com/lit/gpn/sn74HC10" H 5200 4600 50  0001 C CNN
 	2    5200 4600
@@
 F 0 "U1003" H 5500 7200 50  0000 L CNN
 F 1 "74HC10" H 5300 6850 50  0000 L CNN
-F 2 "" H 5450 6850 50  0001 C CNN
+F 2 "Package_DIP:DIP-14_W7.62mm" H 5450 6850 50  0001 C CNN
 F 3 "http://www.ti.com/lit/gpn/sn74HC10" H 5450 6850 50  0001 C CNN
 	4    5450 6850
@@
 F 0 "U1002" H 5200 4075 50  0000 C CNN
 F 1 "74HC30" H 5200 3984 50  0000 C CNN
-F 2 "" H 5200 3550 50  0001 C CNN
+F 2 "Package_DIP:DIP-14_W7.62mm" H 5200 3550 50  0001 C CNN
 F 3 "http://www.ti.com/lit/gpn/sn74HC30" H 5200 3550 50  0001 C CNN
 	1    5200 3550
@@
 F 0 "U1002" H 4600 7200 50  0000 L CNN
 F 1 "74HC30" H 4400 6850 50  0000 L CNN
-F 2 "" H 4550 6850 50  0001 C CNN
+F 2 "Package_DIP:DIP-14_W7.62mm" H 4550 6850 50  0001 C CNN
 F 3 "http://www.ti.com/lit/gpn/sn74HC30" H 4550 6850 50  0001 C CNN
 	2    4550 6850

Commit message: Correcting footprints errors
Parts:
- C1001, C1002, C1003, C1004: footprint Capacitor_THT:CP_Radial_D5.0mm_P2.50mm -> Capacitor_THT:C_Disc_D4.3mm_W1.9mm_P5.00mm
- renumbered U1002 to U1001, U1004 to U1002, U1001 to U1003, U1003 to U1004
Changed lines of the file:
@@
 $EndDescr
 $Comp
-L 74xx:74HC02 U1001
+L 74xx:74HC02 U1003
 U 1 1 610C3622
 P 5200 1650
-F 0 "U1001" H 5200 1975 50  0000 C CNN
+F 0 "U1003" H 5200 1975 50  0000 C CNN
 F 1 "74HC02" H 5200 1884 50  0000 C CNN
 F 2 "Package_DIP:DIP-14_W7.62mm" H 5200 1650 50  0001 C CNN
@@
 $EndComp
 $Comp
-L 74xx:74HC02 U1001
+L 74xx:74HC02 U1003
 U 4 1 610C7DE1
 P 5200 2200
-F 0 "U1001" H 5200 2525 50  0000 C CNN
+F 0 "U1003" H 5200 2525 50  0000 C CNN
 F 1 "74HC02" H 5200 2434 50  0000 C CNN
 F 2 "Package_DIP:DIP-14_W7.62mm" H 5200 2200 50  0001 C CNN
@@
 $EndComp
 $Comp
-L 74xx:74HC02 U1001
+L 74xx:74HC02 U1003
 U 5 1 610C967C
 P 5900 6850
-F 0 "U1001" H 6000 7200 50  0000 L CNN
+F 0 "U1003" H 6000 7200 50  0000 L CNN
 F 1 "74HC02" H 5750 6850 50  0000 L CNN
 F 2 "Package_DIP:DIP-14_W7.62mm" H 5900 6850 50  0001 C CNN
@@
 F 0 "C1001" H 3100 6950 50  0000 L CNN
 F 1 "100nF" H 3100 6750 50  0000 L CNN
-F 2 "Capacitor_THT:CP_Radial_D5.0mm_P2.50mm" H 3088 6700 50  0001 C CNN
+F 2 "Capacitor_THT:C_Disc_D4.3mm_W1.9mm_P5.00mm" H 3088 6700 50  0001 C CNN
 F 3 "~" H 3050 6850 50  0001 C CNN
 	1    3050 6850
@@
 F 0 "C1002" H 3400 6950 50  0000 L CNN
 F 1 "100nF" H 3400 6750 50  0000 L CNN
-F 2 "Capacitor_THT:CP_Radial_D5.0mm_P2.50mm" H 3388 6700 50  0001 C CNN
+F 2 "Capacitor_THT:C_Disc_D4.3mm_W1.9mm_P5.00mm" H 3388 6700 50  0001 C CNN
 F 3 "~" H 3350 6850 50  0001 C CNN
 	1    3350 6850
@@
 F 0 "C1003" H 3700 6950 50  0000 L CNN
 F 1 "100nF" H 3700 6750 50  0000 L CNN
-F 2 "Capacitor_THT:CP_Radial_D5.0mm_P2.50mm" H 3688 6700 50  0001 C CNN
+F 2 "Capacitor_THT:C_Disc_D4.3mm_W1.9mm_P5.00mm" H 3688 6700 50  0001 C CNN
 F 3 "~" H 3650 6850 50  0001 C CNN
 	1    3650 6850
@@
 F 0 "C1004" H 4000 6950 50  0000 L CNN
 F 1 "100nF" H 4000 6750 50  0000 L CNN
-F 2 "Capacitor_THT:CP_Radial_D5.0mm_P2.50mm" H 3988 6700 50  0001 C CNN
+F 2 "Capacitor_THT:C_Disc_D4.3mm_W1.9mm_P5.00mm" H 3988 6700 50  0001 C CNN
 F 3 "~" H 3950 6850 50  0001 C CNN
 	1    3950 6850
@@
 	3350 7100 3500 7100
 $Comp
-L power:VCC #PWR01002
+L power:VCC #PWR01001
 U 1 1 6119B6D1
 P 3500 6600
-F 0 "#PWR01002" H 3500 6450 50  0001 C CNN
+F 0 "#PWR01001" H 3500 6450 50  0001 C CNN
 F 1 "VCC" H 3515 6773 50  0000 C CNN
 F 2 "" H 3500 6600 50  0001 C CNN
@@
 	5200 7450 5450 7450
 $Comp
-L power:GND #PWR01003
+L power:GND #PWR01002
 U 1 1 6119D5D7
 P 3500 7100
-F 0 "#PWR01003" H 3500 6850 50  0001 C CNN
+F 0 "#PWR01002" H 3500 6850 50  0001 C CNN
 F 1 "GND" H 3505 6927 50  0000 C CNN
 F 2 "" H 3500 7100 50  0001 C CNN
@@
 	3950 4700 4900 4700
 $Comp
-L power:VCC #PWR01001
+L power:VCC #PWR01003
 U 1 1 6111F1B8
 P 3950 4700
-F 0 "#PWR01001" H 3950 4550 50  0001 C CNN
+F 0 "#PWR01003" H 3950 4550 50  0001 C CNN
 F 1 "VCC" H 3850 4800 50  0000 C CNN
 F 2 "" H 3950 4700 50  0001 C CNN
@@
 A5
 $Comp
-L 74xx:74HC02 U1001
+L 74xx:74HC02 U1003
 U 3 1 610C6523
 P 6450 4050
-F 0 "U1001" H 6450 4375 50  0000 C CNN
+F 0 "U1003" H 6450 4375 50  0000 C CNN
 F 1 "74HC02" H 6450 4284 50  0000 C CNN
 F 2 "Package_DIP:DIP-14_W7.62mm" H 6450 4050 50  0001 C CNN
@@
 $EndComp
 $Comp
-L CES:74HC08 U1004
+L CES:74HC08 U1002
 U 1 1 608C4157
 P 6450 1750
-F 0 "U1004" H 6450 2075 50  0000 C CNN
+F 0 "U1002" H 6450 2075 50  0000 C CNN
 F 1 "74HC08" H 6450 1984 50  0000 C CNN
 F 2 "Package_DIP:DIP-14_W7.62mm" H 6450 1750 50  0001 C CNN
@@
 $EndComp
 $Comp
-L CES:74HC08 U1004
+L CES:74HC08 U1002
 U 5 1 608CB98B
 P 5000 6850
-F 0 "U1004" H 5050 7200 50  0000 L CNN
+F 0 "U1002" H 5050 7200 50  0000 L CNN
 F 1 "74HC08" H 4850 6850 50  0000 L CNN
 F 2 "Package_DIP:DIP-14_W7.62mm" H 5000 6850 50  0001 C CNN
@@
 $EndComp
 $Comp
-L CES:74HC10 U1003
+L CES:74HC10 U1004
 U 1 1 608E7F40
 P 6450 2450
-F 0 "U1003" H 6450 2775 50  0000 C CNN
+F 0 "U1004" H 6450 2775 50  0000 C CNN
 F 1 "74HC10" H 6450 2684 50  0000 C CNN
 F 2 "Package_DIP:DIP-14_W7.62mm" H 6450 2450 50  0001 C CNN
@@
 $EndComp
 $Comp
-L CES:74HC10 U1003
+L CES:74HC10 U1004
 U 2 1 608E8B0D
 P 5200 4600
-F 0 "U1003" H 5200 4925 50  0000 C CNN
+F 0 "U1004" H 5200 4925 50  0000 C CNN
 F 1 "74HC10" H 5200 4834 50  0000 C CNN
 F 2 "Package_DIP:DIP-14_W7.62mm" H 5200 4600 50  0001 C CNN
@@
 $EndComp
 $Comp
-L CES:74HC10 U1003
+L CES:74HC10 U1004
 U 4 1 608EBE5C
 P 5450 6850
-F 0 "U1003" H 5500 7200 50  0000 L CNN
+F 0 "U1004" H 5500 7200 50  0000 L CNN
 F 1 "74HC10" H 5300 6850 50  0000 L CNN
 F 2 "Package_DIP:DIP-14_W7.62mm" H 5450 6850 50  0001 C CNN
@@
 $EndComp
 $Comp
-L CES:74HC30 U1002
+L CES:74HC30 U1001
 U 1 1 608F4EEB
 P 5200 3550
-F 0 "U1002" H 5200 4075 50  0000 C CNN
+F 0 "U1001" H 5200 4075 50  0000 C CNN
 F 1 "74HC30" H 5200 3984 50  0000 C CNN
 F 2 "Package_DIP:DIP-14_W7.62mm" H 5200 3550 50  0001 C CNN
@@
 $EndComp
 $Comp
-L CES:74HC30 U1002
+L CES:74HC30 U1001
 U 2 1 608F620B
 P 4550 6850
-F 0 "U1002" H 4600 7200 50  0000 L CNN
+F 0 "U1001" H 4600 7200 50  0000 L CNN
 F 1 "74HC30" H 4400 6850 50  0000 L CNN
 F 2 "Package_DIP:DIP-14_W7.62mm" H 4550 6850 50  0001 C CNN
