File: CES/Clock.sch (KiCad schematic (older format))
At the start: 24 parts

Commit message: Control Unit
Parts:
- gave numbers to parts that had none: 13
Changed lines of the file:
@@
 $Descr A4 11693 8268
 encoding utf-8
-Sheet 15 16
+Sheet 15 17
 Title ""
 Date ""
@@
 $EndDescr
 $Comp
-L CES:74HC4040 U?
+L CES:74HC4040 U1602
 U 1 1 611C2E57
 P 3600 3550
-F 0 "U?" H 3850 4200 50  0000 C CNN
+F 0 "U1602" H 3850 4200 50  0000 C CNN
 F 1 "74HC4040" H 3350 4200 50  0000 C CNN
 F 2 "" H 4800 4700 50  0001 C CNN
@@
 $EndComp
 $Comp
-L 74xx:74HC04 U?
+L 74xx:74HC04 U1601
 U 1 1 611C41A7
 P 1150 3450
-F 0 "U?" H 1150 3767 50  0000 C CNN
+F 0 "U1601" H 1150 3767 50  0000 C CNN
 F 1 "74HC04" H 1150 3676 50  0000 C CNN
 F 2 "" H 1150 3450 50  0001 C CNN
@@
 $EndComp
 $Comp
-L 74xx:74HC04 U?
+L 74xx:74HC04 U1601
 U 2 1 611C4BC1
 P 2200 3450
-F 0 "U?" H 2200 3767 50  0000 C CNN
+F 0 "U1601" H 2200 3767 50  0000 C CNN
 F 1 "74HC04" H 2200 3676 50  0000 C CNN
 F 2 "" H 2200 3450 50  0001 C CNN
@@
 $EndComp
 $Comp
-L 74xx:74HC04 U?
+L 74xx:74HC04 U1601
 U 3 1 611C4F48
 P 10750 850
-F 0 "U?" H 10750 1167 50  0000 C CNN
+F 0 "U1601" H 10750 1167 50  0000 C CNN
 F 1 "74HC04" H 10750 1076 50  0000 C CNN
 F 2 "" H 10750 850 50  0001 C CNN
@@
 $EndComp
 $Comp
-L 74xx:74HC04 U?
+L 74xx:74HC04 U1601
 U 5 1 611C5E55
 P 10750 1750
-F 0 "U?" H 10750 2067 50  0000 C CNN
+F 0 "U1601" H 10750 2067 50  0000 C CNN
 F 1 "74HC04" H 10750 1976 50  0000 C CNN
 F 2 "" H 10750 1750 50  0001 C CNN
@@
 $EndComp
 $Comp
-L 74xx:74HC04 U?
+L 74xx:74HC04 U1601
 U 6 1 611C6A1E
 P 10750 2200
-F 0 "U?" H 10750 2517 50  0000 C CNN
+F 0 "U1601" H 10750 2517 50  0000 C CNN
 F 1 "74HC04" H 10750 2426 50  0000 C CNN
 F 2 "" H 10750 2200 50  0001 C CNN
@@
 $EndComp
 $Comp
-L 74xx:74HC04 U?
+L 74xx:74HC04 U1601
 U 7 1 611C732B
 P 2200 6850
-F 0 "U?" H 1800 6900 50  0000 L CNN
+F 0 "U1601" H 1800 6900 50  0000 L CNN
 F 1 "74HC04" H 1700 6750 50  0000 L CNN
 F 2 "" H 2200 6850 50  0001 C CNN
@@
 $EndComp
 $Comp
-L Device:R R?
+L Device:R R1601
 U 1 1 611C8E54
 P 1150 2750
-F 0 "R?" V 943 2750 50  0000 C CNN
+F 0 "R1601" V 943 2750 50  0000 C CNN
 F 1 "1M" V 1034 2750 50  0000 C CNN
 F 2 "" V 1080 2750 50  0001 C CNN
@@
 Connection ~ 1550 3450
 $Comp
-L Device:R R?
+L Device:R R1602
 U 1 1 611C9DC3
 P 1550 3800
-F 0 "R?" H 1620 3846 50  0000 L CNN
+F 0 "R1602" H 1620 3846 50  0000 L CNN
 F 1 "470" H 1620 3755 50  0000 L CNN
 F 2 "" V 1480 3800 50  0001 C CNN
@@
 $EndComp
 $Comp
-L Device:Crystal Y?
+L Device:Crystal Y1601
 U 1 1 611CAB54
 P 1150 4150
-F 0 "Y?" H 1150 4418 50  0000 C CNN
+F 0 "Y1601" H 1150 4418 50  0000 C CNN
 F 1 "8MHz" H 1150 4327 50  0000 C CNN
 F 2 "" H 1150 4150 50  0001 C CNN
@@
 Connection ~ 750  3450
 $Comp
-L Device:C C?
+L Device:C C1602
 U 1 1 611CB7AB
 P 1550 4550
-F 0 "C?" H 1665 4596 50  0000 L CNN
+F 0 "C1602" H 1665 4596 50  0000 L CNN
 F 1 "33pF" H 1665 4505 50  0000 L CNN
 F 2 "" H 1588 4400 50  0001 C CNN
@@
 $EndComp
 $Comp
-L Device:C C?
+L Device:C C1601
 U 1 1 611CBED0
 P 750 4550
-F 0 "C?" H 865 4596 50  0000 L CNN
+F 0 "C1601" H 865 4596 50  0000 L CNN
 F 1 "33pF" H 865 4505 50  0000 L CNN
 F 2 "" H 788 4400 50  0001 C CNN
@@
 Connection ~ 750  4150
 $Comp
-L power:GND #PWR?
+L power:GND #PWR01601
 U 1 1 611CCD7F
 P 750 4850
-F 0 "#PWR?" H 750 4600 50  0001 C CNN
+F 0 "#PWR01601" H 750 4600 50  0001 C CNN
 F 1 "GND" H 755 4677 50  0000 C CNN
 F 2 "" H 750 4850 50  0001 C CNN
@@
 $EndComp
 $Comp
-L power:GND #PWR?
+L power:GND #PWR01602
 U 1 1 611CD204
 P 1550 4850
-F 0 "#PWR?" H 1550 4600 50  0001 C CNN
+F 0 "#PWR01602" H 1550 4600 50  0001 C CNN
 F 1 "GND" H 1555 4677 50  0000 C CNN
 F 2 "" H 1550 4850 50  0001 C CNN
@@
 	2500 3450 3150 3450
 $Comp
-L power:GND #PWR?
+L power:GND #PWR01607
 U 1 1 611D24E4
 P 3600 4650
-F 0 "#PWR?" H 3600 4400 50  0001 C CNN
+F 0 "#PWR01607" H 3600 4400 50  0001 C CNN
 F 1 "GND" H 3605 4477 50  0000 C CNN
 F 2 "" H 3600 4650 50  0001 C CNN
@@
 	3600 4450 3600 4650
 $Comp
-L power:GND #PWR?
+L power:GND #PWR01605
 U 1 1 611D2E1D
 P 3000 4000
-F 0 "#PWR?" H 3000 3750 50  0001 C CNN
+F 0 "#PWR01605" H 3000 3750 50  0001 C CNN
 F 1 "GND" H 3005 3827 50  0000 C CNN
 F 2 "" H 3000 4000 50  0001 C CNN
@@
 	3000 3850 3100 3850
 $Comp
-L power:VCC #PWR?
+L power:VCC #PWR01606
 U 1 1 611D356D
 P 3600 2600
-F 0 "#PWR?" H 3600 2450 50  0001 C CNN
+F 0 "#PWR01606" H 3600 2450 50  0001 C CNN
 F 1 "VCC" H 3615 2773 50  0000 C CNN
 F 2 "" H 3600 2600 50  0001 C CNN
@@
 	3600 2750 3600 2600
 $Comp
-L Connector_Generic:Conn_02x12_Counter_Clockwise J?
+L Connector_Generic:Conn_02x12_Counter_Clockwise J1601
 U 1 1 611D66DC
 P 5100 3550
-F 0 "J?" H 5150 4267 50  0000 C CNN
+F 0 "J1601" H 5150 4267 50  0000 C CNN
 F 1 "ClockSelector" H 5150 4176 50  0000 C CNN
 F 2 "" H 5100 3550 50  0001 C CNN
@@
 NoConn ~ 11050 1300
 $Comp
-L 74xx:74HC04 U?
+L 74xx:74HC04 U1601
 U 4 1 611C52D2
 P 10750 1300
-F 0 "U?" H 10750 1617 50  0000 C CNN
+F 0 "U1601" H 10750 1617 50  0000 C CNN
 F 1 "74HC04" H 10750 1526 50  0000 C CNN
 F 2 "" H 10750 1300 50  0001 C CNN
@@
 	10300 1300 10300 1750
 $Comp
-L power:GND #PWR?
+L power:GND #PWR01610
 U 1 1 611ECC77
 P 10300 2350
-F 0 "#PWR?" H 10300 2100 50  0001 C CNN
+F 0 "#PWR01610" H 10300 2100 50  0001 C CNN
 F 1 "GND" H 10305 2177 50  0000 C CNN
 F 2 "" H 10300 2350 50  0001 C CNN
@@
 Connection ~ 10300 2200
 $Comp
-L 74xx:74HC14 U?
+L 74xx:74HC14 U1502
 U 1 1 611FAED5
 P 6400 3600
-F 0 "U?" H 6400 3917 50  0000 C CNN
+F 0 "U1502" H 6400 3917 50  0000 C CNN
 F 1 "74HC14" H 6400 3826 50  0000 C CNN
 F 2 "" H 6400 3600 50  0001 C CNN
@@
 	5500 3600 5500 3650
 $Comp
-L 74xx:74HC14 U?
+L 74xx:74HC14 U1502
 U 2 1 611FFB13
 P 7600 3600
-F 0 "U?" H 7600 3917 50  0000 C CNN
+F 0 "U1502" H 7600 3917 50  0000 C CNN
 F 1 "74HC14" H 7600 3826 50  0000 C CNN
 F 2 "" H 7600 3600 50  0001 C CNN
@@
 $EndComp
 $Comp
-L 74xx:74HC14 U?
+L 74xx:74HC14 U1502
 U 3 1 612064EB
 P 8650 3600
-F 0 "U?" H 8650 3917 50  0000 C CNN
+F 0 "U1502" H 8650 3917 50  0000 C CNN
 F 1 "74HC14" H 8650 3826 50  0000 C CNN
 F 2 "" H 8650 3600 50  0001 C CNN
@@
 $EndComp
 $Comp
-L 74xx:74HC14 U?
+L 74xx:74HC14 U1502
 U 4 1 6120A909
 P 8650 4200
-F 0 "U?" H 8650 4517 50  0000 C CNN
+F 0 "U1502" H 8650 4517 50  0000 C CNN
 F 1 "74HC14" H 8650 4426 50  0000 C CNN
 F 2 "" H 8650 4200 50  0001 C CNN
@@
 $EndComp
 $Comp
-L 74xx:74HC14 U?
+L 74xx:74HC14 U1502
 U 5 1 6120B129
 P 8650 4750
-F 0 "U?" H 8650 5067 50  0000 C CNN
+F 0 "U1502" H 8650 5067 50  0000 C CNN
 F 1 "74HC14" H 8650 4976 50  0000 C CNN
 F 2 "" H 8650 4750 50  0001 C CNN
@@
 $EndComp
 $Comp
-L 74xx:74HC14 U?
+L 74xx:74HC14 U1502
 U 7 1 6120D4F6
 P 2700 6850
-F 0 "U?" H 2930 6896 50  0000 L CNN
+F 0 "U1502" H 2930 6896 50  0000 L CNN
 F 1 "74HC14" H 2930 6805 50  0000 L CNN
 F 2 "" H 2700 6850 50  0001 C CNN
@@
 $EndComp
 $Comp
-L Device:R R?
+L Device:R R1603
 U 1 1 6120EDAB
 P 7000 3600
-F 0 "R?" V 6793 3600 50  0000 C CNN
+F 0 "R1603" V 6793 3600 50  0000 C CNN
 F 1 "1k5" V 6884 3600 50  0000 C CNN
 F 2 "" V 6930 3600 50  0001 C CNN
@@
 	8950 4750 9300 4750
 $Comp
-L Device:C C?
+L Device:C C1603
 U 1 1 6123036E
 P 3900 6850
-F 0 "C?" H 3950 6950 50  0000 L CNN
+F 0 "C1603" H 3950 6950 50  0000 L CNN
 F 1 "100nF" H 3950 6750 50  0000 L CNN
 F 2 "" H 3938 6700 50  0001 C CNN
@@
 $EndComp
 $Comp
-L Device:C C?
+L Device:C C1604
 U 1 1 61230A4E
 P 4200 6850
-F 0 "C?" H 4250 6950 50  0000 L CNN
+F 0 "C1604" H 4250 6950 50  0000 L CNN
 F 1 "100nF" H 4250 6750 50  0000 L CNN
 F 2 "" H 4238 6700 50  0001 C CNN
@@
 $EndComp
 $Comp
-L Device:C C?
+L Device:C C1605
 U 1 1 61230C97
 P 4500 6850
-F 0 "C?" H 4550 6950 50  0000 L CNN
+F 0 "C1605" H 4550 6950 50  0000 L CNN
 F 1 "100nF" H 4550 6750 50  0000 L CNN
 F 2 "" H 4538 6700 50  0001 C CNN
@@
 	2700 7450 2700 7350
 $Comp
-L power:GND #PWR?
+L power:GND #PWR01604
 U 1 1 6124AD0E
 P 2450 7450
-F 0 "#PWR?" H 2450 7200 50  0001 C CNN
+F 0 "#PWR01604" H 2450 7200 50  0001 C CNN
 F 1 "GND" H 2455 7277 50  0000 C CNN
 F 2 "" H 2450 7450 50  0001 C CNN
@@
 	2450 7450 2700 7450
 $Comp
-L power:GND #PWR?
+L power:GND #PWR01609
 U 1 1 6124B56D
 P 4200 7100
-F 0 "#PWR?" H 4200 6850 50  0001 C CNN
+F 0 "#PWR01609" H 4200 6850 50  0001 C CNN
 F 1 "GND" H 4205 6927 50  0000 C CNN
 F 2 "" H 4200 7100 50  0001 C CNN
@@
 $EndComp
 $Comp
-L power:VCC #PWR?
+L power:VCC #PWR01608
 U 1 1 6124BDDA
 P 4200 6600
-F 0 "#PWR?" H 4200 6450 50  0001 C CNN
+F 0 "#PWR01608" H 4200 6450 50  0001 C CNN
 F 1 "VCC" H 4215 6773 50  0000 C CNN
 F 2 "" H 4200 6600 50  0001 C CNN
@@
 $EndComp
 $Comp
-L power:VCC #PWR?
+L power:VCC #PWR01603
 U 1 1 6124C6AC
 P 2450 6250
-F 0 "#PWR?" H 2450 6100 50  0001 C CNN
+F 0 "#PWR01603" H 2450 6100 50  0001 C CNN
 F 1 "VCC" H 2465 6423 50  0000 C CNN
 F 2 "" H 2450 6250 50  0001 C CNN

Commit message: Correcting ERC issues
Parts:
- removed unit 3 of U1601
- removed unit 4 of U1601
- removed unit 5 of U1601
- removed unit 6 of U1601
Connections:
- net EntRlg: now also R1603.2, U1502.2
- no-connect marks 4 -> 0
Changed lines of the file:
@@
 $Descr A4 11693 8268
 encoding utf-8
-Sheet 15 17
+Sheet 16 18
 Title ""
 Date ""
@@
 $Comp
 L 74xx:74HC04 U1601
-U 3 1 611C4F48
-P 10750 850
-F 0 "U1601" H 10750 1167 50  0000 C CNN
-F 1 "74HC04" H 10750 1076 50  0000 C CNN
-F 2 "" H 10750 850 50  0001 C CNN
-F 3 "https://assets.nexperia.com/documents/data-sheet/74HC_HCT04.pdf" H 10750 850 50  0001 C CNN
-	3    10750 850
-	1    0    0    -1
-$EndComp
-$Comp
-L 74xx:74HC04 U1601
-U 5 1 611C5E55
-P 10750 1750
-F 0 "U1601" H 10750 2067 50  0000 C CNN
-F 1 "74HC04" H 10750 1976 50  0000 C CNN
-F 2 "" H 10750 1750 50  0001 C CNN
-F 3 "https://assets.nexperia.com/documents/data-sheet/74HC_HCT04.pdf" H 10750 1750 50  0001 C CNN
-	5    10750 1750
-	1    0    0    -1
-$EndComp
-$Comp
-L 74xx:74HC04 U1601
-U 6 1 611C6A1E
-P 10750 2200
-F 0 "U1601" H 10750 2517 50  0000 C CNN
-F 1 "74HC04" H 10750 2426 50  0000 C CNN
-F 2 "" H 10750 2200 50  0001 C CNN
-F 3 "https://assets.nexperia.com/documents/data-sheet/74HC_HCT04.pdf" H 10750 2200 50  0001 C CNN
-	6    10750 2200
-	1    0    0    -1
-$EndComp
-$Comp
-L 74xx:74HC04 U1601
 U 7 1 611C732B
 P 2200 6850
@@
 Wire Wire Line
 	5500 3150 5500 3250
-NoConn ~ 11050 850
-NoConn ~ 11050 1750
-NoConn ~ 11050 2200
-NoConn ~ 11050 1300
-$Comp
-L 74xx:74HC04 U1601
-U 4 1 611C52D2
-P 10750 1300
-F 0 "U1601" H 10750 1617 50  0000 C CNN
-F 1 "74HC04" H 10750 1526 50  0000 C CNN
-F 2 "" H 10750 1300 50  0001 C CNN
-F 3 "https://assets.nexperia.com/documents/data-sheet/74HC_HCT04.pdf" H 10750 1300 50  0001 C CNN
-	4    10750 1300
-	1    0    0    -1
-$EndComp
-Wire Wire Line
-	10450 850  10300 850
-Wire Wire Line
-	10300 850  10300 1300
-Wire Wire Line
-	10300 2200 10450 2200
-Wire Wire Line
-	10450 1750 10300 1750
-Connection ~ 10300 1750
-Wire Wire Line
-	10300 1750 10300 2200
-Wire Wire Line
-	10450 1300 10300 1300
-Connection ~ 10300 1300
-Wire Wire Line
-	10300 1300 10300 1750
-$Comp
-L power:GND #PWR01610
-U 1 1 611ECC77
-P 10300 2350
-F 0 "#PWR01610" H 10300 2100 50  0001 C CNN
-F 1 "GND" H 10305 2177 50  0000 C CNN
-F 2 "" H 10300 2350 50  0001 C CNN
-F 3 "" H 10300 2350 50  0001 C CNN
-	1    10300 2350
-	1    0    0    -1
-$EndComp
-Wire Wire Line
-	10300 2200 10300 2350
-Connection ~ 10300 2200
 $Comp
 L 74xx:74HC14 U1502
@@
 $EndComp
 Wire Wire Line
-	6700 3600 6850 3600
+	6700 3600 6750 3600
 Wire Wire Line
 	7150 3600 7300 3600
@@
 Wire Wire Line
 	2450 6250 2200 6250
+Connection ~ 6750 3600
+Wire Wire Line
+	6750 3600 6850 3600
 $EndSCHEMATC

Commit message: Assigning footprints and generating netlist
Parts:
- C1601, C1602, C1603, C1604, C1605: footprint (none) -> Capacitor_THT:CP_Radial_D5.0mm_P2.50mm
- J1601: footprint (none) -> Connector_PinHeader_2.54mm:PinHeader_2x12_P2.54mm_Vertical
- R1601, R1602, R1603: footprint (none) -> Resistor_THT:R_Axial_DIN0204_L3.6mm_D1.6mm_P1.90mm_Vertical
- U1502, U1601: footprint (none) -> Package_DIP:DIP-14_W7.62mm
- U1602: footprint (none) -> Package_DIP:DIP-16_W7.62mm
- Y1601: footprint (none) -> Crystal:Crystal_HC33-U_Vertical
Changed lines of the file:
@@
 F 0 "U1602" H 3850 4200 50  0000 C CNN
 F 1 "74HC4040" H 3350 4200 50  0000 C CNN
-F 2 "" H 4800 4700 50  0001 C CNN
+F 2 "Package_DIP:DIP-16_W7.62mm" H 4800 4700 50  0001 C CNN
 F 3 "" H 4800 4700 50  0001 C CNN
 	1    3600 3550
@@
 F 0 "U1601" H 1150 3767 50  0000 C CNN
 F 1 "74HC04" H 1150 3676 50  0000 C CNN
-F 2 "" H 1150 3450 50  0001 C CNN
+F 2 "Package_DIP:DIP-14_W7.62mm" H 1150 3450 50  0001 C CNN
 F 3 "https://assets.nexperia.com/documents/data-sheet/74HC_HCT04.pdf" H 1150 3450 50  0001 C CNN
 	1    1150 3450
@@
 F 0 "U1601" H 2200 3767 50  0000 C CNN
 F 1 "74HC04" H 2200 3676 50  0000 C CNN
-F 2 "" H 2200 3450 50  0001 C CNN
+F 2 "Package_DIP:DIP-14_W7.62mm" H 2200 3450 50  0001 C CNN
 F 3 "https://assets.nexperia.com/documents/data-sheet/74HC_HCT04.pdf" H 2200 3450 50  0001 C CNN
 	2    2200 3450
@@
 F 0 "U1601" H 1800 6900 50  0000 L CNN
 F 1 "74HC04" H 1700 6750 50  0000 L CNN
-F 2 "" H 2200 6850 50  0001 C CNN
+F 2 "Package_DIP:DIP-14_W7.62mm" H 2200 6850 50  0001 C CNN
 F 3 "https://assets.nexperia.com/documents/data-sheet/74HC_HCT04.pdf" H 2200 6850 50  0001 C CNN
 	7    2200 6850
@@
 F 0 "R1601" V 943 2750 50  0000 C CNN
 F 1 "1M" V 1034 2750 50  0000 C CNN
-F 2 "" V 1080 2750 50  0001 C CNN
+F 2 "Resistor_THT:R_Axial_DIN0204_L3.6mm_D1.6mm_P1.90mm_Vertical" V 1080 2750 50  0001 C CNN
 F 3 "~" H 1150 2750 50  0001 C CNN
 	1    1150 2750
@@
 F 0 "R1602" H 1620 3846 50  0000 L CNN
 F 1 "470" H 1620 3755 50  0000 L CNN
-F 2 "" V 1480 3800 50  0001 C CNN
+F 2 "Resistor_THT:R_Axial_DIN0204_L3.6mm_D1.6mm_P1.90mm_Vertical" V 1480 3800 50  0001 C CNN
 F 3 "~" H 1550 3800 50  0001 C CNN
 	1    1550 3800
@@
 F 0 "Y1601" H 1150 4418 50  0000 C CNN
 F 1 "8MHz" H 1150 4327 50  0000 C CNN
-F 2 "" H 1150 4150 50  0001 C CNN
+F 2 "Crystal:Crystal_HC33-U_Vertical" H 1150 4150 50  0001 C CNN
 F 3 "~" H 1150 4150 50  0001 C CNN
 	1    1150 4150
@@
 F 0 "C1602" H 1665 4596 50  0000 L CNN
 F 1 "33pF" H 1665 4505 50  0000 L CNN
-F 2 "" H 1588 4400 50  0001 C CNN
+F 2 "Capacitor_THT:CP_Radial_D5.0mm_P2.50mm" H 1588 4400 50  0001 C CNN
 F 3 "~" H 1550 4550 50  0001 C CNN
 	1    1550 4550
@@
 F 0 "C1601" H 865 4596 50  0000 L CNN
 F 1 "33pF" H 865 4505 50  0000 L CNN
-F 2 "" H 788 4400 50  0001 C CNN
+F 2 "Capacitor_THT:CP_Radial_D5.0mm_P2.50mm" H 788 4400 50  0001 C CNN
 F 3 "~" H 750 4550 50  0001 C CNN
 	1    750  4550
@@
 F 0 "J1601" H 5150 4267 50  0000 C CNN
 F 1 "ClockSelector" H 5150 4176 50  0000 C CNN
-F 2 "" H 5100 3550 50  0001 C CNN
+F 2 "Connector_PinHeader_2.54mm:PinHeader_2x12_P2.54mm_Vertical" H 5100 3550 50  0001 C CNN
 F 3 "~" H 5100 3550 50  0001 C CNN
 	1    5100 3550
@@
 F 0 "U1502" H 6400 3917 50  0000 C CNN
 F 1 "74HC14" H 6400 3826 50  0000 C CNN
-F 2 "" H 6400 3600 50  0001 C CNN
+F 2 "Package_DIP:DIP-14_W7.62mm" H 6400 3600 50  0001 C CNN
 F 3 "http://www.ti.com/lit/gpn/sn74HC14" H 6400 3600 50  0001 C CNN
 	1    6400 3600
@@
 F 0 "U1502" H 7600 3917 50  0000 C CNN
 F 1 "74HC14" H 7600 3826 50  0000 C CNN
-F 2 "" H 7600 3600 50  0001 C CNN
+F 2 "Package_DIP:DIP-14_W7.62mm" H 7600 3600 50  0001 C CNN
 F 3 "http://www.ti.com/lit/gpn/sn74HC14" H 7600 3600 50  0001 C CNN
 	2    7600 3600
@@
 F 0 "U1502" H 8650 3917 50  0000 C CNN
 F 1 "74HC14" H 8650 3826 50  0000 C CNN
-F 2 "" H 8650 3600 50  0001 C CNN
+F 2 "Package_DIP:DIP-14_W7.62mm" H 8650 3600 50  0001 C CNN
 F 3 "http://www.ti.com/lit/gpn/sn74HC14" H 8650 3600 50  0001 C CNN
 	3    8650 3600
@@
 F 0 "U1502" H 8650 4517 50  0000 C CNN
 F 1 "74HC14" H 8650 4426 50  0000 C CNN
-F 2 "" H 8650 4200 50  0001 C CNN
+F 2 "Package_DIP:DIP-14_W7.62mm" H 8650 4200 50  0001 C CNN
 F 3 "http://www.ti.com/lit/gpn/sn74HC14" H 8650 4200 50  0001 C CNN
 	4    8650 4200
@@
 F 0 "U1502" H 8650 5067 50  0000 C CNN
 F 1 "74HC14" H 8650 4976 50  0000 C CNN
-F 2 "" H 8650 4750 50  0001 C CNN
+F 2 "Package_DIP:DIP-14_W7.62mm" H 8650 4750 50  0001 C CNN
 F 3 "http://www.ti.com/lit/gpn/sn74HC14" H 8650 4750 50  0001 C CNN
 	5    8650 4750
@@
 F 0 "U1502" H 2930 6896 50  0000 L CNN
 F 1 "74HC14" H 2930 6805 50  0000 L CNN
-F 2 "" H 2700 6850 50  0001 C CNN
+F 2 "Package_DIP:DIP-14_W7.62mm" H 2700 6850 50  0001 C CNN
 F 3 "http://www.ti.com/lit/gpn/sn74HC14" H 2700 6850 50  0001 C CNN
 	7    2700 6850
@@
 F 0 "R1603" V 6793 3600 50  0000 C CNN
 F 1 "1k5" V 6884 3600 50  0000 C CNN
-F 2 "" V 6930 3600 50  0001 C CNN
+F 2 "Resistor_THT:R_Axial_DIN0204_L3.6mm_D1.6mm_P1.90mm_Vertical" V 6930 3600 50  0001 C CNN
 F 3 "~" H 7000 3600 50  0001 C CNN
 	1    7000 3600
@@
 F 0 "C1603" H 3950 6950 50  0000 L CNN
 F 1 "100nF" H 3950 6750 50  0000 L CNN
-F 2 "" H 3938 6700 50  0001 C CNN
+F 2 "Capacitor_THT:CP_Radial_D5.0mm_P2.50mm" H 3938 6700 50  0001 C CNN
 F 3 "~" H 3900 6850 50  0001 C CNN
 	1    3900 6850
@@
 F 0 "C1604" H 4250 6950 50  0000 L CNN
 F 1 "100nF" H 4250 6750 50  0000 L CNN
-F 2 "" H 4238 6700 50  0001 C CNN
+F 2 "Capacitor_THT:CP_Radial_D5.0mm_P2.50mm" H 4238 6700 50  0001 C CNN
 F 3 "~" H 4200 6850 50  0001 C CNN
 	1    4200 6850
@@
 F 0 "C1605" H 4550 6950 50  0000 L CNN
 F 1 "100nF" H 4550 6750 50  0000 L CNN
-F 2 "" H 4538 6700 50  0001 C CNN
+F 2 "Capacitor_THT:CP_Radial_D5.0mm_P2.50mm" H 4538 6700 50  0001 C CNN
 F 3 "~" H 4500 6850 50  0001 C CNN
 	1    4500 6850

Commit message: Correcting footprints errors
Parts:
- C1601, C1602, C1603, C1604, C1605: footprint Capacitor_THT:CP_Radial_D5.0mm_P2.50mm -> Capacitor_THT:C_Disc_D4.3mm_W1.9mm_P5.00mm
- J1601: value ClockSelector -> Conn_02x12
- Y1601: footprint Crystal:Crystal_HC33-U_Vertical -> Crystal:Crystal_HC52-U_Vertical
Changed lines of the file:
@@
 U 7 1 611C732B
 P 2200 6850
-F 0 "U1601" H 1800 6900 50  0000 L CNN
-F 1 "74HC04" H 1700 6750 50  0000 L CNN
+F 0 "U1601" H 2050 6900 50  0000 L CNN
+F 1 "74HC04" H 2050 6800 50  0000 L CNN
 F 2 "Package_DIP:DIP-14_W7.62mm" H 2200 6850 50  0001 C CNN
 F 3 "https://assets.nexperia.com/documents/data-sheet/74HC_HCT04.pdf" H 2200 6850 50  0001 C CNN
@@
 F 0 "Y1601" H 1150 4418 50  0000 C CNN
 F 1 "8MHz" H 1150 4327 50  0000 C CNN
-F 2 "Crystal:Crystal_HC33-U_Vertical" H 1150 4150 50  0001 C CNN
+F 2 "Crystal:Crystal_HC52-U_Vertical" H 1150 4150 50  0001 C CNN
 F 3 "~" H 1150 4150 50  0001 C CNN
 	1    1150 4150
@@
 F 0 "C1602" H 1665 4596 50  0000 L CNN
 F 1 "33pF" H 1665 4505 50  0000 L CNN
-F 2 "Capacitor_THT:CP_Radial_D5.0mm_P2.50mm" H 1588 4400 50  0001 C CNN
+F 2 "Capacitor_THT:C_Disc_D4.3mm_W1.9mm_P5.00mm" H 1588 4400 50  0001 C CNN
 F 3 "~" H 1550 4550 50  0001 C CNN
 	1    1550 4550
@@
 F 0 "C1601" H 865 4596 50  0000 L CNN
 F 1 "33pF" H 865 4505 50  0000 L CNN
-F 2 "Capacitor_THT:CP_Radial_D5.0mm_P2.50mm" H 788 4400 50  0001 C CNN
+F 2 "Capacitor_THT:C_Disc_D4.3mm_W1.9mm_P5.00mm" H 788 4400 50  0001 C CNN
 F 3 "~" H 750 4550 50  0001 C CNN
 	1    750  4550
@@
 P 5100 3550
 F 0 "J1601" H 5150 4267 50  0000 C CNN
-F 1 "ClockSelector" H 5150 4176 50  0000 C CNN
+F 1 "Conn_02x12" H 5150 4176 50  0000 C CNN
 F 2 "Connector_PinHeader_2.54mm:PinHeader_2x12_P2.54mm_Vertical" H 5100 3550 50  0001 C CNN
 F 3 "~" H 5100 3550 50  0001 C CNN
@@
 U 7 1 6120D4F6
 P 2700 6850
-F 0 "U1502" H 2930 6896 50  0000 L CNN
-F 1 "74HC14" H 2930 6805 50  0000 L CNN
+F 0 "U1502" H 2550 6900 50  0000 L CNN
+F 1 "74HC14" H 2550 6800 50  0000 L CNN
 F 2 "Package_DIP:DIP-14_W7.62mm" H 2700 6850 50  0001 C CNN
 F 3 "http://www.ti.com/lit/gpn/sn74HC14" H 2700 6850 50  0001 C CNN
@@
 F 0 "C1603" H 3950 6950 50  0000 L CNN
 F 1 "100nF" H 3950 6750 50  0000 L CNN
-F 2 "Capacitor_THT:CP_Radial_D5.0mm_P2.50mm" H 3938 6700 50  0001 C CNN
+F 2 "Capacitor_THT:C_Disc_D4.3mm_W1.9mm_P5.00mm" H 3938 6700 50  0001 C CNN
 F 3 "~" H 3900 6850 50  0001 C CNN
 	1    3900 6850
@@
 F 0 "C1604" H 4250 6950 50  0000 L CNN
 F 1 "100nF" H 4250 6750 50  0000 L CNN
-F 2 "Capacitor_THT:CP_Radial_D5.0mm_P2.50mm" H 4238 6700 50  0001 C CNN
+F 2 "Capacitor_THT:C_Disc_D4.3mm_W1.9mm_P5.00mm" H 4238 6700 50  0001 C CNN
 F 3 "~" H 4200 6850 50  0001 C CNN
 	1    4200 6850
@@
 F 0 "C1605" H 4550 6950 50  0000 L CNN
 F 1 "100nF" H 4550 6750 50  0000 L CNN
-F 2 "Capacitor_THT:CP_Radial_D5.0mm_P2.50mm" H 4538 6700 50  0001 C CNN
+F 2 "Capacitor_THT:C_Disc_D4.3mm_W1.9mm_P5.00mm" H 4538 6700 50  0001 C CNN
 F 3 "~" H 4500 6850 50  0001 C CNN
 	1    4500 6850
