File: CES/ControlUnit.sch (KiCad schematic (older format))
At the start: 0 parts

Commit message: Control Unit
Parts:
- added C801, C802, C803, C804, C805, C806, C807, C808, C809: 100nF, symbol Device:C
- added U801: 74HC21, symbol CES:74HC21
- added U802, U808: 74HC20, symbol CES:74HC20
- added U803, U809: 74HC00, symbol 74xx:74HC00
- added U804, U807: 74HC02, symbol 74xx:74HC02
- added U805, U806: 74HC27, symbol CES:74HC27
Connections:
- new net: U808.4, U808.8
- new net BotEscMem: U803.10
- new net BotParteAtivo: U801.10, U804.11
- new net Desvia: U801.6, U806.4, U806.9, U808.13
- new net EntRlg: U809.4
- new net EscC: U803.12, U805.6
- new net Est1: U802.9, U803.1, U804.9
- new net GND: C801.2, C802.2, C803.2, C804.2, C805.2, C806.2, C807.2, C808.2, C809.2, U801.7 (GND), U802.7 (GND), U803.7 (GND), U804.12, U804.3, U804.7 (GND), U805.11, U805.7 (GND), U806.7 (GND), U807.12, U807.7 (GND), U808.7 (GND), U809.7 (GND)
- new net I0: U801.1, U802.1, U805.13, U805.3
- new net I1: U801.2, U802.12, U805.9
- new net MaisUm: U806.6
- new net MudaP: U807.2, U807.9
- new net MudaT: U807.5, U807.8
- new net Para: U801.12, U803.4, U803.9, U804.5, U804.8, U805.1, U805.4, U806.13, U806.3
- new net Parte: U806.10
- new net RC: U801.4
- new net RlgRC: U803.11
- new net RlgRI: U809.11
- new net VCC: C801.1, C802.1, C803.1, C804.1, C805.1, C806.1, C807.1, C808.1, C809.1, U801.14 (VCC), U802.14 (VCC), U803.14 (VCC), U804.14 (VCC), U805.14 (VCC), U806.14 (VCC), U807.14 (VCC), U808.10, U808.12, U808.14 (VCC), U808.9, U809.14 (VCC)
- new net VaiParar: U806.12
- new net VaiPartir: U801.8
- new net ZComp: U802.8
- new net nand2_1_a: U809.10, U809.3
- new net nand2_1_b: U809.6, U809.9
- new net nand2_2_a: U803.3, U808.2
- new net nor2_1_a: U804.1, U809.13
- new net nor2_1_b: U804.4, U806.11
- new net nor2_1_c: U804.10, U807.3
- new net nor3_1_b: U805.8, U806.5
- new net nor3_1_c: U805.12, U807.6
- new net ~BotEscMem: U809.2
- new net ~BotParteAtivo: U804.13
- new net ~EscM: U802.6, U809.1
- new net ~EscMem: U809.8
- new net ~EscP: U807.1
- new net ~EscT: U807.4
- new net ~Est1: U802.4, U804.6, U805.10, U805.2
- new net ~I0: U802.10
- new net ~I1: U802.2, U805.5
- new net ~IntPara: U806.2
- new net ~Para: U801.5, U802.13, U802.5, U803.2
- new net ~Parte: U801.13, U803.5, U808.5
- new net ~Partiu: U801.9
- new net ~Rlg: U803.13, U809.12, U809.5
- new net ~SaiBD: U803.8
- new net ~SaiBE: U803.6, U807.11
- new net ~SaiBS: U807.10, U808.1
- new net ~SaiRE: U807.13
- new net ~SaiRP: U808.6
- new net ~UltC: U804.2, U806.1, U806.8

Commit message: Assigning footprints and generating netlist
Parts:
- C801, C802, C803, C804, C805, C806, C807, C808, C809: footprint (none) -> Capacitor_THT:CP_Radial_D5.0mm_P2.50mm
- U801, U802, U808: footprint (none) -> Package_DIP:DIP-12_W7.62mm
- U803, U804, U805, U806, U807, U809: footprint (none) -> Package_DIP:DIP-14_W7.62mm

Commit message: Correcting footprints errors
Parts:
- C801, C802, C803, C804, C805, C806, C807, C808, C809: footprint Capacitor_THT:CP_Radial_D5.0mm_P2.50mm -> Capacitor_THT:C_Disc_D4.3mm_W1.9mm_P5.00mm
- U801, U802, U808: footprint Package_DIP:DIP-12_W7.62mm -> Package_DIP:DIP-14_W7.62mm
Changed lines of the file:
@@
 F 0 "U801" H 2050 1150 50  0000 C CNN
 F 1 "74HC21" H 2050 900 50  0000 C CNN
-F 2 "Package_DIP:DIP-12_W7.62mm" H 2050 900 50  0001 C CNN
+F 2 "Package_DIP:DIP-14_W7.62mm" H 2050 900 50  0001 C CNN
 F 3 "http://www.ti.com/lit/gpn/sn74HC21" H 2050 900 50  0001 C CNN
 	1    2050 900
@@
 F 0 "U801" H 2050 1800 50  0000 C CNN
 F 1 "74HC21" H 2050 1550 50  0000 C CNN
-F 2 "Package_DIP:DIP-12_W7.62mm" H 2050 1550 50  0001 C CNN
+F 2 "Package_DIP:DIP-14_W7.62mm" H 2050 1550 50  0001 C CNN
 F 3 "http://www.ti.com/lit/gpn/sn74HC21" H 2050 1550 50  0001 C CNN
 	2    2050 1550
@@
 F 0 "U801" H 7100 7150 50  0000 L CNN
 F 1 "74HC21" H 6900 6800 50  0000 L CNN
-F 2 "Package_DIP:DIP-12_W7.62mm" H 7050 6800 50  0001 C CNN
+F 2 "Package_DIP:DIP-14_W7.62mm" H 7050 6800 50  0001 C CNN
 F 3 "http://www.ti.com/lit/gpn/sn74HC21" H 7050 6800 50  0001 C CNN
 	3    7050 6800
@@
 F 0 "U808" H 5900 3950 50  0000 C CNN
 F 1 "74HC20" H 5900 3700 50  0000 C CNN
-F 2 "Package_DIP:DIP-12_W7.62mm" H 5900 3700 50  0001 C CNN
+F 2 "Package_DIP:DIP-14_W7.62mm" H 5900 3700 50  0001 C CNN
 F 3 "http://www.ti.com/lit/gpn/sn74HC20" H 5900 3700 50  0001 C CNN
 	1    5900 3700
@@
 F 0 "U808" H 4700 3200 50  0000 C CNN
 F 1 "74HC20" H 4700 2950 50  0000 C CNN
-F 2 "Package_DIP:DIP-12_W7.62mm" H 4700 2950 50  0001 C CNN
+F 2 "Package_DIP:DIP-14_W7.62mm" H 4700 2950 50  0001 C CNN
 F 3 "http://www.ti.com/lit/gpn/sn74HC20" H 4700 2950 50  0001 C CNN
 	2    4700 2950
@@
 F 0 "U802" H 7100 6700 50  0000 L CNN
 F 1 "74HC20" H 6900 6350 50  0000 L CNN
-F 2 "Package_DIP:DIP-12_W7.62mm" H 7050 6350 50  0001 C CNN
+F 2 "Package_DIP:DIP-14_W7.62mm" H 7050 6350 50  0001 C CNN
 F 3 "http://www.ti.com/lit/gpn/sn74HC20" H 7050 6350 50  0001 C CNN
 	3    7050 6350
@@
 F 0 "U802" H 2050 2550 50  0000 C CNN
 F 1 "74HC20" H 2050 2300 50  0000 C CNN
-F 2 "Package_DIP:DIP-12_W7.62mm" H 2050 2300 50  0001 C CNN
+F 2 "Package_DIP:DIP-14_W7.62mm" H 2050 2300 50  0001 C CNN
 F 3 "http://www.ti.com/lit/gpn/sn74HC20" H 2050 2300 50  0001 C CNN
 	1    2050 2300
@@
 F 0 "U802" H 2050 3200 50  0000 C CNN
 F 1 "74HC20" H 2050 2950 50  0000 C CNN
-F 2 "Package_DIP:DIP-12_W7.62mm" H 2050 2950 50  0001 C CNN
+F 2 "Package_DIP:DIP-14_W7.62mm" H 2050 2950 50  0001 C CNN
 F 3 "http://www.ti.com/lit/gpn/sn74HC20" H 2050 2950 50  0001 C CNN
 	2    2050 2950
@@
 F 0 "U808" H 7150 9400 50  0000 L CNN
 F 1 "74HC20" H 6900 9050 50  0000 L CNN
-F 2 "Package_DIP:DIP-12_W7.62mm" H 7050 9050 50  0001 C CNN
+F 2 "Package_DIP:DIP-14_W7.62mm" H 7050 9050 50  0001 C CNN
 F 3 "http://www.ti.com/lit/gpn/sn74HC20" H 7050 9050 50  0001 C CNN
 	3    7050 9050
@@
 F 0 "C801" H 950 10500 50  0000 L CNN
 F 1 "100nF" H 900 10300 50  0000 L CNN
-F 2 "Capacitor_THT:CP_Radial_D5.0mm_P2.50mm" H 938 10250 50  0001 C CNN
+F 2 "Capacitor_THT:C_Disc_D4.3mm_W1.9mm_P5.00mm" H 938 10250 50  0001 C CNN
 F 3 "~" H 900 10400 50  0001 C CNN
 	1    900  10400
@@
 F 0 "C802" H 1200 10500 50  0000 L CNN
 F 1 "100nF" H 1150 10300 50  0000 L CNN
-F 2 "Capacitor_THT:CP_Radial_D5.0mm_P2.50mm" H 1188 10250 50  0001 C CNN
+F 2 "Capacitor_THT:C_Disc_D4.3mm_W1.9mm_P5.00mm" H 1188 10250 50  0001 C CNN
 F 3 "~" H 1150 10400 50  0001 C CNN
 	1    1150 10400
@@
 F 0 "C803" H 1450 10500 50  0000 L CNN
 F 1 "100nF" H 1400 10300 50  0000 L CNN
-F 2 "Capacitor_THT:CP_Radial_D5.0mm_P2.50mm" H 1438 10250 50  0001 C CNN
+F 2 "Capacitor_THT:C_Disc_D4.3mm_W1.9mm_P5.00mm" H 1438 10250 50  0001 C CNN
 F 3 "~" H 1400 10400 50  0001 C CNN
 	1    1400 10400
@@
 F 0 "C804" H 1700 10500 50  0000 L CNN
 F 1 "100nF" H 1650 10300 50  0000 L CNN
-F 2 "Capacitor_THT:CP_Radial_D5.0mm_P2.50mm" H 1688 10250 50  0001 C CNN
+F 2 "Capacitor_THT:C_Disc_D4.3mm_W1.9mm_P5.00mm" H 1688 10250 50  0001 C CNN
 F 3 "~" H 1650 10400 50  0001 C CNN
 	1    1650 10400
@@
 F 0 "C805" H 1950 10500 50  0000 L CNN
 F 1 "100nF" H 1900 10300 50  0000 L CNN
-F 2 "Capacitor_THT:CP_Radial_D5.0mm_P2.50mm" H 1938 10250 50  0001 C CNN
+F 2 "Capacitor_THT:C_Disc_D4.3mm_W1.9mm_P5.00mm" H 1938 10250 50  0001 C CNN
 F 3 "~" H 1900 10400 50  0001 C CNN
 	1    1900 10400
@@
 F 0 "C806" H 2200 10500 50  0000 L CNN
 F 1 "100nF" H 2150 10300 50  0000 L CNN
-F 2 "Capacitor_THT:CP_Radial_D5.0mm_P2.50mm" H 2188 10250 50  0001 C CNN
+F 2 "Capacitor_THT:C_Disc_D4.3mm_W1.9mm_P5.00mm" H 2188 10250 50  0001 C CNN
 F 3 "~" H 2150 10400 50  0001 C CNN
 	1    2150 10400
@@
 F 0 "C807" H 2450 10500 50  0000 L CNN
 F 1 "100nF" H 2400 10300 50  0000 L CNN
-F 2 "Capacitor_THT:CP_Radial_D5.0mm_P2.50mm" H 2438 10250 50  0001 C CNN
+F 2 "Capacitor_THT:C_Disc_D4.3mm_W1.9mm_P5.00mm" H 2438 10250 50  0001 C CNN
 F 3 "~" H 2400 10400 50  0001 C CNN
 	1    2400 10400
@@
 F 0 "C808" H 2700 10500 50  0000 L CNN
 F 1 "100nF" H 2650 10300 50  0000 L CNN
-F 2 "Capacitor_THT:CP_Radial_D5.0mm_P2.50mm" H 2688 10250 50  0001 C CNN
+F 2 "Capacitor_THT:C_Disc_D4.3mm_W1.9mm_P5.00mm" H 2688 10250 50  0001 C CNN
 F 3 "~" H 2650 10400 50  0001 C CNN
 	1    2650 10400
@@
 F 0 "C809" H 2950 10500 50  0000 L CNN
 F 1 "100nF" H 2900 10300 50  0000 L CNN
-F 2 "Capacitor_THT:CP_Radial_D5.0mm_P2.50mm" H 2938 10250 50  0001 C CNN
+F 2 "Capacitor_THT:C_Disc_D4.3mm_W1.9mm_P5.00mm" H 2938 10250 50  0001 C CNN
 F 3 "~" H 2900 10400 50  0001 C CNN
 	1    2900 10400
