File: CES/FlipFlops.sch (KiCad schematic (older format))
At the start: 13 parts, among them U901 RC, U902 Est, U903 RS:Parte, U904 74HC112, U905 74HC74, U906 74HC74, U907 RI0, U908 Para, U909 Partiu

Commit message: Correcting ERC issues
Connections:
- net I0: no longer U907.9 (Q)
- net ~I0: no longer U907.8 (~Q)
- net Partiu: no longer names the net of U909.9 (Q)
- new net I1: U907.9 (Q)
- new net ~I1: U907.8 (~Q)
- no-connect marks 2 -> 3
Changed lines of the file:
@@
 $Descr A4 11693 8268
 encoding utf-8
-Sheet 9 17
+Sheet 9 18
 Title ""
 Date ""
@@
 	6000 2750 6650 2750
 Text GLabel 6650 2550 2    50   Output ~ 0
-I0
+I1
 Text GLabel 6650 2750 2    50   Output ~ 0
-~I0
+~I1
 Wire Wire Line
 	7900 1250 8150 1250
@@
 Text GLabel 9900 2750 2    50   Output ~ 0
 ~Partiu
-Text GLabel 9900 2550 2    50   Output ~ 0
-Partiu
-Wire Wire Line
-	9250 2550 9900 2550
 Wire Wire Line
 	9250 2750 9900 2750
@@
 Wire Wire Line
 	3050 4650 3500 4650
+NoConn ~ 9250 2550
 $EndSCHEMATC

Commit message: Assigning footprints and generating netlist
Parts:
- C901, C902, C903, C904: footprint (none) -> Capacitor_THT:CP_Radial_D5.0mm_P2.50mm
- U901, U902, U905, U906, U907: footprint (none) -> Package_DIP:DIP-14_W7.62mm
- U903, U904, U908, U909: footprint (none) -> Package_DIP:DIP-16_W7.62mm
Changed lines of the file:
@@
 F 0 "U901" H 2650 1500 50  0000 C CNN
 F 1 "RC" H 2550 1250 50  0000 C CNN
-F 2 "" H 2550 1250 50  0001 C CNN
+F 2 "Package_DIP:DIP-14_W7.62mm" H 2550 1250 50  0001 C CNN
 F 3 "74xx/74hc_hct74.pdf" H 2550 1250 50  0001 C CNN
 	1    2550 1250
@@
 F 0 "U902" H 2700 2900 50  0000 C CNN
 F 1 "Est" H 2550 2650 50  0000 C CNN
-F 2 "" H 2550 2650 50  0001 C CNN
+F 2 "Package_DIP:DIP-14_W7.62mm" H 2550 2650 50  0001 C CNN
 F 3 "74xx/74hc_hct74.pdf" H 2550 2650 50  0001 C CNN
 	2    2550 2650
@@
 F 0 "U907" H 5850 1500 50  0000 C CNN
 F 1 "RI0" H 5700 1250 50  0000 C CNN
-F 2 "" H 5700 1250 50  0001 C CNN
+F 2 "Package_DIP:DIP-14_W7.62mm" H 5700 1250 50  0001 C CNN
 F 3 "74xx/74hc_hct74.pdf" H 5700 1250 50  0001 C CNN
 	1    5700 1250
@@
 F 0 "U907" H 5850 2900 50  0000 C CNN
 F 1 "RI0" H 5700 2650 50  0000 C CNN
-F 2 "" H 5700 2650 50  0001 C CNN
+F 2 "Package_DIP:DIP-14_W7.62mm" H 5700 2650 50  0001 C CNN
 F 3 "74xx/74hc_hct74.pdf" H 5700 2650 50  0001 C CNN
 	2    5700 2650
@@
 F 0 "U903" H 2750 4950 50  0000 C CNN
 F 1 "RS:Parte" H 2250 4950 50  0000 C CNN
-F 2 "" H 2550 4350 50  0001 C CNN
+F 2 "Package_DIP:DIP-16_W7.62mm" H 2550 4350 50  0001 C CNN
 F 3 "http://www.ti.com/lit/gpn/sn74HC175" H 2550 4350 50  0001 C CNN
 	1    2550 4350
@@
 F 0 "U908" H 9100 1500 50  0000 C CNN
 F 1 "Para" H 8950 1250 50  0000 C CNN
-F 2 "" H 8950 1250 50  0001 C CNN
+F 2 "Package_DIP:DIP-16_W7.62mm" H 8950 1250 50  0001 C CNN
 F 3 "http://www.ti.com/lit/gpn/sn74HC112" H 8950 1250 50  0001 C CNN
 	1    8950 1250
@@
 F 0 "U909" H 9100 2900 50  0000 C CNN
 F 1 "Partiu" H 9000 2650 50  0000 C CNN
-F 2 "" H 8950 2650 50  0001 C CNN
+F 2 "Package_DIP:DIP-16_W7.62mm" H 8950 2650 50  0001 C CNN
 F 3 "http://www.ti.com/lit/gpn/sn74HC112" H 8950 2650 50  0001 C CNN
 	2    8950 2650
@@
 F 0 "U906" H 4650 7050 50  0000 L CNN
 F 1 "74HC74" H 4450 6700 50  0000 L CNN
-F 2 "" H 4600 6700 50  0001 C CNN
+F 2 "Package_DIP:DIP-14_W7.62mm" H 4600 6700 50  0001 C CNN
 F 3 "74xx/74hc_hct74.pdf" H 4600 6700 50  0001 C CNN
 	3    4600 6700
@@
 F 0 "U905" H 4150 7050 50  0000 L CNN
 F 1 "74HC74" H 3950 6700 50  0000 L CNN
-F 2 "" H 4100 6700 50  0001 C CNN
+F 2 "Package_DIP:DIP-14_W7.62mm" H 4100 6700 50  0001 C CNN
 F 3 "74xx/74hc_hct74.pdf" H 4100 6700 50  0001 C CNN
 	3    4100 6700
@@
 F 0 "U904" H 3650 7050 50  0000 L CNN
 F 1 "74HC112" H 3450 6700 50  0000 L CNN
-F 2 "" H 3600 6700 50  0001 C CNN
+F 2 "Package_DIP:DIP-16_W7.62mm" H 3600 6700 50  0001 C CNN
 F 3 "http://www.ti.com/lit/gpn/sn74HC112" H 3600 6700 50  0001 C CNN
 	3    3600 6700
@@
 F 0 "C901" H 5300 6800 50  0000 L CNN
 F 1 "100nF" H 5250 6600 50  0000 L CNN
-F 2 "" H 5288 6550 50  0001 C CNN
+F 2 "Capacitor_THT:CP_Radial_D5.0mm_P2.50mm" H 5288 6550 50  0001 C CNN
 F 3 "~" H 5250 6700 50  0001 C CNN
 	1    5250 6700
@@
 F 0 "C902" H 5550 6800 50  0000 L CNN
 F 1 "100nF" H 5500 6600 50  0000 L CNN
-F 2 "" H 5538 6550 50  0001 C CNN
+F 2 "Capacitor_THT:CP_Radial_D5.0mm_P2.50mm" H 5538 6550 50  0001 C CNN
 F 3 "~" H 5500 6700 50  0001 C CNN
 	1    5500 6700
@@
 F 0 "C903" H 5800 6800 50  0000 L CNN
 F 1 "100nF" H 5750 6600 50  0000 L CNN
-F 2 "" H 5788 6550 50  0001 C CNN
+F 2 "Capacitor_THT:CP_Radial_D5.0mm_P2.50mm" H 5788 6550 50  0001 C CNN
 F 3 "~" H 5750 6700 50  0001 C CNN
 	1    5750 6700
@@
 F 0 "C904" H 6050 6800 50  0000 L CNN
 F 1 "100nF" H 6000 6600 50  0000 L CNN
-F 2 "" H 6038 6550 50  0001 C CNN
+F 2 "Capacitor_THT:CP_Radial_D5.0mm_P2.50mm" H 6038 6550 50  0001 C CNN
 F 3 "~" H 6000 6700 50  0001 C CNN
 	1    6000 6700

Commit message: Correcting footprints errors
Parts:
- C901, C902, C903, C904: footprint Capacitor_THT:CP_Radial_D5.0mm_P2.50mm -> Capacitor_THT:C_Disc_D4.3mm_W1.9mm_P5.00mm
- U901: value RC -> 74HC74
- U901: renamed from U902; value Est -> 74HC74
- U902: renamed from U903; value RS:Parte -> 74HC175
- U903: renamed from U908; value Para -> 74HC112
- U903: renamed from U909; value Partiu -> 74HC112
- U904: renamed from U907; value RI0 -> 74HC74
- renumbered U905 to U901, U904 to U903, U906 to U904
Changed lines of the file:
@@
 AR Path="/60832B98/60A53941" Ref="U?"  Part="1"
 AR Path="/60832B98/60A4DE72/60A53941" Ref="U901"  Part="1"
-F 0 "U901" H 2650 1500 50  0000 C CNN
-F 1 "RC" H 2550 1250 50  0000 C CNN
+F 0 "U901" H 2700 1500 50  0000 C CNN
+F 1 "74HC74" H 2300 1500 50  0000 C CNN
 F 2 "Package_DIP:DIP-14_W7.62mm" H 2550 1250 50  0001 C CNN
 F 3 "74xx/74hc_hct74.pdf" H 2550 1250 50  0001 C CNN
@@
 P 2550 2650
 AR Path="/60832B98/60A53947" Ref="U?"  Part="2"
-AR Path="/60832B98/60A4DE72/60A53947" Ref="U902"  Part="2"
-F 0 "U902" H 2700 2900 50  0000 C CNN
-F 1 "Est" H 2550 2650 50  0000 C CNN
+AR Path="/60832B98/60A4DE72/60A53947" Ref="U901"  Part="2"
+F 0 "U901" H 2700 2900 50  0000 C CNN
+F 1 "74HC74" H 2300 2900 50  0000 C CNN
 F 2 "Package_DIP:DIP-14_W7.62mm" H 2550 2650 50  0001 C CNN
 F 3 "74xx/74hc_hct74.pdf" H 2550 2650 50  0001 C CNN
@@
 P 5700 1250
 AR Path="/60832B98/60A5394D" Ref="U?"  Part="1"
-AR Path="/60832B98/60A4DE72/60A5394D" Ref="U907"  Part="1"
-F 0 "U907" H 5850 1500 50  0000 C CNN
-F 1 "RI0" H 5700 1250 50  0000 C CNN
+AR Path="/60832B98/60A4DE72/60A5394D" Ref="U904"  Part="1"
+F 0 "U904" H 5850 1500 50  0000 C CNN
+F 1 "74HC74" H 5450 1500 50  0000 C CNN
 F 2 "Package_DIP:DIP-14_W7.62mm" H 5700 1250 50  0001 C CNN
 F 3 "74xx/74hc_hct74.pdf" H 5700 1250 50  0001 C CNN
@@
 P 5700 2650
 AR Path="/60832B98/60A53953" Ref="U?"  Part="2"
-AR Path="/60832B98/60A4DE72/60A53953" Ref="U907"  Part="2"
-F 0 "U907" H 5850 2900 50  0000 C CNN
-F 1 "RI0" H 5700 2650 50  0000 C CNN
+AR Path="/60832B98/60A4DE72/60A53953" Ref="U904"  Part="2"
+F 0 "U904" H 5850 2900 50  0000 C CNN
+F 1 "74HC74" H 5450 2900 50  0000 C CNN
 F 2 "Package_DIP:DIP-14_W7.62mm" H 5700 2650 50  0001 C CNN
 F 3 "74xx/74hc_hct74.pdf" H 5700 2650 50  0001 C CNN
@@
 P 2550 4350
 AR Path="/60832B98/60A53959" Ref="U?"  Part="1"
-AR Path="/60832B98/60A4DE72/60A53959" Ref="U903"  Part="1"
-F 0 "U903" H 2750 4950 50  0000 C CNN
-F 1 "RS:Parte" H 2250 4950 50  0000 C CNN
+AR Path="/60832B98/60A4DE72/60A53959" Ref="U902"  Part="1"
+F 0 "U902" H 2750 4950 50  0000 C CNN
+F 1 "74HC175" H 2250 4950 50  0000 C CNN
 F 2 "Package_DIP:DIP-16_W7.62mm" H 2550 4350 50  0001 C CNN
 F 3 "http://www.ti.com/lit/gpn/sn74HC175" H 2550 4350 50  0001 C CNN
@@
 P 8950 1250
 AR Path="/60832B98/60A5395F" Ref="U?"  Part="1"
-AR Path="/60832B98/60A4DE72/60A5395F" Ref="U908"  Part="1"
-F 0 "U908" H 9100 1500 50  0000 C CNN
-F 1 "Para" H 8950 1250 50  0000 C CNN
+AR Path="/60832B98/60A4DE72/60A5395F" Ref="U903"  Part="1"
+F 0 "U903" H 9100 1500 50  0000 C CNN
+F 1 "74HC112" H 8700 1500 50  0000 C CNN
 F 2 "Package_DIP:DIP-16_W7.62mm" H 8950 1250 50  0001 C CNN
 F 3 "http://www.ti.com/lit/gpn/sn74HC112" H 8950 1250 50  0001 C CNN
@@
 P 8950 2650
 AR Path="/60832B98/60A53965" Ref="U?"  Part="2"
-AR Path="/60832B98/60A4DE72/60A53965" Ref="U909"  Part="2"
-F 0 "U909" H 9100 2900 50  0000 C CNN
-F 1 "Partiu" H 9000 2650 50  0000 C CNN
+AR Path="/60832B98/60A4DE72/60A53965" Ref="U903"  Part="2"
+F 0 "U903" H 9100 2900 50  0000 C CNN
+F 1 "74HC112" H 8700 2900 50  0000 C CNN
 F 2 "Package_DIP:DIP-16_W7.62mm" H 8950 2650 50  0001 C CNN
 F 3 "http://www.ti.com/lit/gpn/sn74HC112" H 8950 2650 50  0001 C CNN
@@
 P 4600 6700
 AR Path="/60832B98/60A59845" Ref="U?"  Part="3"
-AR Path="/60832B98/60A4DE72/60A59845" Ref="U906"  Part="3"
-F 0 "U906" H 4650 7050 50  0000 L CNN
+AR Path="/60832B98/60A4DE72/60A59845" Ref="U904"  Part="3"
+F 0 "U904" H 4650 7050 50  0000 L CNN
 F 1 "74HC74" H 4450 6700 50  0000 L CNN
 F 2 "Package_DIP:DIP-14_W7.62mm" H 4600 6700 50  0001 C CNN
@@
 P 4100 6700
 AR Path="/60832B98/60A5984B" Ref="U?"  Part="3"
-AR Path="/60832B98/60A4DE72/60A5984B" Ref="U905"  Part="3"
-F 0 "U905" H 4150 7050 50  0000 L CNN
+AR Path="/60832B98/60A4DE72/60A5984B" Ref="U901"  Part="3"
+F 0 "U901" H 4150 7050 50  0000 L CNN
 F 1 "74HC74" H 3950 6700 50  0000 L CNN
 F 2 "Package_DIP:DIP-14_W7.62mm" H 4100 6700 50  0001 C CNN
@@
 P 3600 6700
 AR Path="/60832B98/60A59851" Ref="U?"  Part="3"
-AR Path="/60832B98/60A4DE72/60A59851" Ref="U904"  Part="3"
-F 0 "U904" H 3650 7050 50  0000 L CNN
+AR Path="/60832B98/60A4DE72/60A59851" Ref="U903"  Part="3"
+F 0 "U903" H 3650 7050 50  0000 L CNN
 F 1 "74HC112" H 3450 6700 50  0000 L CNN
 F 2 "Package_DIP:DIP-16_W7.62mm" H 3600 6700 50  0001 C CNN
@@
 F 0 "C901" H 5300 6800 50  0000 L CNN
 F 1 "100nF" H 5250 6600 50  0000 L CNN
-F 2 "Capacitor_THT:CP_Radial_D5.0mm_P2.50mm" H 5288 6550 50  0001 C CNN
+F 2 "Capacitor_THT:C_Disc_D4.3mm_W1.9mm_P5.00mm" H 5288 6550 50  0001 C CNN
 F 3 "~" H 5250 6700 50  0001 C CNN
 	1    5250 6700
@@
 F 0 "C902" H 5550 6800 50  0000 L CNN
 F 1 "100nF" H 5500 6600 50  0000 L CNN
-F 2 "Capacitor_THT:CP_Radial_D5.0mm_P2.50mm" H 5538 6550 50  0001 C CNN
+F 2 "Capacitor_THT:C_Disc_D4.3mm_W1.9mm_P5.00mm" H 5538 6550 50  0001 C CNN
 F 3 "~" H 5500 6700 50  0001 C CNN
 	1    5500 6700
@@
 F 0 "C903" H 5800 6800 50  0000 L CNN
 F 1 "100nF" H 5750 6600 50  0000 L CNN
-F 2 "Capacitor_THT:CP_Radial_D5.0mm_P2.50mm" H 5788 6550 50  0001 C CNN
+F 2 "Capacitor_THT:C_Disc_D4.3mm_W1.9mm_P5.00mm" H 5788 6550 50  0001 C CNN
 F 3 "~" H 5750 6700 50  0001 C CNN
 	1    5750 6700
@@
 F 0 "C904" H 6050 6800 50  0000 L CNN
 F 1 "100nF" H 6000 6600 50  0000 L CNN
-F 2 "Capacitor_THT:CP_Radial_D5.0mm_P2.50mm" H 6038 6550 50  0001 C CNN
+F 2 "Capacitor_THT:C_Disc_D4.3mm_W1.9mm_P5.00mm" H 6038 6550 50  0001 C CNN
 F 3 "~" H 6000 6700 50  0001 C CNN
 	1    6000 6700
