File: CES/PanelSwitchesBuffers.sch (KiCad schematic (older format))
At the start: 14 parts

Commit message: Control Unit
Parts:
- gave numbers to parts that had none: 14
Changed lines of the file:
@@
 $Descr A4 8268 11693 portrait
 encoding utf-8
-Sheet 13 16
+Sheet 13 17
 Title "CES"
 Date "2021-04-24"
@@
 P 2400 8300
 AR Path="/60832DB9/60D2B9E0" Ref="#PWR?"  Part="1"
-AR Path="/60832DB9/60C5807D/60D2B9E0" Ref="#PWR?"  Part="1"
-F 0 "#PWR?" H 2400 8050 50  0001 C CNN
+AR Path="/60832DB9/60C5807D/60D2B9E0" Ref="#PWR01410"  Part="1"
+F 0 "#PWR01410" H 2400 8050 50  0001 C CNN
 F 1 "GND" H 2400 8150 50  0000 C CNN
 F 2 "" H 2400 8300 50  0001 C CNN
@@
 P 2400 6700
 AR Path="/60832DB9/60D2B9E6" Ref="#PWR?"  Part="1"
-AR Path="/60832DB9/60C5807D/60D2B9E6" Ref="#PWR?"  Part="1"
-F 0 "#PWR?" H 2400 6550 50  0001 C CNN
+AR Path="/60832DB9/60C5807D/60D2B9E6" Ref="#PWR01409"  Part="1"
+F 0 "#PWR01409" H 2400 6550 50  0001 C CNN
 F 1 "VCC" H 2500 6800 50  0000 C CNN
 F 2 "" H 2400 6700 50  0001 C CNN
@@
 P 2400 2700
 AR Path="/60832DB9/60D2B9EE" Ref="#PWR?"  Part="1"
-AR Path="/60832DB9/60C5807D/60D2B9EE" Ref="#PWR?"  Part="1"
-F 0 "#PWR?" H 2400 2550 50  0001 C CNN
+AR Path="/60832DB9/60C5807D/60D2B9EE" Ref="#PWR01405"  Part="1"
+F 0 "#PWR01405" H 2400 2550 50  0001 C CNN
 F 1 "VCC" H 2500 2800 50  0000 C CNN
 F 2 "" H 2400 2700 50  0001 C CNN
@@
 P 2400 4300
 AR Path="/60832DB9/60D2B9F4" Ref="#PWR?"  Part="1"
-AR Path="/60832DB9/60C5807D/60D2B9F4" Ref="#PWR?"  Part="1"
-F 0 "#PWR?" H 2400 4050 50  0001 C CNN
+AR Path="/60832DB9/60C5807D/60D2B9F4" Ref="#PWR01406"  Part="1"
+F 0 "#PWR01406" H 2400 4050 50  0001 C CNN
 F 1 "GND" H 2500 4200 50  0000 C CNN
 F 2 "" H 2400 4300 50  0001 C CNN
@@
 AR Path="/60832B49/60D2B9FB" Ref="U?"  Part="1"
 AR Path="/60832DB9/60D2B9FB" Ref="U?"  Part="1"
-AR Path="/60832DB9/60C5807D/60D2B9FB" Ref="U?"  Part="1"
-F 0 "U?" H 2600 2200 50  0000 C CNN
+AR Path="/60832DB9/60C5807D/60D2B9FB" Ref="U1401"  Part="1"
+F 0 "U1401" H 2600 2200 50  0000 C CNN
 F 1 "BD1" H 2400 1350 50  0000 C CNN
 F 2 "" H 2400 1550 50  0001 C CNN
@@
 P 2400 7500
 AR Path="/60832DB9/60D2BA07" Ref="U?"  Part="1"
-AR Path="/60832DB9/60C5807D/60D2BA07" Ref="U?"  Part="1"
-F 0 "U?" H 2650 8150 50  0000 C CNN
+AR Path="/60832DB9/60C5807D/60D2BA07" Ref="U1404"  Part="1"
+F 0 "U1404" H 2650 8150 50  0000 C CNN
 F 1 "BS2" H 2400 7300 50  0000 C CNN
 F 2 "" H 2400 7500 50  0001 C CNN
@@
 P 700 4200
 AR Path="/60832DB9/60D2BA15" Ref="J?"  Part="1"
-AR Path="/60832DB9/60C5807D/60D2BA15" Ref="J?"  Part="1"
-F 0 "J?" H 800 3350 50  0000 R CNN
+AR Path="/60832DB9/60C5807D/60D2BA15" Ref="J1401"  Part="1"
+F 0 "J1401" H 800 3350 50  0000 R CNN
 F 1 "InputDataSwitches" V 650 4450 50  0000 R CNN
 F 2 "" H 700 4200 50  0001 C CNN
@@
 P 2400 3500
 AR Path="/60832DB9/60D2BA33" Ref="U?"  Part="1"
-AR Path="/60832DB9/60C5807D/60D2BA33" Ref="U?"  Part="1"
-F 0 "U?" H 2650 4150 50  0000 C CNN
+AR Path="/60832DB9/60C5807D/60D2BA33" Ref="U1402"  Part="1"
+F 0 "U1402" H 2650 4150 50  0000 C CNN
 F 1 "BS1" H 2400 3350 50  0000 C CNN
 F 2 "" H 2400 3500 50  0001 C CNN
@@
 P 2400 6300
 AR Path="/60832DB9/60D2BA49" Ref="#PWR?"  Part="1"
-AR Path="/60832DB9/60C5807D/60D2BA49" Ref="#PWR?"  Part="1"
-F 0 "#PWR?" H 2400 6050 50  0001 C CNN
+AR Path="/60832DB9/60C5807D/60D2BA49" Ref="#PWR01408"  Part="1"
+F 0 "#PWR01408" H 2400 6050 50  0001 C CNN
 F 1 "GND" H 2500 6200 50  0000 C CNN
 F 2 "" H 2400 6300 50  0001 C CNN
@@
 P 2400 2350
 AR Path="/60832DB9/60D2BA4F" Ref="#PWR?"  Part="1"
-AR Path="/60832DB9/60C5807D/60D2BA4F" Ref="#PWR?"  Part="1"
-F 0 "#PWR?" H 2400 2100 50  0001 C CNN
+AR Path="/60832DB9/60C5807D/60D2BA4F" Ref="#PWR01404"  Part="1"
+F 0 "#PWR01404" H 2400 2100 50  0001 C CNN
 F 1 "GND" H 2500 2250 50  0000 C CNN
 F 2 "" H 2400 2350 50  0001 C CNN
@@
 P 2400 4700
 AR Path="/60832DB9/60D2BA57" Ref="#PWR?"  Part="1"
-AR Path="/60832DB9/60C5807D/60D2BA57" Ref="#PWR?"  Part="1"
-F 0 "#PWR?" H 2400 4550 50  0001 C CNN
+AR Path="/60832DB9/60C5807D/60D2BA57" Ref="#PWR01407"  Part="1"
+F 0 "#PWR01407" H 2400 4550 50  0001 C CNN
 F 1 "VCC" H 2500 4800 50  0000 C CNN
 F 2 "" H 2400 4700 50  0001 C CNN
@@
 P 2400 750
 AR Path="/60832DB9/60D2BA5D" Ref="#PWR?"  Part="1"
-AR Path="/60832DB9/60C5807D/60D2BA5D" Ref="#PWR?"  Part="1"
-F 0 "#PWR?" H 2400 600 50  0001 C CNN
+AR Path="/60832DB9/60C5807D/60D2BA5D" Ref="#PWR01403"  Part="1"
+F 0 "#PWR01403" H 2400 600 50  0001 C CNN
 F 1 "VCC" H 2500 850 50  0000 C CNN
 F 2 "" H 2400 750 50  0001 C CNN
@@
 AR Path="/60832B49/60D2BA65" Ref="U?"  Part="1"
 AR Path="/60832DB9/60D2BA65" Ref="U?"  Part="1"
-AR Path="/60832DB9/60C5807D/60D2BA65" Ref="U?"  Part="1"
-F 0 "U?" H 2650 6150 50  0000 C CNN
+AR Path="/60832DB9/60C5807D/60D2BA65" Ref="U1403"  Part="1"
+F 0 "U1403" H 2650 6150 50  0000 C CNN
 F 1 "BD2" H 2400 5300 50  0000 C CNN
 F 2 "" H 2400 5500 50  0001 C CNN
@@
 P 3850 4300
 AR Path="/60832DB9/60F4E15C" Ref="J?"  Part="1"
-AR Path="/60832DB9/60C5807D/60F4E15C" Ref="J?"  Part="1"
-F 0 "J?" H 3950 3450 50  0000 R CNN
+AR Path="/60832DB9/60C5807D/60F4E15C" Ref="J1402"  Part="1"
+F 0 "J1402" H 3950 3450 50  0000 R CNN
 F 1 "InputAddressSwitches" V 3800 4550 50  0000 R CNN
 F 2 "" H 3850 4300 50  0001 C CNN
@@
 $EndComp
 $Comp
-L 74xx:74HC244 U?
+L 74xx:74HC244 U1405
 U 1 1 60F52B93
 P 5850 3500
-F 0 "U?" H 6100 4150 50  0000 C CNN
+F 0 "U1405" H 6100 4150 50  0000 C CNN
 F 1 "BE1" H 5850 3200 50  0000 C CNN
 F 2 "" H 5850 3500 50  0001 C CNN
@@
 $EndComp
 $Comp
-L 74xx:74HC244 U?
+L 74xx:74HC244 U1406
 U 1 1 60F55375
 P 5850 5500
-F 0 "U?" H 6100 6150 50  0000 C CNN
+F 0 "U1406" H 6100 6150 50  0000 C CNN
 F 1 "BE2" H 5850 5200 50  0000 C CNN
 F 2 "" H 5850 5500 50  0001 C CNN
@@
 $EndComp
 $Comp
-L power:GND #PWR?
+L power:GND #PWR01415
 U 1 1 60F57664
 P 5850 6300
-F 0 "#PWR?" H 5850 6050 50  0001 C CNN
+F 0 "#PWR01415" H 5850 6050 50  0001 C CNN
 F 1 "GND" H 5855 6127 50  0000 C CNN
 F 2 "" H 5850 6300 50  0001 C CNN
@@
 $EndComp
 $Comp
-L power:GND #PWR?
+L power:GND #PWR01413
 U 1 1 60F57C28
 P 5850 4300
-F 0 "#PWR?" H 5850 4050 50  0001 C CNN
+F 0 "#PWR01413" H 5850 4050 50  0001 C CNN
 F 1 "GND" H 5950 4200 50  0000 C CNN
 F 2 "" H 5850 4300 50  0001 C CNN
@@
 $EndComp
 $Comp
-L power:VCC #PWR?
+L power:VCC #PWR01414
 U 1 1 60F58150
 P 5850 4700
-F 0 "#PWR?" H 5850 4550 50  0001 C CNN
+F 0 "#PWR01414" H 5850 4550 50  0001 C CNN
 F 1 "VCC" H 5950 4800 50  0000 C CNN
 F 2 "" H 5850 4700 50  0001 C CNN
@@
 $EndComp
 $Comp
-L power:VCC #PWR?
+L power:VCC #PWR01412
 U 1 1 60F589E2
 P 5850 2700
-F 0 "#PWR?" H 5850 2550 50  0001 C CNN
+F 0 "#PWR01412" H 5850 2550 50  0001 C CNN
 F 1 "VCC" H 5865 2873 50  0000 C CNN
 F 2 "" H 5850 2700 50  0001 C CNN
@@
 NoConn ~ 6350 5600
 $Comp
-L power:GND #PWR?
+L power:GND #PWR01411
 U 1 1 60FFFD54
 P 5200 5750
-F 0 "#PWR?" H 5200 5500 50  0001 C CNN
+F 0 "#PWR01411" H 5200 5500 50  0001 C CNN
 F 1 "GND" H 5050 5650 50  0000 C CNN
 F 2 "" H 5200 5750 50  0001 C CNN
@@
 	1600 10050 1600 9900
 $Comp
-L Device:C C?
+L Device:C C1402
 U 1 1 61041364
 P 1600 10200
-F 0 "C?" H 1650 10300 50  0000 L CNN
+F 0 "C1402" H 1650 10300 50  0000 L CNN
 F 1 "100nF" H 1600 10100 50  0000 L CNN
 F 2 "" H 1638 10050 50  0001 C CNN
@@
 $EndComp
 $Comp
-L Device:C C?
+L Device:C C1401
 U 1 1 6104136A
 P 1350 10200
-F 0 "C?" H 1400 10300 50  0000 L CNN
+F 0 "C1401" H 1400 10300 50  0000 L CNN
 F 1 "100nF" H 1350 10100 50  0000 L CNN
 F 2 "" H 1388 10050 50  0001 C CNN
@@
 	2100 10050 2100 9900
 $Comp
-L Device:C C?
+L Device:C C1404
 U 1 1 6104DA51
 P 2100 10200
-F 0 "C?" H 2150 10300 50  0000 L CNN
+F 0 "C1404" H 2150 10300 50  0000 L CNN
 F 1 "100nF" H 2100 10100 50  0000 L CNN
 F 2 "" H 2138 10050 50  0001 C CNN
@@
 $EndComp
 $Comp
-L Device:C C?
+L Device:C C1403
 U 1 1 6104DA57
 P 1850 10200
-F 0 "C?" H 1900 10300 50  0000 L CNN
+F 0 "C1403" H 1900 10300 50  0000 L CNN
 F 1 "100nF" H 1850 10100 50  0000 L CNN
 F 2 "" H 1888 10050 50  0001 C CNN
@@
 $EndComp
 $Comp
-L power:VCC #PWR?
+L power:VCC #PWR01401
 U 1 1 6104DA5D
 P 1950 9900
-F 0 "#PWR?" H 1950 9750 50  0001 C CNN
+F 0 "#PWR01401" H 1950 9750 50  0001 C CNN
 F 1 "VCC" H 1965 10073 50  0000 C CNN
 F 2 "" H 1950 9900 50  0001 C CNN
@@
 	1950 9900 1850 9900
 $Comp
-L power:GND #PWR?
+L power:GND #PWR01402
 U 1 1 6104DA65
 P 1950 10500
-F 0 "#PWR?" H 1950 10250 50  0001 C CNN
+F 0 "#PWR01402" H 1950 10250 50  0001 C CNN
 F 1 "GND" H 1950 10350 50  0000 C CNN
 F 2 "" H 1950 10500 50  0001 C CNN
@@
 	2600 10050 2600 9900
 $Comp
-L Device:C C?
+L Device:C C1406
 U 1 1 6105BEA0
 P 2600 10200
-F 0 "C?" H 2650 10300 50  0000 L CNN
+F 0 "C1406" H 2650 10300 50  0000 L CNN
 F 1 "100nF" H 2600 10100 50  0000 L CNN
 F 2 "" H 2638 10050 50  0001 C CNN
@@
 $EndComp
 $Comp
-L Device:C C?
+L Device:C C1405
 U 1 1 6105BEA6
 P 2350 10200
-F 0 "C?" H 2400 10300 50  0000 L CNN
+F 0 "C1405" H 2400 10300 50  0000 L CNN
 F 1 "100nF" H 2350 10100 50  0000 L CNN
 F 2 "" H 2388 10050 50  0001 C CNN

Commit message: Assigning footprints and generating netlist
Parts:
- C1401, C1402, C1403, C1404, C1405, C1406: footprint (none) -> Capacitor_THT:CP_Radial_D5.0mm_P2.50mm
- J1401, J1402: footprint (none) -> Connector_PinHeader_2.54mm:PinHeader_1x16_P2.54mm_Vertical
- U1401, U1402, U1403, U1404, U1405, U1406: footprint (none) -> Package_DIP:DIP-20_W7.62mm
Changed lines of the file:
@@
 F 0 "U1401" H 2600 2200 50  0000 C CNN
 F 1 "BD1" H 2400 1350 50  0000 C CNN
-F 2 "" H 2400 1550 50  0001 C CNN
+F 2 "Package_DIP:DIP-20_W7.62mm" H 2400 1550 50  0001 C CNN
 F 3 "https://assets.nexperia.com/documents/data-sheet/74HC_HCT244.pdf" H 2400 1550 50  0001 C CNN
 	1    2400 1550
@@
 F 0 "U1404" H 2650 8150 50  0000 C CNN
 F 1 "BS2" H 2400 7300 50  0000 C CNN
-F 2 "" H 2400 7500 50  0001 C CNN
+F 2 "Package_DIP:DIP-20_W7.62mm" H 2400 7500 50  0001 C CNN
 F 3 "https://assets.nexperia.com/documents/data-sheet/74HC_HCT244.pdf" H 2400 7500 50  0001 C CNN
 	1    2400 7500
@@
 F 0 "J1401" H 800 3350 50  0000 R CNN
 F 1 "InputDataSwitches" V 650 4450 50  0000 R CNN
-F 2 "" H 700 4200 50  0001 C CNN
+F 2 "Connector_PinHeader_2.54mm:PinHeader_1x16_P2.54mm_Vertical" H 700 4200 50  0001 C CNN
 F 3 "~" H 700 4200 50  0001 C CNN
 	1    700  4200
@@
 F 0 "U1402" H 2650 4150 50  0000 C CNN
 F 1 "BS1" H 2400 3350 50  0000 C CNN
-F 2 "" H 2400 3500 50  0001 C CNN
+F 2 "Package_DIP:DIP-20_W7.62mm" H 2400 3500 50  0001 C CNN
 F 3 "https://assets.nexperia.com/documents/data-sheet/74HC_HCT244.pdf" H 2400 3500 50  0001 C CNN
 	1    2400 3500
@@
 F 0 "U1403" H 2650 6150 50  0000 C CNN
 F 1 "BD2" H 2400 5300 50  0000 C CNN
-F 2 "" H 2400 5500 50  0001 C CNN
+F 2 "Package_DIP:DIP-20_W7.62mm" H 2400 5500 50  0001 C CNN
 F 3 "https://assets.nexperia.com/documents/data-sheet/74HC_HCT244.pdf" H 2400 5500 50  0001 C CNN
 	1    2400 5500
@@
 F 0 "J1402" H 3950 3450 50  0000 R CNN
 F 1 "InputAddressSwitches" V 3800 4550 50  0000 R CNN
-F 2 "" H 3850 4300 50  0001 C CNN
+F 2 "Connector_PinHeader_2.54mm:PinHeader_1x16_P2.54mm_Vertical" H 3850 4300 50  0001 C CNN
 F 3 "~" H 3850 4300 50  0001 C CNN
 	1    3850 4300
@@
 F 0 "U1405" H 6100 4150 50  0000 C CNN
 F 1 "BE1" H 5850 3200 50  0000 C CNN
-F 2 "" H 5850 3500 50  0001 C CNN
+F 2 "Package_DIP:DIP-20_W7.62mm" H 5850 3500 50  0001 C CNN
 F 3 "https://assets.nexperia.com/documents/data-sheet/74HC_HCT244.pdf" H 5850 3500 50  0001 C CNN
 	1    5850 3500
@@
 F 0 "U1406" H 6100 6150 50  0000 C CNN
 F 1 "BE2" H 5850 5200 50  0000 C CNN
-F 2 "" H 5850 5500 50  0001 C CNN
+F 2 "Package_DIP:DIP-20_W7.62mm" H 5850 5500 50  0001 C CNN
 F 3 "https://assets.nexperia.com/documents/data-sheet/74HC_HCT244.pdf" H 5850 5500 50  0001 C CNN
 	1    5850 5500
@@
 F 0 "C1402" H 1650 10300 50  0000 L CNN
 F 1 "100nF" H 1600 10100 50  0000 L CNN
-F 2 "" H 1638 10050 50  0001 C CNN
+F 2 "Capacitor_THT:CP_Radial_D5.0mm_P2.50mm" H 1638 10050 50  0001 C CNN
 F 3 "~" H 1600 10200 50  0001 C CNN
 	1    1600 10200
@@
 F 0 "C1401" H 1400 10300 50  0000 L CNN
 F 1 "100nF" H 1350 10100 50  0000 L CNN
-F 2 "" H 1388 10050 50  0001 C CNN
+F 2 "Capacitor_THT:CP_Radial_D5.0mm_P2.50mm" H 1388 10050 50  0001 C CNN
 F 3 "~" H 1350 10200 50  0001 C CNN
 	1    1350 10200
@@
 F 0 "C1404" H 2150 10300 50  0000 L CNN
 F 1 "100nF" H 2100 10100 50  0000 L CNN
-F 2 "" H 2138 10050 50  0001 C CNN
+F 2 "Capacitor_THT:CP_Radial_D5.0mm_P2.50mm" H 2138 10050 50  0001 C CNN
 F 3 "~" H 2100 10200 50  0001 C CNN
 	1    2100 10200
@@
 F 0 "C1403" H 1900 10300 50  0000 L CNN
 F 1 "100nF" H 1850 10100 50  0000 L CNN
-F 2 "" H 1888 10050 50  0001 C CNN
+F 2 "Capacitor_THT:CP_Radial_D5.0mm_P2.50mm" H 1888 10050 50  0001 C CNN
 F 3 "~" H 1850 10200 50  0001 C CNN
 	1    1850 10200
@@
 F 0 "C1406" H 2650 10300 50  0000 L CNN
 F 1 "100nF" H 2600 10100 50  0000 L CNN
-F 2 "" H 2638 10050 50  0001 C CNN
+F 2 "Capacitor_THT:CP_Radial_D5.0mm_P2.50mm" H 2638 10050 50  0001 C CNN
 F 3 "~" H 2600 10200 50  0001 C CNN
 	1    2600 10200
@@
 F 0 "C1405" H 2400 10300 50  0000 L CNN
 F 1 "100nF" H 2350 10100 50  0000 L CNN
-F 2 "" H 2388 10050 50  0001 C CNN
+F 2 "Capacitor_THT:CP_Radial_D5.0mm_P2.50mm" H 2388 10050 50  0001 C CNN
 F 3 "~" H 2350 10200 50  0001 C CNN
 	1    2350 10200

Commit message: Correcting footprints errors
Parts:
- C1401, C1402, C1403, C1404, C1405, C1406: footprint Capacitor_THT:CP_Radial_D5.0mm_P2.50mm -> Capacitor_THT:C_Disc_D4.3mm_W1.9mm_P5.00mm
- U1401: value BD1 -> 74HC244
- U1402: value BS1 -> 74HC244
- U1403: value BD2 -> 74HC244
- U1404: value BS2 -> 74HC244
- U1405: value BE1 -> 74HC244
- U1406: value BE2 -> 74HC244
Changed lines of the file:
@@
 AR Path="/60832DB9/60C5807D/60D2B9FB" Ref="U1401"  Part="1"
 F 0 "U1401" H 2600 2200 50  0000 C CNN
-F 1 "BD1" H 2400 1350 50  0000 C CNN
+F 1 "74HC244" H 2400 1250 50  0000 C CNN
 F 2 "Package_DIP:DIP-20_W7.62mm" H 2400 1550 50  0001 C CNN
 F 3 "https://assets.nexperia.com/documents/data-sheet/74HC_HCT244.pdf" H 2400 1550 50  0001 C CNN
@@
 AR Path="/60832DB9/60C5807D/60D2BA07" Ref="U1404"  Part="1"
 F 0 "U1404" H 2650 8150 50  0000 C CNN
-F 1 "BS2" H 2400 7300 50  0000 C CNN
+F 1 "74HC244" H 2400 7200 50  0000 C CNN
 F 2 "Package_DIP:DIP-20_W7.62mm" H 2400 7500 50  0001 C CNN
 F 3 "https://assets.nexperia.com/documents/data-sheet/74HC_HCT244.pdf" H 2400 7500 50  0001 C CNN
@@
 AR Path="/60832DB9/60C5807D/60D2BA33" Ref="U1402"  Part="1"
 F 0 "U1402" H 2650 4150 50  0000 C CNN
-F 1 "BS1" H 2400 3350 50  0000 C CNN
+F 1 "74HC244" H 2400 3200 50  0000 C CNN
 F 2 "Package_DIP:DIP-20_W7.62mm" H 2400 3500 50  0001 C CNN
 F 3 "https://assets.nexperia.com/documents/data-sheet/74HC_HCT244.pdf" H 2400 3500 50  0001 C CNN
@@
 AR Path="/60832DB9/60C5807D/60D2BA65" Ref="U1403"  Part="1"
 F 0 "U1403" H 2650 6150 50  0000 C CNN
-F 1 "BD2" H 2400 5300 50  0000 C CNN
+F 1 "74HC244" H 2400 5200 50  0000 C CNN
 F 2 "Package_DIP:DIP-20_W7.62mm" H 2400 5500 50  0001 C CNN
 F 3 "https://assets.nexperia.com/documents/data-sheet/74HC_HCT244.pdf" H 2400 5500 50  0001 C CNN
@@
 P 5850 3500
 F 0 "U1405" H 6100 4150 50  0000 C CNN
-F 1 "BE1" H 5850 3200 50  0000 C CNN
+F 1 "74HC244" H 5850 3200 50  0000 C CNN
 F 2 "Package_DIP:DIP-20_W7.62mm" H 5850 3500 50  0001 C CNN
 F 3 "https://assets.nexperia.com/documents/data-sheet/74HC_HCT244.pdf" H 5850 3500 50  0001 C CNN
@@
 P 5850 5500
 F 0 "U1406" H 6100 6150 50  0000 C CNN
-F 1 "BE2" H 5850 5200 50  0000 C CNN
+F 1 "74HC244" H 5850 5200 50  0000 C CNN
 F 2 "Package_DIP:DIP-20_W7.62mm" H 5850 5500 50  0001 C CNN
 F 3 "https://assets.nexperia.com/documents/data-sheet/74HC_HCT244.pdf" H 5850 5500 50  0001 C CNN
@@
 F 0 "C1402" H 1650 10300 50  0000 L CNN
 F 1 "100nF" H 1600 10100 50  0000 L CNN
-F 2 "Capacitor_THT:CP_Radial_D5.0mm_P2.50mm" H 1638 10050 50  0001 C CNN
+F 2 "Capacitor_THT:C_Disc_D4.3mm_W1.9mm_P5.00mm" H 1638 10050 50  0001 C CNN
 F 3 "~" H 1600 10200 50  0001 C CNN
 	1    1600 10200
@@
 F 0 "C1401" H 1400 10300 50  0000 L CNN
 F 1 "100nF" H 1350 10100 50  0000 L CNN
-F 2 "Capacitor_THT:CP_Radial_D5.0mm_P2.50mm" H 1388 10050 50  0001 C CNN
+F 2 "Capacitor_THT:C_Disc_D4.3mm_W1.9mm_P5.00mm" H 1388 10050 50  0001 C CNN
 F 3 "~" H 1350 10200 50  0001 C CNN
 	1    1350 10200
@@
 F 0 "C1404" H 2150 10300 50  0000 L CNN
 F 1 "100nF" H 2100 10100 50  0000 L CNN
-F 2 "Capacitor_THT:CP_Radial_D5.0mm_P2.50mm" H 2138 10050 50  0001 C CNN
+F 2 "Capacitor_THT:C_Disc_D4.3mm_W1.9mm_P5.00mm" H 2138 10050 50  0001 C CNN
 F 3 "~" H 2100 10200 50  0001 C CNN
 	1    2100 10200
@@
 F 0 "C1403" H 1900 10300 50  0000 L CNN
 F 1 "100nF" H 1850 10100 50  0000 L CNN
-F 2 "Capacitor_THT:CP_Radial_D5.0mm_P2.50mm" H 1888 10050 50  0001 C CNN
+F 2 "Capacitor_THT:C_Disc_D4.3mm_W1.9mm_P5.00mm" H 1888 10050 50  0001 C CNN
 F 3 "~" H 1850 10200 50  0001 C CNN
 	1    1850 10200
@@
 F 0 "C1406" H 2650 10300 50  0000 L CNN
 F 1 "100nF" H 2600 10100 50  0000 L CNN
-F 2 "Capacitor_THT:CP_Radial_D5.0mm_P2.50mm" H 2638 10050 50  0001 C CNN
+F 2 "Capacitor_THT:C_Disc_D4.3mm_W1.9mm_P5.00mm" H 2638 10050 50  0001 C CNN
 F 3 "~" H 2600 10200 50  0001 C CNN
 	1    2600 10200
@@
 F 0 "C1405" H 2400 10300 50  0000 L CNN
 F 1 "100nF" H 2350 10100 50  0000 L CNN
-F 2 "Capacitor_THT:CP_Radial_D5.0mm_P2.50mm" H 2388 10050 50  0001 C CNN
+F 2 "Capacitor_THT:C_Disc_D4.3mm_W1.9mm_P5.00mm" H 2388 10050 50  0001 C CNN
 F 3 "~" H 2350 10200 50  0001 C CNN
 	1    2350 10200
