File: CES/Unused.sch (KiCad schematic (older format))
At the start: 5 parts, among them U1001 74HC02, U1003 74HC10, U1004 74HC08, U1501 74HC00, U1601 74HC04

Commit message: Assigning footprints and generating netlist
Parts:
- U1001, U1003, U1004, U1501, U1601: footprint (none) -> Package_DIP:DIP-14_W7.62mm
Changed lines of the file:
@@
 F 0 "U1501" H 1500 1475 50  0000 C CNN
 F 1 "74HC00" H 1500 1384 50  0000 C CNN
-F 2 "" H 1500 1150 50  0001 C CNN
+F 2 "Package_DIP:DIP-14_W7.62mm" H 1500 1150 50  0001 C CNN
 F 3 "http://www.ti.com/lit/gpn/sn74hc00" H 1500 1150 50  0001 C CNN
 	3    1500 1150
@@
 F 0 "U1501" H 1500 2075 50  0000 C CNN
 F 1 "74HC00" H 1500 1984 50  0000 C CNN
-F 2 "" H 1500 1750 50  0001 C CNN
+F 2 "Package_DIP:DIP-14_W7.62mm" H 1500 1750 50  0001 C CNN
 F 3 "http://www.ti.com/lit/gpn/sn74hc00" H 1500 1750 50  0001 C CNN
 	4    1500 1750
@@
 F 0 "U1601" H 1500 3117 50  0000 C CNN
 F 1 "74HC04" H 1500 3026 50  0000 C CNN
-F 2 "" H 1500 2800 50  0001 C CNN
+F 2 "Package_DIP:DIP-14_W7.62mm" H 1500 2800 50  0001 C CNN
 F 3 "https://assets.nexperia.com/documents/data-sheet/74HC_HCT04.pdf" H 1500 2800 50  0001 C CNN
 	3    1500 2800
@@
 F 0 "U1601" H 1500 4017 50  0000 C CNN
 F 1 "74HC04" H 1500 3926 50  0000 C CNN
-F 2 "" H 1500 3700 50  0001 C CNN
+F 2 "Package_DIP:DIP-14_W7.62mm" H 1500 3700 50  0001 C CNN
 F 3 "https://assets.nexperia.com/documents/data-sheet/74HC_HCT04.pdf" H 1500 3700 50  0001 C CNN
 	5    1500 3700
@@
 F 0 "U1601" H 1500 4467 50  0000 C CNN
 F 1 "74HC04" H 1500 4376 50  0000 C CNN
-F 2 "" H 1500 4150 50  0001 C CNN
+F 2 "Package_DIP:DIP-14_W7.62mm" H 1500 4150 50  0001 C CNN
 F 3 "https://assets.nexperia.com/documents/data-sheet/74HC_HCT04.pdf" H 1500 4150 50  0001 C CNN
 	6    1500 4150
@@
 F 0 "U1601" H 1500 3567 50  0000 C CNN
 F 1 "74HC04" H 1500 3476 50  0000 C CNN
-F 2 "" H 1500 3250 50  0001 C CNN
+F 2 "Package_DIP:DIP-14_W7.62mm" H 1500 3250 50  0001 C CNN
 F 3 "https://assets.nexperia.com/documents/data-sheet/74HC_HCT04.pdf" H 1500 3250 50  0001 C CNN
 	4    1500 3250
@@
 F 0 "U1001" H 3700 1525 50  0000 C CNN
 F 1 "74HC02" H 3700 1434 50  0000 C CNN
-F 2 "" H 3700 1200 50  0001 C CNN
+F 2 "Package_DIP:DIP-14_W7.62mm" H 3700 1200 50  0001 C CNN
 F 3 "http://www.ti.com/lit/gpn/sn74hc02" H 3700 1200 50  0001 C CNN
 	2    3700 1200
@@
 F 0 "U1004" H 3700 3225 50  0000 C CNN
 F 1 "74HC08" H 3700 3134 50  0000 C CNN
-F 2 "" H 3700 2900 50  0001 C CNN
+F 2 "Package_DIP:DIP-14_W7.62mm" H 3700 2900 50  0001 C CNN
 F 3 "http://www.ti.com/lit/gpn/sn74HC08" H 3700 2900 50  0001 C CNN
 	4    3700 2900
@@
 F 0 "U1004" H 3700 2675 50  0000 C CNN
 F 1 "74HC08" H 3700 2584 50  0000 C CNN
-F 2 "" H 3700 2350 50  0001 C CNN
+F 2 "Package_DIP:DIP-14_W7.62mm" H 3700 2350 50  0001 C CNN
 F 3 "http://www.ti.com/lit/gpn/sn74HC08" H 3700 2350 50  0001 C CNN
 	3    3700 2350
@@
 F 0 "U1004" H 3700 2075 50  0000 C CNN
 F 1 "74HC08" H 3700 1984 50  0000 C CNN
-F 2 "" H 3700 1750 50  0001 C CNN
+F 2 "Package_DIP:DIP-14_W7.62mm" H 3700 1750 50  0001 C CNN
 F 3 "http://www.ti.com/lit/gpn/sn74HC08" H 3700 1750 50  0001 C CNN
 	2    3700 1750
@@
 F 0 "U1003" H 3700 3775 50  0000 C CNN
 F 1 "74HC10" H 3700 3684 50  0000 C CNN
-F 2 "" H 3700 3450 50  0001 C CNN
+F 2 "Package_DIP:DIP-14_W7.62mm" H 3700 3450 50  0001 C CNN
 F 3 "http://www.ti.com/lit/gpn/sn74HC10" H 3700 3450 50  0001 C CNN
 	3    3700 3450

Commit message: Correcting footprints errors
Parts:
- renumbered U1004 to U1002, U1001 to U1003, U1003 to U1004
Changed lines of the file:
@@
 	1100 1250 1100 1650
 $Comp
-L power:GND #PWR0103
+L power:GND #PWR01802
 U 1 1 6101549C
 P 1100 1950
-F 0 "#PWR0103" H 1100 1700 50  0001 C CNN
+F 0 "#PWR01802" H 1100 1700 50  0001 C CNN
 F 1 "GND" H 1105 1777 50  0000 C CNN
 F 2 "" H 1100 1950 50  0001 C CNN
@@
 P 1050 4300
 AR Path="/611BF25E/6101E694" Ref="#PWR?"  Part="1"
-AR Path="/610111E8/6101E694" Ref="#PWR0104"  Part="1"
-F 0 "#PWR0104" H 1050 4050 50  0001 C CNN
+AR Path="/610111E8/6101E694" Ref="#PWR01801"  Part="1"
+F 0 "#PWR01801" H 1050 4050 50  0001 C CNN
 F 1 "GND" H 1055 4127 50  0000 C CNN
 F 2 "" H 1050 4300 50  0001 C CNN
@@
 P 3300 1950
 AR Path="/60832C87/61038A08" Ref="#PWR?"  Part="1"
-AR Path="/610111E8/61038A08" Ref="#PWR0105"  Part="1"
-F 0 "#PWR0105" H 3300 1700 50  0001 C CNN
+AR Path="/610111E8/61038A08" Ref="#PWR01804"  Part="1"
+F 0 "#PWR01804" H 3300 1700 50  0001 C CNN
 F 1 "GND" H 3305 1777 50  0000 C CNN
 F 2 "" H 3300 1950 50  0001 C CNN
@@
 P 3300 1400
 AR Path="/60832C87/61038A13" Ref="#PWR?"  Part="1"
-AR Path="/610111E8/61038A13" Ref="#PWR0106"  Part="1"
-F 0 "#PWR0106" H 3300 1150 50  0001 C CNN
+AR Path="/610111E8/61038A13" Ref="#PWR01803"  Part="1"
+F 0 "#PWR01803" H 3300 1150 50  0001 C CNN
 F 1 "GND" H 3305 1227 50  0000 C CNN
 F 2 "" H 3300 1400 50  0001 C CNN
@@
 P 3300 2550
 AR Path="/60832C87/61038A1F" Ref="#PWR?"  Part="1"
-AR Path="/610111E8/61038A1F" Ref="#PWR0107"  Part="1"
-F 0 "#PWR0107" H 3300 2300 50  0001 C CNN
+AR Path="/610111E8/61038A1F" Ref="#PWR01805"  Part="1"
+F 0 "#PWR01805" H 3300 2300 50  0001 C CNN
 F 1 "GND" H 3305 2377 50  0000 C CNN
 F 2 "" H 3300 2550 50  0001 C CNN
@@
 P 3300 3100
 AR Path="/60832C87/61038A2A" Ref="#PWR?"  Part="1"
-AR Path="/610111E8/61038A2A" Ref="#PWR0108"  Part="1"
-F 0 "#PWR0108" H 3300 2850 50  0001 C CNN
+AR Path="/610111E8/61038A2A" Ref="#PWR01806"  Part="1"
+F 0 "#PWR01806" H 3300 2850 50  0001 C CNN
 F 1 "GND" H 3305 2927 50  0000 C CNN
 F 2 "" H 3300 3100 50  0001 C CNN
@@
 P 3300 3650
 AR Path="/60832C87/61038A35" Ref="#PWR?"  Part="1"
-AR Path="/610111E8/61038A35" Ref="#PWR0109"  Part="1"
-F 0 "#PWR0109" H 3300 3400 50  0001 C CNN
+AR Path="/610111E8/61038A35" Ref="#PWR01807"  Part="1"
+F 0 "#PWR01807" H 3300 3400 50  0001 C CNN
 F 1 "GND" H 3305 3477 50  0000 C CNN
 F 2 "" H 3300 3650 50  0001 C CNN
@@
 P 3700 1200
 AR Path="/60832C87/61038A46" Ref="U?"  Part="2"
-AR Path="/610111E8/61038A46" Ref="U1001"  Part="2"
-F 0 "U1001" H 3700 1525 50  0000 C CNN
+AR Path="/610111E8/61038A46" Ref="U1003"  Part="2"
+F 0 "U1003" H 3700 1525 50  0000 C CNN
 F 1 "74HC02" H 3700 1434 50  0000 C CNN
 F 2 "Package_DIP:DIP-14_W7.62mm" H 3700 1200 50  0001 C CNN
@@
 P 3700 2900
 AR Path="/60832C87/61038A4C" Ref="U?"  Part="4"
-AR Path="/610111E8/61038A4C" Ref="U1004"  Part="4"
-F 0 "U1004" H 3700 3225 50  0000 C CNN
+AR Path="/610111E8/61038A4C" Ref="U1002"  Part="4"
+F 0 "U1002" H 3700 3225 50  0000 C CNN
 F 1 "74HC08" H 3700 3134 50  0000 C CNN
 F 2 "Package_DIP:DIP-14_W7.62mm" H 3700 2900 50  0001 C CNN
@@
 P 3700 2350
 AR Path="/60832C87/61038A52" Ref="U?"  Part="3"
-AR Path="/610111E8/61038A52" Ref="U1004"  Part="3"
-F 0 "U1004" H 3700 2675 50  0000 C CNN
+AR Path="/610111E8/61038A52" Ref="U1002"  Part="3"
+F 0 "U1002" H 3700 2675 50  0000 C CNN
 F 1 "74HC08" H 3700 2584 50  0000 C CNN
 F 2 "Package_DIP:DIP-14_W7.62mm" H 3700 2350 50  0001 C CNN
@@
 P 3700 1750
 AR Path="/60832C87/61038A58" Ref="U?"  Part="2"
-AR Path="/610111E8/61038A58" Ref="U1004"  Part="2"
-F 0 "U1004" H 3700 2075 50  0000 C CNN
+AR Path="/610111E8/61038A58" Ref="U1002"  Part="2"
+F 0 "U1002" H 3700 2075 50  0000 C CNN
 F 1 "74HC08" H 3700 1984 50  0000 C CNN
 F 2 "Package_DIP:DIP-14_W7.62mm" H 3700 1750 50  0001 C CNN
@@
 P 3700 3450
 AR Path="/60832C87/61038A5E" Ref="U?"  Part="3"
-AR Path="/610111E8/61038A5E" Ref="U1003"  Part="3"
-F 0 "U1003" H 3700 3775 50  0000 C CNN
+AR Path="/610111E8/61038A5E" Ref="U1004"  Part="3"
+F 0 "U1004" H 3700 3775 50  0000 C CNN
 F 1 "74HC10" H 3700 3684 50  0000 C CNN
 F 2 "Package_DIP:DIP-14_W7.62mm" H 3700 3450 50  0001 C CNN
