File: CES/CES.kicad_pcb (KiCad board)
At the start: 2 copper layers, 170 parts, among them J101 Barrel_Jack, J1201 PannelPowerConnector, J1301 Conn_01x16, J1302 Conn_01x16, J1303 Conn_01x16, J1401 InputDataSwitches, J1402 InputAddressSwitches, J1501 PannelButtonsConnector, J1601 Conn_02x12, J1701 Conn_01x16, J1702 Conn_01x16, J1703 Conn_01x16, J1704 Conn_01x07, U1001 74HC30, U1002 74HC08, U1003 74HC02, U1004 74HC10, U1101 SST39SF020, U1102 SST39SF020, U1103 IS61C256, U1104 IS61C256, U1301 74HC04, U1302 74HC04, U1303 74HC04, U1304 74HC04, U1305 74HC04, U1306 74HC04, U1307 74HC04, U1308 74HC04, U1401 74HC244, U1402 74HC244, U1403 74HC244, U1404 74HC244, U1405 74HC244, U1406 74HC244, U1501 74HC00, U1502 74HC14, U1601 74HC04, U1602 74HC4040, U201 74HC02, U202 74HC02, U203 74HC02, U204 74HC02, U205 74HC283, U206 74HC283, U207 74HC283, U208 74HC283, U209 74HC257, U210 74HC257, U211 74HC257, U212 74HC257, U401 74HC173, U402 74HC173, U403 74HC173, U404 74HC173, U405 74HC244, U406 74HC244, U501 74HC173, U502 74HC173, U503 74HC173, U504 74HC173, U601 74HC173, U602 74HC173, U603 74HC173, U604 74HC173, U701 74HC173, U702 74HC173, U703 74HC173, U704 74HC173, U801 74HC21, U802 74HC20, U803 74HC00, U804 74HC02, U805 74HC27, U806 74HC27, U807 74HC02, U808 74HC20, U809 74HC00, U901 74HC74, U902 74HC175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

Commit message: All adders, registers and multiplexers in place
Parts:
- moved C1401 1359.2 mm to (-630.4, -118.2)
- moved C1402 1359.2 mm to (-614.1, -118.2)
- moved C1405 1359.2 mm to (-622.3, -118.2)
- moved U1403 1359.2 mm to (-597.8, -144.9)
- moved U1405 1359.2 mm to (-619.5, -144.9)
- moved U1406 1359.2 mm to (-630.4, -144.9)
- moved C1501 1071.3 mm to (-560.1, 67.9)
- moved C1601 1071.3 mm to (-402.7, 147.9)
- moved C1602 1071.3 mm to (-391.8, 133.7)
- moved C1603 1071.3 mm to (-413.5, 153.8)
- moved C1604 1071.3 mm to (-413.5, 157.3)
- moved C1605 1071.3 mm to (-413.5, 150.4)
- moved J1201 1071.3 mm to (-588.8, 89.2)
- moved J1501 1071.3 mm to (-564.0, 49.1)
- moved J1601 1071.3 mm to (-420.0, 129.1)
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Connections:
- J1703 pad 7: SRT5 -> SRT6
- U1302 pad 1: SRT5 -> SRT6
- U202 pad 8: SRT5 -> SRT6
- U402 pad 5: SRT5 -> SRT6
- U405 pad 13: SRT5 -> SRT6
Routing:
- net (no net): track 1549.6 -> 0.08 mm, vias 28 -> 0
- net VDB8: track 0.00 -> 153.7 mm, vias 0 -> 2
- net VDB9: track 0.00 -> 153.3 mm, vias 0 -> 3
- net VDB11: track 0.00 -> 148.2 mm, vias 0 -> 3
- net VDB10: track 0.00 -> 144.2 mm, vias 0 -> 3
- net VDB13: track 0.00 -> 114.9 mm, vias 0 -> 3
- net SRT15: track 0.00 -> 112.5 mm, vias 0 -> 1
- net VDB12: track 0.00 -> 109.8 mm, vias 0 -> 2
- net VDB15: track 0.00 -> 107.8 mm, vias 0 -> 3
- net VDB14: track 0.00 -> 104.0 mm, vias 0 -> 3
- net SRT13: track 0.00 -> 104.0 mm, vias 0 -> 1
- net SRT14: track 0.00 -> 96.7 mm, vias 0 -> 1
- net SRT6: track 0.00 -> 96.3 mm, vias 0 -> 1
- net SRT12: track 0.00 -> 92.2 mm, vias 0 -> 1
- net SS9: track 0.00 -> 78.8 mm, vias 0 -> 2
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